Commit message: semi working version of challenge2 example

File: mbzirc_gazebo_simulation/challenge_worlds/urdf/blue_pile.xacro (robot description, xacro)
@@ -1,2 +1,2 @@
-<?xml version="1.0"?><robot xmlns:xacro="http://www.ros.org/wiki/xacro"><xacro:include filename="$(find challenge_worlds)/urdf/includes/brick_link.xacro" /><macro name="blue_pile" params="id pose"><model name="${id}.pile"><pose>${pose}</pose><self_collide>true</self_collide>
-<brick_link id="0" type="brick" sx="1.2" sy="0.2" sz="0.2" mass="1.5" material="Gazebo/Blue" pose="0.0 0.0 0.1 0 0 0" /><brick_link id="1" type="brick" sx="1.2" sy="0.2" sz="0.2" mass="1.5" material="Gazebo/Blue" pose="0.0 0.0 0.32 0 0 0" /><brick_link id="2" type="brick" sx="1.2" sy="0.2" sz="0.2" mass="1.5" material="Gazebo/Blue" pose="0.0 0.2 0.1 0 0 0" /><brick_link id="3" type="brick" sx="1.2" sy="0.2" sz="0.2" mass="1.5" material="Gazebo/Blue" pose="0.0 0.2 0.32 0 0 0" /><brick_link id="4" type="brick" sx="1.2" sy="0.2" sz="0.2" mass="1.5" material="Gazebo/Blue" pose="0.0 0.4 0.1 0 0 0" /><brick_link id="5" type="brick" sx="1.2" sy="0.2" sz="0.2" mass="1.5" material="Gazebo/Blue" pose="0.0 0.4 0.32 0 0 0" /><brick_link id="6" type="brick" sx="1.2" sy="0.2" sz="0.2" mass="1.5" material="Gazebo/Blue" pose="1.2 0.0 0.1 0 0 0" /><brick_link id="7" type="brick" sx="1.2" sy="0.2" sz="0.2" mass="1.5" material="Gazebo/Blue" pose="1.2 0.0 0.32 0 0 0" /><brick_link id="8" type="brick" sx="1.2" sy="0.2" sz="0.2" mass="1.5" material="Gazebo/Blue" pose="1.2 0.2 0.1 0 0 0" /><brick_link id="9" type="brick" sx="1.2" sy="0.2" sz="0.2" mass="1.5" material="Gazebo/Blue" pose="1.2 0.2 0.32 0 0 0" /><brick_link id="10" type="brick" sx="1.2" sy="0.2" sz="0.2" mass="1.5" material="Gazebo/Blue" pose="1.2 0.4 0.1 0 0 0" /><brick_link id="11" type="brick" sx="1.2" sy="0.2" sz="0.2" mass="1.5" material="Gazebo/Blue" pose="1.2 0.4 0.32 0 0 0" /><brick_link id="12" type="brick" sx="1.2" sy="0.2" sz="0.2" mass="1.5" material="Gazebo/Blue" pose="2.4 0.0 0.1 0 0 0" /><brick_link id="13" type="brick" sx="1.2" sy="0.2" sz="0.2" mass="1.5" material="Gazebo/Blue" pose="2.4 0.0 0.32 0 0 0" /><brick_link id="14" type="brick" sx="1.2" sy="0.2" sz="0.2" mass="1.5" material="Gazebo/Blue" pose="2.4 0.2 0.1 0 0 0" /><brick_link id="15" type="brick" sx="1.2" sy="0.2" sz="0.2" mass="1.5" material="Gazebo/Blue" pose="2.4 0.2 0.32 0 0 0" /><brick_link id="16" type="brick" sx="1.2" sy="0.2" sz="0.2" mass="1.5" material="Gazebo/Blue" pose="2.4 0.4 0.1 0 0 0" /><brick_link id="17" type="brick" sx="1.2" sy="0.2" sz="0.2" mass="1.5" material="Gazebo/Blue" pose="2.4 0.4 0.32 0 0 0" /></model></macro></robot>
+<?xml version="1.0"?><robot xmlns:xacro="http://www.ros.org/wiki/xacro"><xacro:include filename="$(find challenge_worlds)/urdf/includes/brick_link.xacro" /><macro name="blue_pile" params="id pose"><model name="${id}.pile"><pose>${pose}</pose>
+<brick_link id="0" id2="${id}" type="brick" sx="1.2" sy="0.2" sz="0.2" mass="1.5" material="Gazebo/Blue" pose="0.0 0.0 0.1 0 0 0" /><brick_link id="1" id2="${id}" type="brick" sx="1.2" sy="0.2" sz="0.2" mass="1.5" material="Gazebo/Blue" pose="0.0 0.2 0.1 0 0 0" /><brick_link id="2" id2="${id}" type="brick" sx="1.2" sy="0.2" sz="0.2" mass="1.5" material="Gazebo/Blue" pose="1.2 0.0 0.1 0 0 0" /><brick_link id="3" id2="${id}" type="brick" sx="1.2" sy="0.2" sz="0.2" mass="1.5" material="Gazebo/Blue" pose="1.2 0.2 0.1 0 0 0" /></model></macro></robot>

File: mbzirc_gazebo_simulation/challenge_worlds/urdf/green_pile.xacro (robot description, xacro)
@@ -1,2 +1,2 @@
-<?xml version="1.0"?><robot xmlns:xacro="http://www.ros.org/wiki/xacro"><xacro:include filename="$(find challenge_worlds)/urdf/includes/brick_link.xacro" /><macro name="green_pile" params="id pose"><model name="${id}.pile"><pose>${pose}</pose><self_collide>true</self_collide>
-<brick_link id="0" type="brick" sx="0.6" sy="0.2" sz="0.2" mass="1.0" material="Gazebo/Green" pose="0.0 0.0 0.1 0 0 0" /><brick_link id="1" type="brick" sx="0.6" sy="0.2" sz="0.2" mass="1.0" material="Gazebo/Green" pose="0.0 0.0 0.32 0 0 0" /><brick_link id="2" type="brick" sx="0.6" sy="0.2" sz="0.2" mass="1.0" material="Gazebo/Green" pose="0.0 0.2 0.1 0 0 0" /><brick_link id="3" type="brick" sx="0.6" sy="0.2" sz="0.2" mass="1.0" material="Gazebo/Green" pose="0.0 0.2 0.32 0 0 0" /><brick_link id="4" type="brick" sx="0.6" sy="0.2" sz="0.2" mass="1.0" material="Gazebo/Green" pose="0.0 0.4 0.1 0 0 0" /><brick_link id="5" type="brick" sx="0.6" sy="0.2" sz="0.2" mass="1.0" material="Gazebo/Green" pose="0.0 0.4 0.32 0 0 0" /><brick_link id="6" type="brick" sx="0.6" sy="0.2" sz="0.2" mass="1.0" material="Gazebo/Green" pose="0.6 0.0 0.1 0 0 0" /><brick_link id="7" type="brick" sx="0.6" sy="0.2" sz="0.2" mass="1.0" material="Gazebo/Green" pose="0.6 0.0 0.32 0 0 0" /><brick_link id="8" type="brick" sx="0.6" sy="0.2" sz="0.2" mass="1.0" material="Gazebo/Green" pose="0.6 0.2 0.1 0 0 0" /><brick_link id="9" type="brick" sx="0.6" sy="0.2" sz="0.2" mass="1.0" material="Gazebo/Green" pose="0.6 0.2 0.32 0 0 0" /><brick_link id="10" type="brick" sx="0.6" sy="0.2" sz="0.2" mass="1.0" material="Gazebo/Green" pose="0.6 0.4 0.1 0 0 0" /><brick_link id="11" type="brick" sx="0.6" sy="0.2" sz="0.2" mass="1.0" material="Gazebo/Green" pose="0.6 0.4 0.32 0 0 0" /><brick_link id="12" type="brick" sx="0.6" sy="0.2" sz="0.2" mass="1.0" material="Gazebo/Green" pose="1.2 0.0 0.1 0 0 0" /><brick_link id="13" type="brick" sx="0.6" sy="0.2" sz="0.2" mass="1.0" material="Gazebo/Green" pose="1.2 0.0 0.32 0 0 0" /><brick_link id="14" type="brick" sx="0.6" sy="0.2" sz="0.2" mass="1.0" material="Gazebo/Green" pose="1.2 0.2 0.1 0 0 0" /><brick_link id="15" type="brick" sx="0.6" sy="0.2" sz="0.2" mass="1.0" material="Gazebo/Green" pose="1.2 0.2 0.32 0 0 0" /><brick_link id="16" type="brick" sx="0.6" sy="0.2" sz="0.2" mass="1.0" material="Gazebo/Green" pose="1.2 0.4 0.1 0 0 0" /><brick_link id="17" type="brick" sx="0.6" sy="0.2" sz="0.2" mass="1.0" material="Gazebo/Green" pose="1.2 0.4 0.32 0 0 0" /></model></macro></robot>
+<?xml version="1.0"?><robot xmlns:xacro="http://www.ros.org/wiki/xacro"><xacro:include filename="$(find challenge_worlds)/urdf/includes/brick_link.xacro" /><macro name="green_pile" params="id pose"><model name="${id}.pile"><pose>${pose}</pose>
+<brick_link id="0" id2="${id}" type="brick" sx="0.6" sy="0.2" sz="0.2" mass="1.0" material="Gazebo/Green" pose="0.0 0.0 0.1 0 0 0" /><brick_link id="1" id2="${id}" type="brick" sx="0.6" sy="0.2" sz="0.2" mass="1.0" material="Gazebo/Green" pose="0.0 0.2 0.1 0 0 0" /><brick_link id="2" id2="${id}" type="brick" sx="0.6" sy="0.2" sz="0.2" mass="1.0" material="Gazebo/Green" pose="0.6 0.0 0.1 0 0 0" /><brick_link id="3" id2="${id}" type="brick" sx="0.6" sy="0.2" sz="0.2" mass="1.0" material="Gazebo/Green" pose="0.6 0.2 0.1 0 0 0" /></model></macro></robot>

File: mbzirc_gazebo_simulation/challenge_worlds/urdf/includes/brick_link.xacro (robot description, xacro)
@@ -1,5 +1,6 @@
 <?xml version="1.0"?>
 <robot xmlns:xacro="http://www.ros.org/wiki/xacro">
-<macro name="brick_link" params="id type pose sx sy sz mass material">
+<macro name="brick_link" params="id id2 type pose sx sy sz mass material">
+<model name="${id2}.${id}.pile">
 	<link name="${id}.${type}">
             <pose>${pose}</pose>
@@ -33,4 +34,5 @@
             </collision>
         </link>
+</model>
 </macro>
 </robot>

File: mbzirc_gazebo_simulation/challenge_worlds/urdf/orange_pile.xacro (robot description, xacro)
@@ -1,2 +1,2 @@
-<?xml version="1.0"?><robot xmlns:xacro="http://www.ros.org/wiki/xacro"><xacro:include filename="$(find challenge_worlds)/urdf/includes/brick_link.xacro" /><macro name="orange_pile" params="id pose"><model name="${id}.pile"><pose>${pose}</pose><self_collide>true</self_collide>
-<brick_link id="0" type="brick" sx="1.8" sy="0.2" sz="0.2" mass="2.0" material="Gazebo/Orange" pose="0.0 0.0 0.1 0 0 0" /><brick_link id="1" type="brick" sx="1.8" sy="0.2" sz="0.2" mass="2.0" material="Gazebo/Orange" pose="0.0 0.0 0.32 0 0 0" /><brick_link id="2" type="brick" sx="1.8" sy="0.2" sz="0.2" mass="2.0" material="Gazebo/Orange" pose="0.0 0.0 0.54 0 0 0" /><brick_link id="3" type="brick" sx="1.8" sy="0.2" sz="0.2" mass="2.0" material="Gazebo/Orange" pose="0.0 0.2 0.1 0 0 0" /><brick_link id="4" type="brick" sx="1.8" sy="0.2" sz="0.2" mass="2.0" material="Gazebo/Orange" pose="0.0 0.2 0.32 0 0 0" /><brick_link id="5" type="brick" sx="1.8" sy="0.2" sz="0.2" mass="2.0" material="Gazebo/Orange" pose="0.0 0.2 0.54 0 0 0" /><brick_link id="6" type="brick" sx="1.8" sy="0.2" sz="0.2" mass="2.0" material="Gazebo/Orange" pose="0.0 0.4 0.1 0 0 0" /><brick_link id="7" type="brick" sx="1.8" sy="0.2" sz="0.2" mass="2.0" material="Gazebo/Orange" pose="0.0 0.4 0.32 0 0 0" /><brick_link id="8" type="brick" sx="1.8" sy="0.2" sz="0.2" mass="2.0" material="Gazebo/Orange" pose="0.0 0.4 0.54 0 0 0" /><brick_link id="9" type="brick" sx="1.8" sy="0.2" sz="0.2" mass="2.0" material="Gazebo/Orange" pose="1.8 0.0 0.1 0 0 0" /><brick_link id="10" type="brick" sx="1.8" sy="0.2" sz="0.2" mass="2.0" material="Gazebo/Orange" pose="1.8 0.0 0.32 0 0 0" /><brick_link id="11" type="brick" sx="1.8" sy="0.2" sz="0.2" mass="2.0" material="Gazebo/Orange" pose="1.8 0.0 0.54 0 0 0" /><brick_link id="12" type="brick" sx="1.8" sy="0.2" sz="0.2" mass="2.0" material="Gazebo/Orange" pose="1.8 0.2 0.1 0 0 0" /><brick_link id="13" type="brick" sx="1.8" sy="0.2" sz="0.2" mass="2.0" material="Gazebo/Orange" pose="1.8 0.2 0.32 0 0 0" /><brick_link id="14" type="brick" sx="1.8" sy="0.2" sz="0.2" mass="2.0" material="Gazebo/Orange" pose="1.8 0.2 0.54 0 0 0" /><brick_link id="15" type="brick" sx="1.8" sy="0.2" sz="0.2" mass="2.0" material="Gazebo/Orange" pose="1.8 0.4 0.1 0 0 0" /><brick_link id="16" type="brick" sx="1.8" sy="0.2" sz="0.2" mass="2.0" material="Gazebo/Orange" pose="1.8 0.4 0.32 0 0 0" /><brick_link id="17" type="brick" sx="1.8" sy="0.2" sz="0.2" mass="2.0" material="Gazebo/Orange" pose="1.8 0.4 0.54 0 0 0" /><brick_link id="18" type="brick" sx="1.8" sy="0.2" sz="0.2" mass="2.0" material="Gazebo/Orange" pose="3.6 0.0 0.1 0 0 0" /><brick_link id="19" type="brick" sx="1.8" sy="0.2" sz="0.2" mass="2.0" material="Gazebo/Orange" pose="3.6 0.0 0.32 0 0 0" /><brick_link id="20" type="brick" sx="1.8" sy="0.2" sz="0.2" mass="2.0" material="Gazebo/Orange" pose="3.6 0.0 0.54 0 0 0" /><brick_link id="21" type="brick" sx="1.8" sy="0.2" sz="0.2" mass="2.0" material="Gazebo/Orange" pose="3.6 0.2 0.1 0 0 0" /><brick_link id="22" type="brick" sx="1.8" sy="0.2" sz="0.2" mass="2.0" material="Gazebo/Orange" pose="3.6 0.2 0.32 0 0 0" /><brick_link id="23" type="brick" sx="1.8" sy="0.2" sz="0.2" mass="2.0" material="Gazebo/Orange" pose="3.6 0.2 0.54 0 0 0" /><brick_link id="24" type="brick" sx="1.8" sy="0.2" sz="0.2" mass="2.0" material="Gazebo/Orange" pose="3.6 0.4 0.1 0 0 0" /><brick_link id="25" type="brick" sx="1.8" sy="0.2" sz="0.2" mass="2.0" material="Gazebo/Orange" pose="3.6 0.4 0.32 0 0 0" /><brick_link id="26" type="brick" sx="1.8" sy="0.2" sz="0.2" mass="2.0" material="Gazebo/Orange" pose="3.6 0.4 0.54 0 0 0" /></model></macro></robot>
+<?xml version="1.0"?><robot xmlns:xacro="http://www.ros.org/wiki/xacro"><xacro:include filename="$(find challenge_worlds)/urdf/includes/brick_link.xacro" /><macro name="orange_pile" params="id pose"><model name="${id}.pile"><pose>${pose}</pose>
+<brick_link id="0" id2="${id}" type="brick" sx="1.8" sy="0.2" sz="0.2" mass="2.0" material="Gazebo/Orange" pose="0.0 0.0 0.1 0 0 0" /><brick_link id="1" id2="${id}" type="brick" sx="1.8" sy="0.2" sz="0.2" mass="2.0" material="Gazebo/Orange" pose="0.0 0.2 0.1 0 0 0" /><brick_link id="2" id2="${id}" type="brick" sx="1.8" sy="0.2" sz="0.2" mass="2.0" material="Gazebo/Orange" pose="1.8 0.0 0.1 0 0 0" /><brick_link id="3" id2="${id}" type="brick" sx="1.8" sy="0.2" sz="0.2" mass="2.0" material="Gazebo/Orange" pose="1.8 0.2 0.1 0 0 0" /></model></macro></robot>

File: mbzirc_gazebo_simulation/challenge_worlds/urdf/red_pile.xacro (robot description, xacro)
@@ -1,2 +1,2 @@
-<?xml version="1.0"?><robot xmlns:xacro="http://www.ros.org/wiki/xacro"><xacro:include filename="$(find challenge_worlds)/urdf/includes/brick_link.xacro" /><macro name="red_pile" params="id pose"><model name="${id}.pile"><pose>${pose}</pose><self_collide>true</self_collide>
-<brick_link id="0" type="brick" sx="0.3" sy="0.2" sz="0.2" mass="1.0" material="Gazebo/Red" pose="0.0 0.0 0.1 0 0 0" /><brick_link id="1" type="brick" sx="0.3" sy="0.2" sz="0.2" mass="1.0" material="Gazebo/Red" pose="0.0 0.0 0.32 0 0 0" /><brick_link id="2" type="brick" sx="0.3" sy="0.2" sz="0.2" mass="1.0" material="Gazebo/Red" pose="0.0 0.2 0.1 0 0 0" /><brick_link id="3" type="brick" sx="0.3" sy="0.2" sz="0.2" mass="1.0" material="Gazebo/Red" pose="0.0 0.2 0.32 0 0 0" /><brick_link id="4" type="brick" sx="0.3" sy="0.2" sz="0.2" mass="1.0" material="Gazebo/Red" pose="0.0 0.4 0.1 0 0 0" /><brick_link id="5" type="brick" sx="0.3" sy="0.2" sz="0.2" mass="1.0" material="Gazebo/Red" pose="0.0 0.4 0.32 0 0 0" /><brick_link id="6" type="brick" sx="0.3" sy="0.2" sz="0.2" mass="1.0" material="Gazebo/Red" pose="0.3 0.0 0.1 0 0 0" /><brick_link id="7" type="brick" sx="0.3" sy="0.2" sz="0.2" mass="1.0" material="Gazebo/Red" pose="0.3 0.0 0.32 0 0 0" /><brick_link id="8" type="brick" sx="0.3" sy="0.2" sz="0.2" mass="1.0" material="Gazebo/Red" pose="0.3 0.2 0.1 0 0 0" /><brick_link id="9" type="brick" sx="0.3" sy="0.2" sz="0.2" mass="1.0" material="Gazebo/Red" pose="0.3 0.2 0.32 0 0 0" /><brick_link id="10" type="brick" sx="0.3" sy="0.2" sz="0.2" mass="1.0" material="Gazebo/Red" pose="0.3 0.4 0.1 0 0 0" /><brick_link id="11" type="brick" sx="0.3" sy="0.2" sz="0.2" mass="1.0" material="Gazebo/Red" pose="0.3 0.4 0.32 0 0 0" /><brick_link id="12" type="brick" sx="0.3" sy="0.2" sz="0.2" mass="1.0" material="Gazebo/Red" pose="0.6 0.0 0.1 0 0 0" /><brick_link id="13" type="brick" sx="0.3" sy="0.2" sz="0.2" mass="1.0" material="Gazebo/Red" pose="0.6 0.0 0.32 0 0 0" /><brick_link id="14" type="brick" sx="0.3" sy="0.2" sz="0.2" mass="1.0" material="Gazebo/Red" pose="0.6 0.2 0.1 0 0 0" /><brick_link id="15" type="brick" sx="0.3" sy="0.2" sz="0.2" mass="1.0" material="Gazebo/Red" pose="0.6 0.2 0.32 0 0 0" /><brick_link id="16" type="brick" sx="0.3" sy="0.2" sz="0.2" mass="1.0" material="Gazebo/Red" pose="0.6 0.4 0.1 0 0 0" /><brick_link id="17" type="brick" sx="0.3" sy="0.2" sz="0.2" mass="1.0" material="Gazebo/Red" pose="0.6 0.4 0.32 0 0 0" /></model></macro></robot>
+<?xml version="1.0"?><robot xmlns:xacro="http://www.ros.org/wiki/xacro"><xacro:include filename="$(find challenge_worlds)/urdf/includes/brick_link.xacro" /><macro name="red_pile" params="id pose"><model name="${id}.pile"><pose>${pose}</pose>
+<brick_link id="0" id2="${id}" type="brick" sx="0.3" sy="0.2" sz="0.2" mass="1.0" material="Gazebo/Red" pose="0.0 0.0 0.1 0 0 0" /><brick_link id="1" id2="${id}" type="brick" sx="0.3" sy="0.2" sz="0.2" mass="1.0" material="Gazebo/Red" pose="0.0 0.2 0.1 0 0 0" /><brick_link id="2" id2="${id}" type="brick" sx="0.3" sy="0.2" sz="0.2" mass="1.0" material="Gazebo/Red" pose="0.3 0.0 0.1 0 0 0" /><brick_link id="3" id2="${id}" type="brick" sx="0.3" sy="0.2" sz="0.2" mass="1.0" material="Gazebo/Red" pose="0.3 0.2 0.1 0 0 0" /></model></macro></robot>

File: mbzirc_gazebo_simulation/mbzirc_gazebo_plugins/urdf/fake_camera.xacro (robot description, xacro)
@@ -1,5 +1,5 @@
 <?xml version="1.0"?>
 <robot>
-  <macro name="fake_camera" params="parent *origin">
+  <macro name="fake_camera" params="parent *origin robot_name">
   	<joint name="camera_frame_joint" type="fixed">
       <insert_block name="origin" />
@@ -54,5 +54,5 @@
           <plugin name="ros_object_detection" filename="libfake_object_detection_plugin.so">
               	    <topic_name>sensed_objects</topic_name>
-  	                <robot_name>cool_robot</robot_name>
+  	                <robot_name>${robot_name}</robot_name>
           </plugin>
           <always_on>1</always_on>

File: mbzirc_gazebo_simulation/mbzirc_gazebo_plugins/urdf/magnetic_gripper.xacro (robot description, xacro)
@@ -1,5 +1,5 @@
 <?xml version="1.0"?>
 <robot>
-  <macro name="magnetic_gripper" params="parent *origin">
+  <macro name="magnetic_gripper" params="parent *origin robot_name">
     <joint name="gripper_attach_joint" type="fixed">
       <insert_block name="origin" />
@@ -17,5 +17,5 @@
         <origin xyz="0 0 0" rpy="0 0 0"/>
         <geometry>
-          <box size="0.01 0.01 0.01" />
+          <box size="0.1 0.1 0.05" />
         </geometry>
       </collision>
@@ -23,5 +23,5 @@
         <origin xyz="0 0 0" rpy="0 0 0"/>
         <geometry>
-          <box size="0.01 0.01 0.01" />
+          <box size="0.1 0.1 0.05" />
         </geometry>
       </visual>
@@ -29,5 +29,5 @@
     <gazebo>
       <plugin name="ros_gripper" filename="libmagnetic_gripper_plugin.so">
-            <robot_name>test_gripper</robot_name>
+            <robot_name>${robot_name}</robot_name>
             <!-- We are forced to magnetize the parent link because of gazebo
                  automatically lumping fixed joints. This can be prevented just from
