Commit message: Fixing ch1 simulation. Configuring balloons as the new rules describe

File: mbzirc_gazebo_simulation/challenge_worlds/urdf/balloon.xacro (robot description, xacro)
@@ -9,5 +9,4 @@
     <xacro:arg name="height"     default="2"/>
     <xacro:arg name="colour"      default="Gazebo/red"/>
-    <xacro:property name="mesh_balloon"                value="$(find challenge_worlds)/meshes/balloon.dae" />
     <xacro:property name="balloon_radio"               value="0.24"/>
     <xacro:property name="balloon_height"              value="0.36"/>
@@ -524,8 +523,7 @@
         <visual name='visual'>
           <geometry>
-            <mesh>
-              <uri>${mesh_balloon}</uri>
-              <scale>${balloon_model_scale_factor*balloon_radio} ${balloon_model_scale_factor*balloon_radio} ${balloon_model_scale_factor*balloon_radio}</scale>
-            </mesh>
+            <sphere>
+              <radius>0.3</radius>
+            </sphere>
           </geometry>
           <material>

File: mbzirc_gazebo_simulation/uavs_description/models/iris_target_drone/model.xacro (robot description, xacro)
@@ -2,10 +2,13 @@
 <robot name="iris" xmlns:xacro="http://ros.org/wiki/xacro">
   <xacro:arg name="bar_l"           default="1.0"/>
-  <xacro:arg name="ball_r"          default="0.09"/>
-  <xacro:arg name="ball_colour"     default="Gazebo/Green"/>
+  <xacro:arg name="bar_r"           default="0.005"/>
+  <xacro:arg name="bar_mass"        default="0.005"/>
+  <xacro:arg name="ball_r"          default="0.07"/>
+  <xacro:arg name="ball_colour"     default="Gazebo/Red"/>
+  <xacro:arg name="ball_mass"       default="0.09"/>
   <!-- Instantiate robots_description iris -->
   <xacro:include filename="$(find robots_description)/models/iris/model.xacro" />
   <!-- Bar-ball system -->
-  <link name="foo">
+  <link name="base_union">
     <inertial>
       <origin xyz="0 0 0"/>
@@ -26,33 +29,33 @@
     </collision>
   </link>
-  <joint name="base_link_to_foo_joint" type="continuous">
+  <joint name="base_link_to_base_union_joint" type="continuous">
     <origin xyz="0 0 0"/>
     <axis xyz="1 0 0"/>
     <parent link="base_link"/>
-    <child link="foo"/>
+    <child link="base_union"/>
   </joint>
   <link name="bar">
     <inertial>
-      <origin xyz="0 0 -${$(arg bar_l)/2}"/>
-      <mass value="0.005"/>
-      <inertia ixx="1e-06" ixy="0" ixz="0" iyy="1e-06" iyz="0" izz="9e-06"/>
+      <origin xyz="0 ${$(arg bar_l)/2} 0" rpy="1.5707963267948966 0 0"/>
+      <mass value="${arg bar_mass}"/>
+      <inertia ixx="${(1/12)*${arg bar_mass}*(3*${arg bar_r}*${arg bar_r}+${arg bar_l}*${arg bar_l})}" ixy="0" ixz="0" iyy="${(1/12)*${arg bar_mass}*(3*${arg bar_r}*${arg bar_r}+${arg bar_l}*${arg bar_l})}" iyz="0" izz="${(1/12)*${arg bar_mass}*(3*${arg bar_r}*${arg bar_r}+${arg bar_l}*${arg bar_l})}"/>
     </inertial>
     <visual>
-      <origin xyz="0 0 -${$(arg bar_l)/2}"/>
+      <origin xyz="0 ${$(arg bar_l)/2} 0" rpy="1.5707963267948966 0 0"/>
       <geometry>
-        <cylinder radius="0.0005" length="$(arg bar_l)"/>
+        <cylinder radius="${arg bar_r}" length="$(arg bar_l)"/>
       </geometry>
     </visual>
     <collision>
-      <origin xyz="0 0 -${$(arg bar_l)/2}"/>
+      <origin xyz="0 ${$(arg bar_l)/2} 0" rpy="1.5707963267948966 0 0"/>
       <geometry>
-        <cylinder radius="0.0005" length="$(arg bar_l)"/>
+        <cylinder radius="${arg bar_r}" length="$(arg bar_l)"/>
       </geometry>
     </collision>
   </link>
-  <joint name="foo_to_bar_joint" type="continuous">
+  <joint name="base_union_to_bar_joint" type="continuous">
     <origin xyz="0 0 0"/>
     <axis xyz="1 0 0"/>
-    <parent link="foo"/>
+    <parent link="base_union"/>
     <child link="bar"/>
   </joint>
@@ -60,6 +63,7 @@
     <inertial>
       <origin xyz="0 0 0"/>
-      <mass value="0.005"/>
-      <inertia ixx="1e-06" ixy="0" ixz="0" iyy="1e-06" iyz="0" izz="9e-06"/>
+      <mass value="${arg ball_mass}"/>
+      <inertia ixx="${(2/5)*${arg ball_mass}*${arg ball_r}*${arg ball_r}}" ixy="0" ixz="0"
+               iyy="${(2/5)*${arg ball_mass}*${arg ball_r}*${arg ball_r}}" iyz="0" izz="${(2/5)*${arg ball_mass}*${arg ball_r}*${arg ball_r}}"/>
     </inertial>
     <visual>
@@ -77,5 +81,5 @@
   </link>
   <joint name="ball_joint" type="fixed">
-    <origin xyz="0 0 -${$(arg bar_l) + $(arg ball_r)}"/>
+    <origin xyz="0 ${$(arg bar_l) + $(arg ball_r)} 0"/>
     <parent link="bar"/>
     <child link="ball"/>

Commit message: Reducing balloon bar radius

File: mbzirc_gazebo_simulation/challenge_worlds/urdf/balloon.xacro (robot description, xacro)
@@ -13,4 +13,5 @@
     <xacro:property name="balloon_model_scale_factor"  value="0.0025"/>
     <xacro:property name="bar_length"                  value="$(arg height)"/>
+    <xacro:property name="bar_rad"                     value="0.001"/>
     <xacro:property name="sphere_rad"                  value="0.02"/>
     <xacro:property name="base_height"                 value="0.1"/>
@@ -226,5 +227,5 @@
           <geometry>
             <cylinder>
-              <radius>0.006</radius>
+              <radius>${bar_rad}</radius>
               <length>${bar_length}</length>
             </cylinder>
@@ -249,5 +250,5 @@
           <geometry>
             <cylinder>
-              <radius>0.006</radius>
+              <radius>${bar_rad}</radius>
               <length>${bar_length}</length>
             </cylinder>
