Commit message: adding bricks with white fm plates

File: mbzirc_gazebo_simulation/challenge_worlds/urdf/single_blue_brick.xacro (robot description, xacro)
@@ -7,5 +7,5 @@
             <inertial>
 		    <mass>${mass}</mass>
-            <pose frame=''>0.1 0.6 0.1 0 -0 0</pose>
+            <!-- <pose frame=''>0.1 0.6 0.1 0 -0 0</pose> -->
                 <inertia>
 			<ixx>${(1.0/12.0)*mass*(pow(sy,2)+pow(sz,2))}</ixx> <ixy>0</ixy>
@@ -22,16 +22,36 @@
 		</material>
                 <geometry>
-                    <mesh>
+                    <!-- <mesh>
                         <uri>model://single_blue_brick/meshes/Brick_RibShape_Blue_redux.stl</uri>
                         <scale>0.01 0.01 0.01</scale>
-                    </mesh>
+                    </mesh> -->
+                    <box>
+                      <size>0.2 1.2 0.2</size>
+                    </box>
                 </geometry>
+            </visual>
+            <visual name="visual FM plate">
+            <pose>0 0 0.1 0 -0 0</pose>
+		      <material>
+			    <script>
+				  <uri>gazebo.material</uri>
+				  <name>Gazebo/White</name>
+			    </script>
+		      </material>
+              <geometry>
+                <box>
+                  <size>0.150 0.300 0.001</size>
+                </box>
+              </geometry>
             </visual>
             <collision name="collision">
                 <geometry>
-                    <mesh>
+                    <!-- <mesh>
                         <uri>model://single_blue_brick/meshes/Brick_RibShape_Blue_redux.stl</uri>
                         <scale>0.01 0.01 0.01</scale>
-                   </mesh>
+                   </mesh> -->
+                   <box>
+                      <size>0.2 1.2 0.2</size>
+                    </box>
                 </geometry>
             </collision>

File: mbzirc_gazebo_simulation/challenge_worlds/urdf/single_green_brick.xacro (robot description, xacro)
@@ -7,5 +7,5 @@
             <inertial>
 		    <mass>${mass}</mass>
-            <pose frame=''>0.1 0.3 0.1 0 -0 0</pose>
+            <!-- <pose frame=''>0.1 0.3 0.1 0 -0 0</pose> -->
                 <inertia>
 			<ixx>${(1.0/12.0)*mass*(pow(sy,2)+pow(sz,2))}</ixx> <ixy>0</ixy>
@@ -22,16 +22,36 @@
 		</material>
                 <geometry>
-                    <mesh>
+                    <!-- <mesh>
                         <uri>model://single_green_brick/meshes/Brick_RibShape_Green_redux.stl</uri>
                         <scale>0.01 0.01 0.01</scale>
-                    </mesh>
+                    </mesh> -->
+                    <box>
+                      <size>0.2 0.6 0.2</size>
+                    </box>
                 </geometry>
+            </visual>
+            <visual name="visual FM plate">
+            <pose>0 0 0.1 0 -0 0</pose>
+		      <material>
+			    <script>
+				  <uri>gazebo.material</uri>
+				  <name>Gazebo/White</name>
+			    </script>
+		      </material>
+              <geometry>
+                <box>
+                  <size>0.150 0.300 0.001</size>
+                </box>
+              </geometry>
             </visual>
             <collision name="collision">
                 <geometry>
-                    <mesh>
+                    <!-- <mesh>
                         <uri>model://single_green_brick/meshes/Brick_RibShape_Green_redux.stl</uri>
                         <scale>0.01 0.01 0.01</scale>
-                   </mesh>
+                    </mesh> -->
+                    <box>
+                      <size>0.2 0.6 0.2</size>
+                    </box>
                 </geometry>
             </collision>

File: mbzirc_gazebo_simulation/challenge_worlds/urdf/single_orange_brick.xacro (robot description, xacro)
@@ -7,5 +7,5 @@
             <inertial>
 		      <mass>${mass}</mass>
-              <pose frame=''>0.1 0.9 0.1 0 -0 0</pose>
+              <!-- <pose frame=''>0.1 0.9 0.1 0 -0 0</pose> -->
               <inertia>
 			    <ixx>${(1.0/12.0)*mass*(pow(sy,2)+pow(sz,2))}</ixx> <ixy>0</ixy>
@@ -22,16 +22,68 @@
 		      </material>
               <geometry>
-                <mesh>
+                <!-- <mesh>
                   <uri>model://single_orange_brick/meshes/Brick_RibShape_Orange_redux.stl</uri>
                   <scale>0.01 0.01 0.01</scale>
-                </mesh>
+                </mesh> -->
+                <box>
+                      <size>0.2 1.8 0.2</size>
+                </box>
+              </geometry>
+            </visual>
+            <visual name="visual FM plate 1">
+            <pose>0 -0.805 0.1 0 -0 0</pose>
+              <material>
+			    <script>
+				  <uri>gazebo.material</uri>
+				  <name>Gazebo/White</name>
+			    </script>
+		      </material>
+              <geometry>
+                <!-- <mesh>
+                  <uri>model://single_orange_brick/meshes/Brick_RibShape_Orange_redux.stl</uri>
+                  <scale>0.01 0.01 0.01</scale>
+                </mesh> -->
+                <box>
+                      <size>0.150 0.190 0.001</size>
+                </box>
+              </geometry>
+            </visual>
+            <visual name="visual FM plate 2">
+            <pose>0 0 0.1 0 -0 0</pose>
+              <material>
+			    <script>
+				  <uri>gazebo.material</uri>
+				  <name>Gazebo/White</name>
+			    </script>
+		      </material>
+              <geometry>
+                <box>
+                      <size>0.150 0.190 0.001</size>
+                </box>
+              </geometry>
+            </visual>
+            <visual name="visual FM plate 3">
+            <pose>0 0.805 0.1 0 -0 0</pose>
+              <material>
+			    <script>
+				  <uri>gazebo.material</uri>
+				  <name>Gazebo/White</name>
+			    </script>
+		      </material>
+              <geometry>
+                <box>
+                      <size>0.150 0.190 0.001</size>
+                </box>
               </geometry>
             </visual>
             <collision name="collision">
               <geometry>
-                <mesh>
+                <!-- <mesh>
                   <uri>model://single_orange_brick/meshes/Brick_RibShape_Orange_redux.stl</uri>
                   <scale>0.01 0.01 0.01</scale>
-                </mesh>
+                </mesh> -->
+                <box>
+                      <size>0.2 1.8 0.2</size>
+                </box>
               </geometry>
             </collision>

File: mbzirc_gazebo_simulation/challenge_worlds/urdf/single_red_brick.xacro (robot description, xacro)
@@ -7,5 +7,5 @@
             <inertial>
 		      <mass>${mass}</mass>
-              <pose frame=''>0.1 0.15 0.1 0 -0 0</pose>
+              <!-- <pose frame=''>0.1 0.15 0.1 0 -0 0</pose> -->
               <inertia>
 			    <ixx>${(1.0/12.0)*mass*(pow(sy,2)+pow(sz,2))}</ixx> <ixy>0</ixy>
@@ -22,16 +22,36 @@
 		      </material>
               <geometry>
-                <mesh>
+                <!-- <mesh>
                   <uri>model://single_red_brick/meshes/Brick_RibShape_Red_redux.stl</uri>
                   <scale>0.01 0.01 0.01</scale>
-                </mesh>
+                </mesh> -->
+                <box>
+                  <size>0.2 0.3 0.2</size>
+                </box>
+              </geometry>
+            </visual>
+            <visual name="visual FM plate">
+            <pose>0 0 0.1 0 -0 0</pose>
+		      <material>
+			    <script>
+				  <uri>gazebo.material</uri>
+				  <name>Gazebo/White</name>
+			    </script>
+		      </material>
+              <geometry>
+                <box>
+                  <size>0.150 0.200 0.001</size>
+                </box>
               </geometry>
             </visual>
             <collision name="collision">
               <geometry>
-                <mesh>
+                <!-- <mesh>
                   <uri>model://single_red_brick/meshes/Brick_RibShape_Red_redux.stl</uri>
                   <scale>0.01 0.01 0.01</scale>
-                </mesh>
+                </mesh> -->
+                <box>
+                  <size>0.200 0.300 0.2</size>
+                </box>
               </geometry>
             </collision>

File: mbzirc_gazebo_simulation/challenge_worlds/worlds/challenge2.world.xacro (robot description, xacro)
@@ -28,5 +28,5 @@
 <xacro:property name="orange03" value="${[39,26,0,0]}"/>
 <xacro:property name="orange04" value="${[39,24,0,0]}"/>
-<xacro:property name="L_frame" value="${[0.5,0.5,0.005,0.3]}"/>
+<xacro:property name="L_frame" value="${[30,25,0.005,0.0]}"/>
   <world name="default">
     <!-- GRIPPER PLUGIN TO AVOID THE NEED OF COLLISIONS -->
@@ -43,16 +43,16 @@
     <single_red_brick id="Red_brick_03" pose="${red03[0]*cos(yaw)-red03[1]*sin(yaw)} ${red03[0]*sin(yaw)+red03[1]*cos(yaw)} ${red03[2]} 0 0 ${red03[3]+yaw}" sx="0.2" sy="0.3" sz="0.2" mass="1.0" mat="Gazebo/Red" />
     <single_red_brick id="Red_brick_04" pose="${red04[0]*cos(yaw)-red04[1]*sin(yaw)} ${red04[0]*sin(yaw)+red04[1]*cos(yaw)} ${red04[2]} 0 0 ${red04[3]+yaw}" sx="0.2" sy="0.3" sz="0.2" mass="1.0" mat="Gazebo/Red" />
-    <single_blue_brick id="Blue_brick_01" pose="${blue01[0]*cos(yaw)-blue01[1]*sin(yaw)} ${blue01[0]*sin(yaw)+blue01[1]*cos(yaw)} ${blue01[2]} 0 0 ${blue01[3]+yaw}" sx="0.2" sy="1.2" sz="0.2" mass="1.0" mat="Gazebo/Blue" />
-    <single_blue_brick id="Blue_brick_02" pose="${blue02[0]*cos(yaw)-blue02[1]*sin(yaw)} ${blue02[0]*sin(yaw)+blue02[1]*cos(yaw)} ${blue02[2]} 0 0 ${blue02[3]+yaw}" sx="0.2" sy="1.2" sz="0.2" mass="1.0" mat="Gazebo/Blue" />
-    <single_blue_brick id="Blue_brick_03" pose="${blue03[0]*cos(yaw)-blue03[1]*sin(yaw)} ${blue03[0]*sin(yaw)+blue03[1]*cos(yaw)} ${blue03[2]} 0 0 ${blue03[3]+yaw}" sx="0.2" sy="1.2" sz="0.2" mass="1.0" mat="Gazebo/Blue" />
-    <single_blue_brick id="Blue_brick_04" pose="${blue04[0]*cos(yaw)-blue04[1]*sin(yaw)} ${blue04[0]*sin(yaw)+blue04[1]*cos(yaw)} ${blue04[2]} 0 0 ${blue04[3]+yaw}" sx="0.2" sy="1.2" sz="0.2" mass="1.0" mat="Gazebo/Blue" />
+    <single_blue_brick id="Blue_brick_01" pose="${blue01[0]*cos(yaw)-blue01[1]*sin(yaw)} ${blue01[0]*sin(yaw)+blue01[1]*cos(yaw)} ${blue01[2]} 0 0 ${blue01[3]+yaw}" sx="0.2" sy="1.2" sz="0.2" mass="1.5" mat="Gazebo/Blue" />
+    <single_blue_brick id="Blue_brick_02" pose="${blue02[0]*cos(yaw)-blue02[1]*sin(yaw)} ${blue02[0]*sin(yaw)+blue02[1]*cos(yaw)} ${blue02[2]} 0 0 ${blue02[3]+yaw}" sx="0.2" sy="1.2" sz="0.2" mass="1.5" mat="Gazebo/Blue" />
+    <single_blue_brick id="Blue_brick_03" pose="${blue03[0]*cos(yaw)-blue03[1]*sin(yaw)} ${blue03[0]*sin(yaw)+blue03[1]*cos(yaw)} ${blue03[2]} 0 0 ${blue03[3]+yaw}" sx="0.2" sy="1.2" sz="0.2" mass="1.5" mat="Gazebo/Blue" />
+    <single_blue_brick id="Blue_brick_04" pose="${blue04[0]*cos(yaw)-blue04[1]*sin(yaw)} ${blue04[0]*sin(yaw)+blue04[1]*cos(yaw)} ${blue04[2]} 0 0 ${blue04[3]+yaw}" sx="0.2" sy="1.2" sz="0.2" mass="1.5" mat="Gazebo/Blue" />
     <single_green_brick id="Green_brick_01" pose="${green01[0]*cos(yaw)-green01[1]*sin(yaw)} ${green01[0]*sin(yaw)+green01[1]*cos(yaw)} ${green01[2]} 0 0 ${green01[3]+yaw}" sx="0.2" sy="0.6" sz="0.2" mass="1.0" mat="Gazebo/Green" />
     <single_green_brick id="Green_brick_02" pose="${green02[0]*cos(yaw)-green02[1]*sin(yaw)} ${green02[0]*sin(yaw)+green02[1]*cos(yaw)} ${green02[2]} 0 0 ${green02[3]+yaw}" sx="0.2" sy="0.6" sz="0.2" mass="1.0" mat="Gazebo/Green" />
     <single_green_brick id="Green_brick_03" pose="${green03[0]*cos(yaw)-green03[1]*sin(yaw)} ${green03[0]*sin(yaw)+green03[1]*cos(yaw)} ${green03[2]} 0 0 ${green03[3]+yaw}" sx="0.2" sy="0.6" sz="0.2" mass="1.0" mat="Gazebo/Green" />
     <single_green_brick id="Green_brick_04" pose="${green04[0]*cos(yaw)-green04[1]*sin(yaw)} ${green04[0]*sin(yaw)+green04[1]*cos(yaw)} ${green04[2]} 0 0 ${green04[3]+yaw}" sx="0.2" sy="0.6" sz="0.2" mass="1.0" mat="Gazebo/Green" />
-    <single_orange_brick id="Orange_brick_01" pose="${orange01[0]*cos(yaw)-orange01[1]*sin(yaw)} ${orange01[0]*sin(yaw)+orange01[1]*cos(yaw)} ${orange01[2]} 0 0 ${orange01[3]+yaw}" sx="0.2" sy="1.8" sz="0.2" mass="1.0" mat="Gazebo/Orange" />
-    <single_orange_brick id="Orange_brick_02" pose="${orange02[0]*cos(yaw)-orange02[1]*sin(yaw)} ${orange02[0]*sin(yaw)+orange02[1]*cos(yaw)} ${orange02[2]} 0 0 ${orange02[3]+yaw}" sx="0.2" sy="1.8" sz="0.2" mass="1.0" mat="Gazebo/Orange" />
-    <single_orange_brick id="Orange_brick_03" pose="${orange03[0]*cos(yaw)-orange03[1]*sin(yaw)} ${orange03[0]*sin(yaw)+orange03[1]*cos(yaw)} ${orange03[2]} 0 0 ${orange03[3]+yaw}" sx="0.2" sy="1.8" sz="0.2" mass="1.0" mat="Gazebo/Orange" />
-    <single_orange_brick id="Orange_brick_04" pose="${orange04[0]*cos(yaw)-orange04[1]*sin(yaw)} ${orange04[0]*sin(yaw)+orange04[1]*cos(yaw)} ${orange04[2]} 0 0 ${orange04[3]+yaw}" sx="0.2" sy="1.8" sz="0.2" mass="1.0" mat="Gazebo/Orange" />
+    <single_orange_brick id="Orange_brick_01" pose="${orange01[0]*cos(yaw)-orange01[1]*sin(yaw)} ${orange01[0]*sin(yaw)+orange01[1]*cos(yaw)} ${orange01[2]} 0 0 ${orange01[3]+yaw}" sx="0.2" sy="1.8" sz="0.2" mass="2.0" mat="Gazebo/Orange" />
+    <single_orange_brick id="Orange_brick_02" pose="${orange02[0]*cos(yaw)-orange02[1]*sin(yaw)} ${orange02[0]*sin(yaw)+orange02[1]*cos(yaw)} ${orange02[2]} 0 0 ${orange02[3]+yaw}" sx="0.2" sy="1.8" sz="0.2" mass="2.0" mat="Gazebo/Orange" />
+    <single_orange_brick id="Orange_brick_03" pose="${orange03[0]*cos(yaw)-orange03[1]*sin(yaw)} ${orange03[0]*sin(yaw)+orange03[1]*cos(yaw)} ${orange03[2]} 0 0 ${orange03[3]+yaw}" sx="0.2" sy="1.8" sz="0.2" mass="2.0" mat="Gazebo/Orange" />
+    <single_orange_brick id="Orange_brick_04" pose="${orange04[0]*cos(yaw)-orange04[1]*sin(yaw)} ${orange04[0]*sin(yaw)+orange04[1]*cos(yaw)} ${orange04[2]} 0 0 ${orange04[3]+yaw}" sx="0.2" sy="1.8" sz="0.2" mass="2.0" mat="Gazebo/Orange" />
     <model name="L_wooden_frame">
       <include>
