Commit message: pregrasp planner added

File: atrvjr_ur5/atrvjr/description/atrvjr_description/urdf/atrvjr.xacro (robot description, xacro)
@@ -12,5 +12,5 @@
     <xacro:property name="chassis_width" value="0.385" />
     <!-- This is not including equipment and racks on the top -->
-    <xacro:property name="chassis_height" value="0.52" />
+    <xacro:property name="chassis_height" value="0.45" />
         <!-- wheel properties -->
     <xacro:property name="wheel_radius" value="0.155" />
@@ -37,9 +37,21 @@
     <!-- is needed for the navigation stack to work properly -->
     <link name="base_link">
-       <!--  <inertial>
-            <origin xyz="0 0.3 0.2" rpy="1.57 0 0"/>
-            <mass value="100"/>
-            <inertia ixx="1.00" ixy="0.0" ixz="0.0" iyy="1.01" iyz="0.0" izz="1.01"/>
-        </inertial> -->
+        <!-- <visual>
+            <origin xyz="0.0 0.0 0.3" rpy="0 0 0" />
+            <geometry>
+                <box size="${chassis_length} ${chassis_width} ${chassis_height}" />
+            </geometry>
+        </visual> -->
+        <collision>
+            <origin xyz="0.0 0.0 0.3" rpy="0 0 0" />
+            <geometry>
+                <box size="${chassis_length} ${chassis_width} ${chassis_height-0.05}" />
+            </geometry>
+        </collision>
+        <inertial>
+            <origin xyz="0.0 0.0 0.2" rpy="0 0 0"/>
+            <mass value="60"/>
+            <inertia ixx="2.01" ixy="0.0" ixz="0.0" iyy="2.51" iyz="0.0" izz="2.01"/>
+        </inertial>
     </link>
     <!-- center_link -->
@@ -53,15 +65,4 @@
             </geometry>
         </visual>
-        <collision>
-            <origin xyz="0.1 0.25 0.19" rpy="0 0 0" />
-            <geometry>
-                <box size="${chassis_length} ${chassis_width+0.07} ${chassis_height-0.13}" />
-            </geometry>
-        </collision>
-        <inertial>
-            <origin xyz="0.1 0.25 0.2" rpy="1.57 0 0"/>
-            <mass value="1000"/>
-            <inertia ixx="2.01" ixy="0.0" ixz="0.0" iyy="2.01" iyz="0.0" izz="2.01"/>
-        </inertial>
     </link>
     <!-- base_link -> center_link -->
@@ -82,5 +83,5 @@
     <joint name="base_cbimu_joint" type="fixed">
         <origin xyz="0 0 0.267" rpy="0 ${M_PI} 0"/>
-        <parent link="center_link"/>
+        <parent link="base_link"/>
         <child link="cbimu_frame"/>
     </joint>
@@ -89,5 +90,5 @@
     <joint name="base_mpuimu_joint" type="fixed">
         <origin xyz="0 0 0.35" rpy="0 0 ${M_PI/2.0}"/>
-        <parent link="center_link"/>
+        <parent link="base_link"/>
         <child link="mpuimu_frame"/>
     </joint>
@@ -96,5 +97,5 @@
     <joint name="lrf_joint" type="fixed">
         <origin xyz="0.2 0 0.35" rpy="0 0 0"/>
-        <parent link="center_link"/>
+        <parent link="base_link"/>
         <child link="lrf_frame"/>
     </joint>
@@ -103,5 +104,5 @@
     <joint name="novatel_joint" type="fixed">
         <origin xyz="-0.15 0.1 0.4" rpy="0 0 0"/>
-        <parent link="center_link"/>
+        <parent link="base_link"/>
         <child link="novatel"/>
     </joint>

File: atrvjr_ur5/atrvjr/description/atrvjr_description/urdf/atrvjr_wheels.xacro (robot description, xacro)
@@ -37,5 +37,5 @@
       <inertial>
         <origin xyz="0 0 0" rpy="0 0 0"/>
-        <mass value="20"/>
+        <mass value="5"/>
         <inertia ixx="0.021" ixy="0.0" ixz="0.0" iyy="0.04" iyz="0.0" izz="0.021"/>
       </inertial>

Commit message: improve navigation

File: atrvjr_ur5/atrvjr/description/atrvjr_description/urdf/atrvjr.xacro (robot description, xacro)
@@ -51,5 +51,5 @@
         <inertial>
             <origin xyz="0.0 0.0 0.2" rpy="0 0 0"/>
-            <mass value="60"/>
+            <mass value="500"/>
             <inertia ixx="2.01" ixy="0.0" ixz="0.0" iyy="2.51" iyz="0.0" izz="2.01"/>
         </inertial>
@@ -93,12 +93,4 @@
         <child link="mpuimu_frame"/>
     </joint>
-    <!-- Hokuyo Link -->
-    <link name="lrf_frame"/>
-    <joint name="lrf_joint" type="fixed">
-        <origin xyz="0.2 0 0.35" rpy="0 0 0"/>
-        <parent link="base_link"/>
-        <child link="lrf_frame"/>
-    </joint>
-    <!-- Hokuyo Link -->
     <link name="novatel"/>
     <joint name="novatel_joint" type="fixed">
@@ -107,4 +99,21 @@
         <child link="novatel"/>
     </joint>
+    <link name="hokuyo"/>
+<!--         <visual>
+            <geometry>
+                <box size="0.02 0.035 0.002"/>
+            </geometry>
+        </visual>
+        <inertial>
+            <mass value="0.001"/>
+            <origin xyz="0 0 0"/>
+            <inertia ixx="0.0001" ixy="0.0" ixz="0.0" iyy="0.0001" iyz="0.0" izz="0.0001"/>
+        </inertial>
+    </link> -->
+    <joint name="laser_joint" type="fixed">
+        <origin xyz="0.35 0 0.25" rpy="0 0 0"/>
+        <parent link="base_link" />
+        <child link="hokuyo" />
+    </joint>
     </xacro:macro>
 </robot>

File: atrvjr_ur5/universal_robot/ur_description/urdf/common.gazebo.xacro (robot description, xacro)
@@ -22,3 +22,58 @@
 -->
   </gazebo>
+  <gazebo reference="hokuyo">
+    <sensor type="ray" name="hokuyo_sensor">
+      <pose>0 0 0 0 0 0</pose>
+      <visualize>true</visualize>
+      <update_rate>34.5</update_rate>
+      <ray>
+        <scan>
+          <horizontal>
+            <samples>720</samples>
+            <resolution>1</resolution>
+            <min_angle>-1.570796</min_angle>
+            <max_angle>1.570796</max_angle>
+          </horizontal>
+        </scan>
+        <range>
+          <min>0.05</min>
+          <max>20.0</max>
+          <resolution>0.01</resolution>
+        </range>
+        <noise>
+          <type>gaussian</type>
+          <!-- Noise parameters based on published spec for Hokuyo laser
+               achieving "+-30mm" accuracy at range < 10m.  A mean of 0.0m and
+               stddev of 0.01m will put 99.7% of samples within 0.03m of the true
+               reading. -->
+          <mean>0.0</mean>
+          <stddev>0.01</stddev>
+        </noise>
+      </ray>
+      <plugin name="gazebo_ros_hokuyo_controller" filename="libgazebo_ros_laser.so">
+        <topicName>/laser_scan</topicName>
+        <frameName>hokuyo</frameName>
+      </plugin>
+    </sensor>
+  </gazebo>
+  <gazebo reference="front_left_wheel_link">
+    <material>Gazebo/DarkGrey</material>
+    <mu1>0.5</mu1>
+    <mu2>0.5</mu2>
+  </gazebo>
+  <gazebo reference="front_right_wheel_link">
+    <material>Gazebo/DarkGrey</material>
+    <mu1>0.5</mu1>
+    <mu2>0.5</mu2>
+  </gazebo>
+  <gazebo reference="rear_left_wheel_link">
+    <material>Gazebo/DarkGrey</material>
+    <mu1>0.5</mu1>
+    <mu2>0.5</mu2>
+  </gazebo>
+  <gazebo reference="rear_right_wheel_link">
+    <material>Gazebo/DarkGrey</material>
+    <mu1>0.5</mu1>
+    <mu2>0.5</mu2>
+  </gazebo>
 </robot>

File: atrvjr_ur5/universal_robot/ur_description/urdf/ur5.urdf.xacro (robot description, xacro)
@@ -21,9 +21,9 @@
     <!-- Inertia parameters -->
     <xacro:property name="base_mass" value="1.0" />  <!-- This mass might be incorrect -->
-    <xacro:property name="shoulder_mass" value="3.7000" />
-    <xacro:property name="upper_arm_mass" value="8.3930" />
-    <xacro:property name="forearm_mass" value="2.2750" />
-    <xacro:property name="wrist_1_mass" value="1.2190" />
-    <xacro:property name="wrist_2_mass" value="1.2190" />
+    <xacro:property name="shoulder_mass" value="0.7000" />
+    <xacro:property name="upper_arm_mass" value="0.3930" />
+    <xacro:property name="forearm_mass" value="0.2750" />
+    <xacro:property name="wrist_1_mass" value="0.2190" />
+    <xacro:property name="wrist_2_mass" value="0.2190" />
     <xacro:property name="wrist_3_mass" value="0.1879" />
     <xacro:property name="shoulder_cog" value="0.0 0.00193 -0.02561" />

Commit message: moveit planning with base + some stuff for the camera - dope

File: atrvjr_ur5/atrvjr/description/atrvjr_description/urdf/atrvjr.xacro (robot description, xacro)
@@ -32,4 +32,55 @@
         <origin xyz="0 0 0" rpy="0 0 0" />
     </xacro:wheel>
+    <link name="teste_link">
+        <!-- <visual>
+            <origin xyz="0.0 0.0 0.0" rpy="0 0 0" />
+            <geometry>
+                <box size="0.001 0.001 0.001" />
+            </geometry>
+        </visual> -->
+        <collision>
+            <origin xyz="0.0 0.0 0.3" rpy="0 0 0" />
+            <geometry>
+                <box size="${chassis_length} ${chassis_width} ${chassis_height-0.05}" />
+            </geometry>
+        </collision>
+        <inertial>
+            <origin xyz="0.0 0.0 0.0" rpy="0 0 0"/>
+            <mass value="0.001"/>
+            <inertia ixx="0.001" ixy="0.0" ixz="0.0" iyy="0.001" iyz="0.0" izz="0.001"/>
+        </inertial>
+    </link>
+    <joint name="teste_joint" type="prismatic">
+        <origin xyz="0 0 0" rpy="0 0 0"/>
+        <parent link="base_link"/>
+        <child link="teste_link"/>
+        <axis xyz="1 0 0"/>
+        <limit effort="80.0" lower="-1" upper="1" velocity="0.5"/>
+    </joint>
+    <link name="teste2_link">
+        <!-- <visual>
+            <origin xyz="0.0 0.0 0.0" rpy="0 0 0" />
+            <geometry>
+                <box size="0.001 0.001 0.001" />
+            </geometry>
+        </visual> -->
+        <collision>
+            <origin xyz="0.0 0.0 0.3" rpy="0 0 0" />
+            <geometry>
+                <box size="${chassis_length} ${chassis_width} ${chassis_height}" />
+            </geometry>
+        </collision>
+        <inertial>
+            <origin xyz="0.0 0.0 0.0" rpy="0 0 0"/>
+            <mass value="0.001"/>
+            <inertia ixx="0.001" ixy="0.0" ixz="0.0" iyy="0.001" iyz="0.0" izz="0.001"/>
+        </inertial>
+    </link>
+    <joint name="teste2_joint" type="continuous">
+        <origin xyz="0 0 0" rpy="0 0 0"/>
+        <parent link="teste_link"/>
+        <child link="teste2_link"/>
+        <axis xyz="0 0 1"/>
+    </joint>
     <!-- links -->
     <!-- base_link -->
@@ -43,13 +94,13 @@
             </geometry>
         </visual> -->
-        <collision>
+        <!-- <collision>
             <origin xyz="0.0 0.0 0.3" rpy="0 0 0" />
             <geometry>
                 <box size="${chassis_length} ${chassis_width} ${chassis_height-0.05}" />
             </geometry>
-        </collision>
+        </collision> -->
         <inertial>
             <origin xyz="0.0 0.0 0.2" rpy="0 0 0"/>
-            <mass value="500"/>
+            <mass value="50"/>
             <inertia ixx="2.01" ixy="0.0" ixz="0.0" iyy="2.51" iyz="0.0" izz="2.01"/>
         </inertial>
@@ -69,5 +120,5 @@
     <joint name="base_link_joint" type="fixed">
         <origin xyz="-0.1 0.19 ${center_height-0.1}" rpy="1.57 0 0"/>
-        <parent link="base_link"/>
+        <parent link="teste2_link"/>
         <child link="center_link"/>
     </joint>
@@ -76,5 +127,5 @@
     <joint name="$to_{armConnectionFrame}_joint" type="fixed">
         <origin xyz="0.12 0 0.56" rpy="0 0 0"/>
-        <parent link="base_link"/>
+        <parent link="teste2_link"/>
         <child link="${armConnectionFrame}"/>
     </joint>
@@ -83,5 +134,5 @@
     <joint name="base_cbimu_joint" type="fixed">
         <origin xyz="0 0 0.267" rpy="0 ${M_PI} 0"/>
-        <parent link="base_link"/>
+        <parent link="teste_link"/>
         <child link="cbimu_frame"/>
     </joint>
@@ -90,5 +141,5 @@
     <joint name="base_mpuimu_joint" type="fixed">
         <origin xyz="0 0 0.35" rpy="0 0 ${M_PI/2.0}"/>
-        <parent link="base_link"/>
+        <parent link="teste_link"/>
         <child link="mpuimu_frame"/>
     </joint>
@@ -96,5 +147,5 @@
     <joint name="novatel_joint" type="fixed">
         <origin xyz="-0.15 0.1 0.4" rpy="0 0 0"/>
-        <parent link="base_link"/>
+        <parent link="teste_link"/>
         <child link="novatel"/>
     </joint>
@@ -112,8 +163,26 @@
     </link> -->
     <joint name="laser_joint" type="fixed">
-        <origin xyz="0.35 0 0.25" rpy="0 0 0"/>
-        <parent link="base_link" />
+        <origin xyz="0.35 0 0.1" rpy="0 0 0"/>
+        <parent link="teste_link" />
         <child link="hokuyo" />
     </joint>
+    <transmission name="teste_prismatic_trans">
+      <type>transmission_interface/SimpleTransmission</type>
+      <joint name="teste_joint">
+        <hardwareInterface>hardware_interface/VelocityJointInterface</hardwareInterface>
+      </joint>
+      <actuator name="teste_prismatic_actuator">
+        <mechanicalReduction>1</mechanicalReduction>
+      </actuator>
+    </transmission>
+    <transmission name="teste2_prismatic_trans">
+      <type>transmission_interface/SimpleTransmission</type>
+      <joint name="teste2_joint">
+        <hardwareInterface>hardware_interface/VelocityJointInterface</hardwareInterface>
+      </joint>
+      <actuator name="teste2_prismatic_actuator">
+        <mechanicalReduction>1</mechanicalReduction>
+      </actuator>
+    </transmission>
     </xacro:macro>
 </robot>

File: atrvjr_ur5/universal_robot/ur_description/urdf/common.gazebo.xacro (robot description, xacro)
@@ -77,3 +77,10 @@
     <mu2>0.5</mu2>
   </gazebo>
+<!--   <gazebo>
+    <plugin name="ros_gripper" filename="libmagnetic_gripper_plugin.so">
+      <agent_name>test_gripper</agent_name>
+      <gripper_link_name>gripper_link</gripper_link_name>
+    </plugin>
+  </gazebo>
+ -->
 </robot>

File: atrvjr_ur5/universal_robot/ur_description/urdf/ur.transmission.xacro (robot description, xacro)
@@ -5,5 +5,5 @@
       <type>transmission_interface/SimpleTransmission</type>
       <joint name="${prefix}shoulder_pan_joint">
-        <hardwareInterface>hardware_interface/PositionJointInterface</hardwareInterface>
+        <hardwareInterface>hardware_interface/VelocityJointInterface</hardwareInterface>
       </joint>
       <actuator name="${prefix}shoulder_pan_motor">
@@ -14,5 +14,5 @@
       <type>transmission_interface/SimpleTransmission</type>
       <joint name="${prefix}shoulder_lift_joint">
-        <hardwareInterface>hardware_interface/PositionJointInterface</hardwareInterface>
+        <hardwareInterface>hardware_interface/VelocityJointInterface</hardwareInterface>
       </joint>
       <actuator name="${prefix}shoulder_lift_motor">
@@ -23,5 +23,5 @@
       <type>transmission_interface/SimpleTransmission</type>
       <joint name="${prefix}elbow_joint">
-        <hardwareInterface>hardware_interface/PositionJointInterface</hardwareInterface>
+        <hardwareInterface>hardware_interface/VelocityJointInterface</hardwareInterface>
       </joint>
       <actuator name="${prefix}elbow_motor">
@@ -32,5 +32,5 @@
       <type>transmission_interface/SimpleTransmission</type>
       <joint name="${prefix}wrist_1_joint">
-        <hardwareInterface>hardware_interface/PositionJointInterface</hardwareInterface>
+        <hardwareInterface>hardware_interface/VelocityJointInterface</hardwareInterface>
       </joint>
       <actuator name="${prefix}wrist_1_motor">
@@ -41,5 +41,5 @@
       <type>transmission_interface/SimpleTransmission</type>
       <joint name="${prefix}wrist_2_joint">
-        <hardwareInterface>hardware_interface/PositionJointInterface</hardwareInterface>
+        <hardwareInterface>hardware_interface/VelocityJointInterface</hardwareInterface>
       </joint>
       <actuator name="${prefix}wrist_2_motor">
@@ -50,5 +50,5 @@
       <type>transmission_interface/SimpleTransmission</type>
       <joint name="${prefix}wrist_3_joint">
-        <hardwareInterface>hardware_interface/PositionJointInterface</hardwareInterface>
+        <hardwareInterface>hardware_interface/VelocityJointInterface</hardwareInterface>
       </joint>
       <actuator name="${prefix}wrist_3_motor">

Commit message: planning arm+base working, need tuning in navigation

File: atrvjr_ur5/atrvjr/description/atrvjr_description/urdf/atrvjr.xacro (robot description, xacro)
@@ -44,5 +44,5 @@
         <child link="teste_link"/>
         <axis xyz="1 0 0"/>
-        <limit effort="80.0" lower="-1" upper="1" velocity="0.5"/>
+        <limit effort="80.0" lower="-2" upper="2" velocity="0.5"/>
     </joint>
     <link name="teste2_link">
@@ -64,5 +64,5 @@
         <child link="teste2_link"/>
         <axis xyz="0 1 0"/>
-        <limit effort="80.0" lower="-1" upper="1" velocity="0.5"/>
+        <limit effort="80.0" lower="-2" upper="2" velocity="0.5"/>
     </joint>
     <!-- links -->
