Commit message: changed: modified atrv gazebo model; added: fake localization and navigation setup

File: mbzirc_gazebo_simulation/atrvjr_description/urdf/atrvjr.xacro (robot description, xacro)
@@ -115,5 +115,5 @@
           <child link="center_link"/>
       </joint>
-      <!-- Hokuyo Link
+      <!-- Hokuyo Link -->
       <link name="hokuyo_link">
         <collision>
@@ -136,12 +136,12 @@
       </link>
       <joint name="hokuyo_joint" type="fixed">
-          <origin xyz="${chassis_length/2+0.2} 0 -0.1" rpy="0 0 0"/>
+          <origin xyz="${chassis_length/2+0.1} 0 0" rpy="0 0 0"/>
           <parent link="center_link"/>
           <child link="hokuyo_link"/>
       </joint>
       <gazebo reference="hokuyo_link">
-        <sensor type="gpu_ray" name="head_hokuyo_sensor">
+        <sensor type="ray" name="head_hokuyo_sensor">
           <pose>0 0 0 0 0 0</pose>
-          <visualize>true</visualize>
+          <visualize>false</visualize>
           <update_rate>40</update_rate>
           <ray>
@@ -165,38 +165,27 @@
             </noise>
           </ray>
-          <plugin name="gazebo_ros_head_hokuyo_controller" filename="libgazebo_ros_gpu_laser.so">
+          <plugin name="gazebo_ros_head_hokuyo_controller" filename="libgazebo_ros_laser.so">
             <topicName>/scan</topicName>
             <frameName>hokuyo_link</frameName>
           </plugin>
         </sensor>
-      </gazebo>-->
-      <!-- Crossbow Imu Link
-      <link name="cbimu_frame"/>
-      <joint name="base_cbimu_joint" type="fixed">
-          <origin xyz="0 0 0.267" rpy="0 ${M_PI} 0"/>
-          <parent link="center_link"/>
-          <child link="cbimu_frame"/>
-      </joint> -->
-          <!-- MPU Imu Link
-      <link name="mpuimu_frame"/>
-      <joint name="base_mpuimu_joint" type="fixed">
-          <origin xyz="0 0 0.35" rpy="0 0 ${M_PI/2.0}"/>
-          <parent link="center_link"/>
-          <child link="mpuimu_frame"/>
-      </joint> -->
-      <!-- Novatel Link
-      <link name="novatel"/>
-      <joint name="novatel_joint" type="fixed">
-          <origin xyz="-0.15 0.1 0.4" rpy="0 0 0"/>
-          <parent link="center_link"/>
-          <child link="novatel"/>
-      </joint>-->
-      <!--<gazebo>
-        <plugin name="gazebo_ros_control" filename="libgazebo_ros_control.so">
+      </gazebo>
+      <gazebo>
+        <!-- <plugin name="gazebo_ros_control" filename="libgazebo_ros_control.so">
           <robotNamespace></robotNamespace>
           <robotSimType>gazebo_ros_control/DefaultRobotHWSim</robotSimType>
           <legacyModeNS>true</legacyModeNS>
+        </plugin> -->
+        <plugin name="p3d_base_controller" filename="libgazebo_ros_p3d.so">
+              <alwaysOn>true</alwaysOn>
+              <updateRate>30.0</updateRate>
+              <bodyName>base_link</bodyName>
+              <topicName>base_pose_ground_truth</topicName>
+              <gaussianNoise>0.01</gaussianNoise>
+              <frameName>map</frameName>
+              <xyzOffsets>0 0 0</xyzOffsets>
+              <rpyOffsets>0 0 0</rpyOffsets>
         </plugin>
-      </gazebo>-->
+      </gazebo>
     </xacro:macro>
 </robot>

File: mbzirc_gazebo_simulation/atrvjr_description/urdf/atrvjr_ur5.urdf.xacro (robot description, xacro)
@@ -15,3 +15,13 @@
         <origin xyz="-0.1 0 0.32" rpy="0.0 0.0 0.0" />
     </joint>
+    <!-- gripper
+    <include filename="$(find mbzirc_gazebo_plugins)/urdf/magnetic_gripper.xacro" />
+    <magnetic_gripper parent="ur5_ee_link" robot_name="">
+    		<origin xyz="0 0 0" rpy="1.57 0 0" />
+    </magnetic_gripper> -->
+    <!-- camera -->
+    <include filename="$(find mbzirc_gazebo_plugins)/urdf/fake_camera.xacro" />
+    <fake_camera parent="center_link" robot_name="">
+    		<origin xyz="0 0.5 0" rpy="0 0 1.57" />
+    </fake_camera>
 </robot>
