Commit message: Use hue detection instead of fake camera

File: mbzirc_gazebo_simulation/uavs_description/models/dji_f550/geometry.xacro (robot description, xacro)
@@ -73,5 +73,5 @@
     >
     <box size="0.01 0.01 0.01"/>
-    <origin xyz="0 0 0.005" rpy="0 1.57079632679 0" />
+    <origin xyz="0 0 -0.275" rpy="0 1.57079632679 0" />
   </xacro:camera_macro>
   <!-- Instantiate rotors -->

File: mbzirc_gazebo_simulation/uavs_description/models/dji_f550/model.xacro (robot description, xacro)
@@ -21,8 +21,8 @@
 		<origin xyz="0 0 -0.275" rpy="0 0 0" />
 </magnetic_gripper>
-<include filename="$(find mbzirc_gazebo_plugins)/urdf/fake_camera.xacro" />
+<!--include filename="$(find mbzirc_gazebo_plugins)/urdf/fake_camera.xacro" />
 <fake_camera parent="base_link" robot_name="dji_f550_$(arg robot_id)">
 		<origin xyz="0.5 0 -0.27" rpy="0 1.57 0" />
-</fake_camera>
+</fake_camera-->
   <xacro:if value="$(arg enable_gps_plugin)">
     <!-- Instantiate gps plugin. -->

Commit message: Copied iris drone blades inertial values to avoid f550 oscilating bug

File: mbzirc_gazebo_simulation/uavs_description/models/dji_f550/geometry.xacro (robot description, xacro)
@@ -5,5 +5,5 @@
   <xacro:property name="description_package" value="uavs_description" />
   <xacro:property name="namespace" value="" />
-  <xacro:property name="rotor_velocity_slowdown_sim" value="10" />
+  <xacro:property name="rotor_velocity_slowdown_sim" value="1" />
   <xacro:property name="mesh_file" value="visual.dae" />
   <xacro:property name="mesh_scale" value="1 1 1"/>
@@ -19,5 +19,5 @@
   <xacro:property name="time_constant_up" value="0.0125" /> <!-- [s] -->
   <xacro:property name="time_constant_down" value="0.025" /> <!-- [s] -->
-  <xacro:property name="max_rot_velocity" value="1100" /> <!-- [rad/s] -->
+  <xacro:property name="max_rot_velocity" value="2100" /> <!-- [rad/s] -->
   <xacro:property name="sin30" value="0.5" />
   <xacro:property name="cos30" value="0.866025403784" />
@@ -30,10 +30,10 @@
     <inertia ixx="0.287" ixy="0.0" ixz="0.0" iyy="0.287" iyz="0.0" izz="0.468" /> <!-- [kg.m^2] [kg.m^2] [kg.m^2] [kg.m^2] [kg.m^2] [kg.m^2] -->
   </xacro:property>
-  <!-- inertia of a single rotor, assuming it is a cuboid. Height=3mm, width=15mm -->
+  <!-- inertia of a single rotor, copied from iris drone blades -->
   <xacro:property name="rotor_inertia">
     <inertia
-    ixx="${1/12 * mass_rotor * (0.015 * 0.015 + 0.003 * 0.003) * rotor_velocity_slowdown_sim}"
-    iyy="${1/12 * mass_rotor * (4 * radius_rotor * radius_rotor + 0.003 * 0.003) * rotor_velocity_slowdown_sim}"
-    izz="${1/12 * mass_rotor * (4 * radius_rotor * radius_rotor + 0.015 * 0.015) * rotor_velocity_slowdown_sim}"
+    ixx="0.00000097"
+    iyy="0.00027310"
+    izz="0.00027310"
     ixy="0.0" ixz="0.0"  iyz="0.0" /> <!-- [kg.m^2] [kg.m^2] [kg.m^2] [kg.m^2] [kg.m^2] [kg.m^2] -->
   </xacro:property>
