Commit message: added gripper

File: mbzirc_gazebo_simulation/atrvjr_gazebo/atrvjr_description/urdf/atrvjr_ur5.urdf.xacro (robot description, xacro)
@@ -15,9 +15,9 @@
         <origin xyz="-0.1 0 0.32" rpy="0.0 0.0 0.0" />
     </joint>
-    <!-- gripper
+    <!-- gripper -->
     <include filename="$(find mbzirc_gazebo_plugins)/urdf/magnetic_gripper.xacro" />
-    <magnetic_gripper parent="ur5_ee_link" robot_name="">
-    		<origin xyz="0 0 0" rpy="1.57 0 0" />
-    </magnetic_gripper> -->
+    <magnetic_gripper parent="ur5_wrist_3_link" robot_name="">
+    		<origin xyz="0 0.1 0" rpy="1.5708 0 0" />
+    </magnetic_gripper>
     <!-- camera -->
     <include filename="$(find mbzirc_gazebo_plugins)/urdf/fake_camera.xacro" />

Commit message: adjustments in atrv navigation configuration and gazebo model

File: mbzirc_gazebo_simulation/atrvjr_gazebo/atrvjr_description/urdf/atrvjr_ur5.urdf.xacro (robot description, xacro)
@@ -23,5 +23,5 @@
     <include filename="$(find mbzirc_gazebo_plugins)/urdf/fake_camera.xacro" />
     <fake_camera parent="center_link" robot_name="">
-    		<origin xyz="0 0.5 0" rpy="0 0 1.57" />
+    		<origin xyz="0 0.3 0" rpy="0 0 1.57" />
     </fake_camera>
 </robot>

Commit message: adapted ugv tasks to run on real robot

File: mbzirc_gazebo_simulation/atrvjr_gazebo/atrvjr_description/urdf/atrvjr_ur5.urdf.xacro (robot description, xacro)
@@ -13,5 +13,5 @@
         <parent link="center_link" />
         <child link = "ur5_base_link" />
-        <origin xyz="-0.1 0 0.32" rpy="0.0 0.0 0.0" />
+        <origin xyz="-0.1 0 0.32" rpy="0.0 0.0 1.5707963267948966" />
     </joint>
     <!-- gripper -->

Commit message: Solve some xacro namespacing issues

File: mbzirc_gazebo_simulation/atrvjr_gazebo/atrvjr_description/urdf/atrvjr_ur5.urdf.xacro (robot description, xacro)
@@ -16,10 +16,10 @@
     </joint>
     <!-- gripper -->
-    <include filename="$(find mbzirc_gazebo_plugins)/urdf/magnetic_gripper.xacro" />
+    <xacro:include filename="$(find mbzirc_gazebo_plugins)/urdf/magnetic_gripper.xacro" />
     <magnetic_gripper parent="ur5_wrist_3_link" robot_name="">
     		<origin xyz="0 0.1 0" rpy="1.5708 0 0" />
     </magnetic_gripper>
     <!-- camera -->
-    <include filename="$(find mbzirc_gazebo_plugins)/urdf/fake_camera.xacro" />
+    <xacro:include filename="$(find mbzirc_gazebo_plugins)/urdf/fake_camera.xacro" />
     <fake_camera parent="center_link" robot_name="">
     		<origin xyz="0 0.3 0" rpy="0 0 1.57" />

File: mbzirc_gazebo_simulation/challenge_worlds/urdf/blue_pile.xacro (robot description, xacro)
@@ -1,2 +1,2 @@
-<?xml version="1.0"?><robot xmlns:xacro="http://www.ros.org/wiki/xacro"><xacro:include filename="$(find challenge_worlds)/urdf/includes/brick_link.xacro" /><macro name="blue_pile" params="id pose"><model name="${id}.pile"><pose>${pose}</pose>
-<brick_link id="0" id2="${id}" type="brick" sx="1.2" sy="0.2" sz="0.2" mass="1.5" material="Gazebo/Blue" pose="0.0 0.0 0.1 0 0 0" /><brick_link id="1" id2="${id}" type="brick" sx="1.2" sy="0.2" sz="0.2" mass="1.5" material="Gazebo/Blue" pose="0.0 0.25 0.1 0 0 0" /><brick_link id="2" id2="${id}" type="brick" sx="1.2" sy="0.2" sz="0.2" mass="1.5" material="Gazebo/Blue" pose="1.25 0.0 0.1 0 0 0" /><brick_link id="3" id2="${id}" type="brick" sx="1.2" sy="0.2" sz="0.2" mass="1.5" material="Gazebo/Blue" pose="1.25 0.25 0.1 0 0 0" /></model></macro></robot>
+<?xml version="1.0"?><robot xmlns:xacro="http://www.ros.org/wiki/xacro"><xacro:include filename="$(find challenge_worlds)/urdf/includes/brick_link.xacro" /><xacro:macro name="blue_pile" params="id pose"><model name="${id}.pile"><pose>${pose}</pose>
+<brick_link id="0" id2="${id}" type="brick" sx="1.2" sy="0.2" sz="0.2" mass="1.5" material="Gazebo/Blue" pose="0.0 0.0 0.1 0 0 0" /><brick_link id="1" id2="${id}" type="brick" sx="1.2" sy="0.2" sz="0.2" mass="1.5" material="Gazebo/Blue" pose="0.0 0.25 0.1 0 0 0" /><brick_link id="2" id2="${id}" type="brick" sx="1.2" sy="0.2" sz="0.2" mass="1.5" material="Gazebo/Blue" pose="1.25 0.0 0.1 0 0 0" /><brick_link id="3" id2="${id}" type="brick" sx="1.2" sy="0.2" sz="0.2" mass="1.5" material="Gazebo/Blue" pose="1.25 0.25 0.1 0 0 0" /></model></xacro:macro></robot>

File: mbzirc_gazebo_simulation/challenge_worlds/urdf/green_pile.xacro (robot description, xacro)
@@ -1,2 +1,2 @@
-<?xml version="1.0"?><robot xmlns:xacro="http://www.ros.org/wiki/xacro"><xacro:include filename="$(find challenge_worlds)/urdf/includes/brick_link.xacro" /><macro name="green_pile" params="id pose"><model name="${id}.pile"><pose>${pose}</pose>
-<brick_link id="0" id2="${id}" type="brick" sx="0.6" sy="0.2" sz="0.2" mass="1.0" material="Gazebo/Green" pose="0.0 0.0 0.1 0 0 0" /><brick_link id="1" id2="${id}" type="brick" sx="0.6" sy="0.2" sz="0.2" mass="1.0" material="Gazebo/Green" pose="0.0 0.25 0.1 0 0 0" /><brick_link id="2" id2="${id}" type="brick" sx="0.6" sy="0.2" sz="0.2" mass="1.0" material="Gazebo/Green" pose="0.65 0.0 0.1 0 0 0" /><brick_link id="3" id2="${id}" type="brick" sx="0.6" sy="0.2" sz="0.2" mass="1.0" material="Gazebo/Green" pose="0.65 0.25 0.1 0 0 0" /></model></macro></robot>
+<?xml version="1.0"?><robot xmlns:xacro="http://www.ros.org/wiki/xacro"><xacro:include filename="$(find challenge_worlds)/urdf/includes/brick_link.xacro" /><xacro:macro name="green_pile" params="id pose"><model name="${id}.pile"><pose>${pose}</pose>
+<brick_link id="0" id2="${id}" type="brick" sx="0.6" sy="0.2" sz="0.2" mass="1.0" material="Gazebo/Green" pose="0.0 0.0 0.1 0 0 0" /><brick_link id="1" id2="${id}" type="brick" sx="0.6" sy="0.2" sz="0.2" mass="1.0" material="Gazebo/Green" pose="0.0 0.25 0.1 0 0 0" /><brick_link id="2" id2="${id}" type="brick" sx="0.6" sy="0.2" sz="0.2" mass="1.0" material="Gazebo/Green" pose="0.65 0.0 0.1 0 0 0" /><brick_link id="3" id2="${id}" type="brick" sx="0.6" sy="0.2" sz="0.2" mass="1.0" material="Gazebo/Green" pose="0.65 0.25 0.1 0 0 0" /></model></xacro:macro></robot>

File: mbzirc_gazebo_simulation/challenge_worlds/urdf/includes/brick_link.xacro (robot description, xacro)
@@ -1,5 +1,5 @@
 <?xml version="1.0"?>
 <robot xmlns:xacro="http://www.ros.org/wiki/xacro">
-<macro name="brick_link" params="id id2 type pose sx sy sz mass material">
+<xacro:macro name="brick_link" params="id id2 type pose sx sy sz mass material">
 <model name="${id2}.${id}.pile">
 	<link name="${id}.${type}">
@@ -35,4 +35,4 @@
         </link>
 </model>
-</macro>
+</xacro:macro>
 </robot>

File: mbzirc_gazebo_simulation/challenge_worlds/urdf/orange_pile.xacro (robot description, xacro)
@@ -1,2 +1,2 @@
-<?xml version="1.0"?><robot xmlns:xacro="http://www.ros.org/wiki/xacro"><xacro:include filename="$(find challenge_worlds)/urdf/includes/brick_link.xacro" /><macro name="orange_pile" params="id pose"><model name="${id}.pile"><pose>${pose}</pose>
-<brick_link id="0" id2="${id}" type="brick" sx="1.8" sy="0.2" sz="0.2" mass="2.0" material="Gazebo/Orange" pose="0.0 0.0 0.1 0 0 0" /><brick_link id="1" id2="${id}" type="brick" sx="1.8" sy="0.2" sz="0.2" mass="2.0" material="Gazebo/Orange" pose="0.0 0.25 0.1 0 0 0" /><brick_link id="2" id2="${id}" type="brick" sx="1.8" sy="0.2" sz="0.2" mass="2.0" material="Gazebo/Orange" pose="1.85 0.0 0.1 0 0 0" /><brick_link id="3" id2="${id}" type="brick" sx="1.8" sy="0.2" sz="0.2" mass="2.0" material="Gazebo/Orange" pose="1.85 0.25 0.1 0 0 0" /></model></macro></robot>
+<?xml version="1.0"?><robot xmlns:xacro="http://www.ros.org/wiki/xacro"><xacro:include filename="$(find challenge_worlds)/urdf/includes/brick_link.xacro" /><xacro:macro name="orange_pile" params="id pose"><model name="${id}.pile"><pose>${pose}</pose>
+<brick_link id="0" id2="${id}" type="brick" sx="1.8" sy="0.2" sz="0.2" mass="2.0" material="Gazebo/Orange" pose="0.0 0.0 0.1 0 0 0" /><brick_link id="1" id2="${id}" type="brick" sx="1.8" sy="0.2" sz="0.2" mass="2.0" material="Gazebo/Orange" pose="0.0 0.25 0.1 0 0 0" /><brick_link id="2" id2="${id}" type="brick" sx="1.8" sy="0.2" sz="0.2" mass="2.0" material="Gazebo/Orange" pose="1.85 0.0 0.1 0 0 0" /><brick_link id="3" id2="${id}" type="brick" sx="1.8" sy="0.2" sz="0.2" mass="2.0" material="Gazebo/Orange" pose="1.85 0.25 0.1 0 0 0" /></model></xacro:macro></robot>

File: mbzirc_gazebo_simulation/challenge_worlds/urdf/red_pile.xacro (robot description, xacro)
@@ -1,2 +1,2 @@
-<?xml version="1.0"?><robot xmlns:xacro="http://www.ros.org/wiki/xacro"><xacro:include filename="$(find challenge_worlds)/urdf/includes/brick_link.xacro" /><macro name="red_pile" params="id pose"><model name="${id}.pile"><pose>${pose}</pose>
-<brick_link id="0" id2="${id}" type="brick" sx="0.3" sy="0.2" sz="0.2" mass="1.0" material="Gazebo/Red" pose="0.0 0.0 0.1 0 0 0" /><brick_link id="1" id2="${id}" type="brick" sx="0.3" sy="0.2" sz="0.2" mass="1.0" material="Gazebo/Red" pose="0.0 0.25 0.1 0 0 0" /><brick_link id="2" id2="${id}" type="brick" sx="0.3" sy="0.2" sz="0.2" mass="1.0" material="Gazebo/Red" pose="0.35 0.0 0.1 0 0 0" /><brick_link id="3" id2="${id}" type="brick" sx="0.3" sy="0.2" sz="0.2" mass="1.0" material="Gazebo/Red" pose="0.35 0.25 0.1 0 0 0" /></model></macro></robot>
+<?xml version="1.0"?><robot xmlns:xacro="http://www.ros.org/wiki/xacro"><xacro:include filename="$(find challenge_worlds)/urdf/includes/brick_link.xacro" /><xacro:macro name="red_pile" params="id pose"><model name="${id}.pile"><pose>${pose}</pose>
+<brick_link id="0" id2="${id}" type="brick" sx="0.3" sy="0.2" sz="0.2" mass="1.0" material="Gazebo/Red" pose="0.0 0.0 0.1 0 0 0" /><brick_link id="1" id2="${id}" type="brick" sx="0.3" sy="0.2" sz="0.2" mass="1.0" material="Gazebo/Red" pose="0.0 0.25 0.1 0 0 0" /><brick_link id="2" id2="${id}" type="brick" sx="0.3" sy="0.2" sz="0.2" mass="1.0" material="Gazebo/Red" pose="0.35 0.0 0.1 0 0 0" /><brick_link id="3" id2="${id}" type="brick" sx="0.3" sy="0.2" sz="0.2" mass="1.0" material="Gazebo/Red" pose="0.35 0.25 0.1 0 0 0" /></model></xacro:macro></robot>

File: mbzirc_gazebo_simulation/challenge_worlds/urdf/single_brick.xacro (robot description, xacro)
@@ -1,2 +1,2 @@
-<?xml version="1.0"?><robot xmlns:xacro="http://www.ros.org/wiki/xacro"><xacro:include filename="$(find challenge_worlds)/urdf/includes/brick_link.xacro" /><macro name="single_brick" params="id pose"><model name="${id}.pile"><pose>${pose}</pose><self_collide>true</self_collide>
-<brick_link id2="0" id="0" type="brick" sx="0.6" sy="0.2" sz="0.2" mass="1.0" material="Gazebo/Orange" pose="0.0 0.0 0.1 0 0 0" /></model></macro></robot>
+<?xml version="1.0"?><robot xmlns:xacro="http://www.ros.org/wiki/xacro"><xacro:include filename="$(find challenge_worlds)/urdf/includes/brick_link.xacro" /><xacro:macro name="single_brick" params="id pose"><model name="${id}.pile"><pose>${pose}</pose><self_collide>true</self_collide>
+<brick_link id2="0" id="0" type="brick" sx="0.6" sy="0.2" sz="0.2" mass="1.0" material="Gazebo/Orange" pose="0.0 0.0 0.1 0 0 0" /></model></xacro:macro></robot>

File: mbzirc_gazebo_simulation/challenge_worlds/worlds/challenge2.world.xacro (robot description, xacro)
@@ -6,10 +6,10 @@
 <xacro:include filename="$(find challenge_worlds)/urdf/green_pile.xacro" />
   <world name="default">
-    <include>
+    <xacro:include>
       <uri>model://ground_plane</uri>
-    </include>
-    <include>
+    </xacro:include>
+    <xacro:include>
       <uri>model://sun</uri>
-    </include>
+    </xacro:include>
    <orange_pile id="1" pose="10 0 0 0 0 0" />
    <blue_pile id="2" pose="-10 0 0 0 0 0" />

File: mbzirc_gazebo_simulation/challenge_worlds/worlds/single_brick.world.xacro (robot description, xacro)
@@ -3,10 +3,10 @@
 <xacro:include filename="$(find challenge_worlds)/urdf/single_brick.xacro" />
   <world name="default">
-    <include>
+    <xacro:include>
       <uri>model://ground_plane</uri>
-    </include>
-    <include>
+    </xacro:include>
+    <xacro:include>
       <uri>model://sun</uri>
-    </include>
+    </xacro:include>
    <single_brick id="1" pose="10 0 0 0 0 0" />
   </world>

File: mbzirc_gazebo_simulation/mbzirc_gazebo_plugins/urdf/fake_camera.xacro (robot description, xacro)
@@ -1,7 +1,7 @@
 <?xml version="1.0"?>
 <robot>
-  <macro name="fake_camera" params="parent *origin robot_name">
+  <xacro:macro name="fake_camera" params="parent *origin robot_name">
   	<joint name="camera_frame_joint" type="fixed">
-      <insert_block name="origin" />
+      <xacro:insert_block name="origin" />
       <parent link="${parent}"/>
       <child link="camera_link"/>
@@ -62,4 +62,4 @@
         </sensor>
     </gazebo>
-  </macro>
+  </xacro:macro>
 </robot>

File: mbzirc_gazebo_simulation/mbzirc_gazebo_plugins/urdf/magnetic_gripper.xacro (robot description, xacro)
@@ -1,7 +1,7 @@
 <?xml version="1.0"?>
-<robot>
-  <macro name="magnetic_gripper" params="parent *origin robot_name">
+<robot xmlns:xacro="http://ros.org/wiki/xacro">
+  <xacro:macro name="magnetic_gripper" params="parent *origin robot_name">
     <joint name="gripper_attach_joint" type="fixed">
-      <insert_block name="origin" />
+      <xacro:insert_block name="origin" />
       <parent link="${parent}"/>
       <child link="gripper_link"/>
@@ -37,4 +37,4 @@
           </plugin>
     </gazebo>
-  </macro>
+  </xacro:macro>
 </robot>

File: mbzirc_gazebo_simulation/mbzirc_gazebo_plugins/urdf/robot.urdf.xacro (robot description, xacro)
@@ -5,5 +5,5 @@
     xmlns:interface="http://playerstage.sourceforge.net/gazebo/xmlschema/#interface">
     <!-- Included URDF Files -->
-  <include filename="$(find mbzirc_gazebo_plugins)/urdf/fake_camera.xacro" />
+  <xacro:include filename="$(find mbzirc_gazebo_plugins)/urdf/fake_camera.xacro" />
   <link name="robot_body">
       <inertial>

File: mbzirc_gazebo_simulation/uavs_description/models/dji_f550/model.xacro (robot description, xacro)
@@ -17,5 +17,5 @@
   <!-- Instantiate dji_f550 "mechanics" -->
   <xacro:include filename="$(find uavs_description)/models/dji_f550/geometry.xacro" />
-<include filename="$(find mbzirc_gazebo_plugins)/urdf/magnetic_gripper.xacro" />
+<xacro:include filename="$(find mbzirc_gazebo_plugins)/urdf/magnetic_gripper.xacro" />
 <magnetic_gripper parent="base_link" robot_name="dji_f550_$(arg robot_id)">
 		<origin xyz="0 0 -0.275" rpy="0 0 0" />
