Commit message: Trick gazebo with a fake revolute joint

File: mbzirc_gazebo_simulation/mbzirc_gazebo_plugins/urdf/magnetic_gripper.xacro (robot description, xacro)
@@ -2,8 +2,9 @@
 <robot xmlns:xacro="http://ros.org/wiki/xacro">
   <xacro:macro name="magnetic_gripper" params="parent *origin robot_name">
-    <joint name="gripper_attach_joint" type="fixed">
+    <joint name="gripper_attach_joint" type="revolute">
       <xacro:insert_block name="origin" />
       <parent link="${parent}"/>
       <child link="gripper_link"/>
+      <limit effort="0" lower="0" upper="0" velocity="0"/>
     </joint>
     <link name="gripper_link">
@@ -30,9 +31,5 @@
       <plugin name="ros_gripper" filename="libmagnetic_gripper_plugin.so">
             <robot_name>${robot_name}</robot_name>
-            <!-- We are forced to magnetize the parent link because of gazebo
-                 automatically lumping fixed joints. This can be prevented just from
-                 SDF 5.0 onwards:
-                 http://answers.gazebosim.org/question/21118/converting-urdf-to-sdf-preservefixedjoint-not-working -->
-            <gripper_link_name>${parent}</gripper_link_name>
+            <gripper_link_name>gripper_link</gripper_link_name>
           </plugin>
     </gazebo>
