Commit message: Fix challenge 3 simulation issues

File: mbzirc_gazebo_simulation/mbzirc_gazebo_plugins/urdf/fake_camera.xacro (robot description, xacro)
@@ -1,4 +1,4 @@
 <?xml version="1.0"?>
-<robot>
+<robot xmlns:xacro="http://ros.org/wiki/xacro">
   <xacro:macro name="fake_camera" params="parent *origin robot_name">
   	<joint name="camera_frame_joint" type="fixed">

File: mbzirc_gazebo_simulation/uavs_description/models/mbzirc2020/geometry.xacro (robot description, xacro)
@@ -40,5 +40,4 @@
   <!-- Included URDF Files -->
   <xacro:include filename="$(find robots_description)/urdf/multirotor_base.xacro" />
-  <xacro:include filename="$(find robots_description)/urdf/component_snippets.xacro" />
   <!-- Instantiate multirotor_base_macro once -->
   <xacro:multirotor_base_macro
@@ -55,49 +54,4 @@
     <xacro:insert_block name="body_inertia" />
   </xacro:multirotor_base_macro>
-<!-- Installing Camera 0 -->
-  <xacro:camera_macro
-    namespace="${namespace}"
-    parent_link="base_link"
-    camera_suffix="0"
-    frame_rate="10"
-    horizontal_fov="1.07079633"
-    image_width="800"
-    image_height="600"
-    image_format="R8G8B8"
-    min_distance="0.01"
-    max_distance="100"
-    noise_mean="0"
-    noise_stddev="0"
-    enable_visual="true"
-    >
-    <box size="0.01 0.01 0.01"/>
-    <origin xyz="0 0 -0.295" rpy="0 1.57079632679 0" />
-  </xacro:camera_macro>
-<!-- Installing Camera 1 -->
-  <!-- <xacro:camera_macro
-    namespace="${namespace}"
-    parent_link="base_link"
-    camera_suffix="1"
-    frame_rate="10"
-    horizontal_fov="1.07079633"
-    image_width="800"
-    image_height="600"
-    image_format="R8G8B8"
-    min_distance="0.01"
-    max_distance="100"
-    noise_mean="0"
-    noise_stddev="0"
-    enable_visual="true"
-    >
-    <xacro:insert_block name="camera_cylinder"/>
-    <origin xyz="0 0.24 -0.24" rpy="0 0 0" />
-  </xacro:camera_macro> -->
-<!-- Installing Teraranger Evo frontal-->
-  <!-- <xacro:teraranger_macro
-    namespace="${model_name}"
-    parent_link="base_link"
-    teraranger_suffix="0"
-  >
-  </xacro:teraranger_macro> -->
   <!-- Instantiate rotors -->
   <xacro:vertical_rotor

File: mbzirc_gazebo_simulation/uavs_description/models/mbzirc2020/model.xacro (robot description, xacro)
@@ -13,12 +13,67 @@
   <xacro:arg name='enable_ground_truth' default='false' />
   <xacro:arg name='enable_logging' default='false' />
+  <xacro:arg name='challenge' default='2' />
   <!-- macros for gazebo plugins, sensors -->
   <xacro:include filename="$(find robots_description)/urdf/component_snippets.xacro" />
   <!-- Instantiate mbzirc "mechanics" -->
   <xacro:include filename="$(find uavs_description)/models/mbzirc2020/geometry.xacro" />
-  <xacro:include filename="$(find mbzirc_gazebo_plugins)/urdf/magnetic_gripper.xacro" />
-  <xacro:magnetic_gripper parent="base_link" robot_name="mbzirc2020_$(arg robot_id)">
-    <origin xyz="0 0 -0.275" rpy="0 0 0" />
-  </xacro:magnetic_gripper>
+  <xacro:if value="${$(arg challenge) == 2}">
+    <!-- Installing magnetic gripper -->
+    <xacro:include filename="$(find mbzirc_gazebo_plugins)/urdf/magnetic_gripper.xacro" />
+    <xacro:magnetic_gripper parent="base_link" robot_name="mbzirc2020_$(arg robot_id)">
+      <origin xyz="0 0 -0.275" rpy="0 0 0" />
+    </xacro:magnetic_gripper>
+    <!-- Installing Camera 0 -->
+    <xacro:camera_macro
+      namespace="${namespace}"
+      parent_link="base_link"
+      camera_suffix="0"
+      frame_rate="10"
+      horizontal_fov="1.07079633"
+      image_width="800"
+      image_height="600"
+      image_format="R8G8B8"
+      min_distance="0.01"
+      max_distance="100"
+      noise_mean="0"
+      noise_stddev="0"
+      enable_visual="true"
+      >
+      <box size="0.01 0.01 0.01"/>
+      <origin xyz="0 0 -0.295" rpy="0 1.57079632679 0" />
+    </xacro:camera_macro>
+  </xacro:if>
+<!-- Installing Camera 1 -->
+  <!-- <xacro:camera_macro
+    namespace="${namespace}"
+    parent_link="base_link"
+    camera_suffix="1"
+    frame_rate="10"
+    horizontal_fov="1.07079633"
+    image_width="800"
+    image_height="600"
+    image_format="R8G8B8"
+    min_distance="0.01"
+    max_distance="100"
+    noise_mean="0"
+    noise_stddev="0"
+    enable_visual="true"
+    >
+    <xacro:insert_block name="camera_cylinder"/>
+    <origin xyz="0 0.24 -0.24" rpy="0 0 0" />
+  </xacro:camera_macro> -->
+<!-- Installing Teraranger Evo frontal-->
+  <!-- <xacro:teraranger_macro
+    namespace="${model_name}"
+    parent_link="base_link"
+    teraranger_suffix="0"
+  >
+  </xacro:teraranger_macro> -->
+  <xacro:include filename="$(find mbzirc_gazebo_plugins)/urdf/fake_camera.xacro" />
+  <xacro:if value="${$(arg challenge) == 3}">
+    <xacro:fake_camera parent="base_link" robot_name="mbzirc2020_$(arg robot_id)">
+      <origin xyz="0.5 0 -0.27" rpy="0 1.57 0" />
+    </xacro:fake_camera>
+  </xacro:if>
   <xacro:if value="$(arg enable_gps_plugin)">
     <!-- Instantiate gps plugin. -->

Commit message: Shrink fake object detection visualization for fov

File: mbzirc_gazebo_simulation/mbzirc_gazebo_plugins/urdf/fake_camera.xacro (robot description, xacro)
@@ -23,5 +23,5 @@
         <origin xyz="0 0 0" rpy="0 0 0"/>
         <geometry>
-          <mesh filename="$(find mbzirc_gazebo_plugins)/mesh/obj_detect_fov.dae"/>
+          <box size="0.01 0.01 0.01" />
         </geometry>
       </visual>
