Commit message: Reduce boilerplate in target iris description

File: mbzirc_gazebo_simulation/uavs_description/models/iris_target_drone/model.xacro (robot description, xacro)
@@ -1,115 +1,86 @@
 <?xml version="1.0"?>
 <robot name="iris" xmlns:xacro="http://ros.org/wiki/xacro">
-  <!-- Properties that can be assigned at build time as arguments.
-  Is there a reason not to make all properties arguments?
-  -->
-  <xacro:arg name='mavlink_addr' default='INADDR_ANY' />
-  <xacro:arg name='mavlink_udp_port' default='14560' />
-  <xacro:arg name='visual_material' default='DarkGrey' />
-  <xacro:arg name='enable_mavlink_interface' default='true' />
-  <xacro:arg name='enable_gps_plugin' default='true' />
-  <xacro:arg name='gps_noise' default='true' />
-  <xacro:arg name='enable_ground_truth' default='false' />
-  <xacro:arg name='enable_logging' default='false' />
-  <!-- macros for gazebo plugins, sensors -->
-  <xacro:include filename="$(find robots_description)/urdf/component_snippets.xacro" />
-  <!-- Instantiate iris "mechanics" -->
-  <xacro:include filename="$(find uavs_description)/models/iris_target_drone/geometry.xacro" />
-  <xacro:if value="$(arg enable_gps_plugin)">
-    <!-- Instantiate gps plugin. -->
-    <xacro:gps_plugin_macro
-      namespace="${namespace}"
-      gps_noise="$(arg gps_noise)"
-      >
-    </xacro:gps_plugin_macro>
-  </xacro:if>
-  <xacro:if value="$(arg enable_mavlink_interface)">
-  <!-- Instantiate mavlink telemetry interface. -->
-  <xacro:mavlink_interface_macro
-    namespace="${namespace}"
-    imu_sub_topic="/imu"
-    mavlink_addr="$(arg mavlink_addr)"
-    mavlink_udp_port="$(arg mavlink_udp_port)"
-    >
-  </xacro:mavlink_interface_macro>
-  </xacro:if>
-  <!-- Mount an ADIS16448 IMU. -->
-  <xacro:imu_plugin_macro
-    namespace="${namespace}"
-    imu_suffix=""
-    parent_link="base_link"
-    imu_topic="/imu"
-    mass_imu_sensor="0.015"
-    gyroscope_noise_density="0.0003394"
-    gyroscopoe_random_walk="0.000038785"
-    gyroscope_bias_correlation_time="1000.0"
-    gyroscope_turn_on_bias_sigma="0.0087"
-    accelerometer_noise_density="0.004"
-    accelerometer_random_walk="0.006"
-    accelerometer_bias_correlation_time="300.0"
-    accelerometer_turn_on_bias_sigma="0.1960"
-  >
-    <inertia ixx="0.00001" ixy="0.0" ixz="0.0" iyy="0.00001" iyz="0.0" izz="0.00001" />
-    <origin xyz="0 0 0" rpy="0 0 0" />
-  </xacro:imu_plugin_macro>
-  <xacro:if value="$(arg enable_ground_truth)">
-    <!-- Mount an IMU providing ground truth. -->
-    <xacro:imu_plugin_macro
-      namespace="${namespace}"
-      imu_suffix="gt"
-      parent_link="base_link"
-      imu_topic="ground_truth/imu"
-      mass_imu_sensor="0.00001"
-      gyroscope_noise_density="0.0"
-      gyroscopoe_random_walk="0.0"
-      gyroscope_bias_correlation_time="1000.0"
-      gyroscope_turn_on_bias_sigma="0.0"
-      accelerometer_noise_density="0.0"
-      accelerometer_random_walk="0.0"
-      accelerometer_bias_correlation_time="300.0"
-      accelerometer_turn_on_bias_sigma="0.0"
-    >
-      <inertia ixx="0.00001" ixy="0.0" ixz="0.0" iyy="0.00001" iyz="0.0" izz="0.00001" />
-      <origin xyz="0 0 0" rpy="0 0 0" />
-    </xacro:imu_plugin_macro>
-    <!-- Mount a generic odometry sensor providing ground truth. -->
-    <xacro:odometry_plugin_macro
-      namespace="${namespace}/ground_truth"
-      odometry_sensor_suffix="gt"
-      parent_link="base_link"
-      pose_topic="pose"
-      pose_with_covariance_topic="pose_with_covariance"
-      position_topic="position"
-      transform_topic="transform"
-      odometry_topic="odometry"
-      parent_frame_id="world"
-      mass_odometry_sensor="0.00001"
-      measurement_divisor="1"
-      measurement_delay="0"
-      unknown_delay="0.0"
-      noise_normal_position="0 0 0"
-      noise_normal_quaternion="0 0 0"
-      noise_normal_linear_velocity="0 0 0"
-      noise_normal_angular_velocity="0 0 0"
-      noise_uniform_position="0 0 0"
-      noise_uniform_quaternion="0 0 0"
-      noise_uniform_linear_velocity="0 0 0"
-      noise_uniform_angular_velocity="0 0 0"
-      enable_odometry_map="false"
-      odometry_map=""
-      image_scale=""
-    >
-      <inertia ixx="0.00001" ixy="0.0" ixz="0.0" iyy="0.00001" iyz="0.0" izz="0.00001" /> <!-- [kg.m^2] [kg.m^2] [kg.m^2] [kg.m^2] [kg.m^2] [kg.m^2] -->
-      <origin xyz="0.0 0.0 0.0" rpy="0.0 0.0 0.0" />
-    </xacro:odometry_plugin_macro>
-  </xacro:if>
-  <xacro:if value="$(arg enable_logging)">
-    <!-- Instantiate a logger -->
-    <xacro:bag_plugin_macro
-      namespace="${namespace}"
-      bag_file="$(arg log_file)"
-      rotor_velocity_slowdown_sim="${rotor_velocity_slowdown_sim}"
-    >
-    </xacro:bag_plugin_macro>
-  </xacro:if>
+  <xacro:arg name="bar_l"           default="1.0"/>
+  <xacro:arg name="ball_r"          default="0.09"/>
+  <xacro:arg name="ball_colour"     default="Gazebo/Green"/>
+  <!-- Instantiate robots_description iris -->
+  <xacro:include filename="$(find robots_description)/models/iris/model.xacro" />
+  <!-- Bar-ball system -->
+  <link name="foo">
+    <inertial>
+      <origin xyz="0 0 0"/>
+      <mass value="0.005"/>
+      <inertia ixx="1e-06" ixy="0" ixz="0" iyy="1e-06" iyz="0" izz="9e-06"/>
+    </inertial>
+    <visual>
+      <origin xyz="0 0 0"/>
+      <geometry>
+        <cylinder radius="0.0005" length="0.001"/>
+      </geometry>
+    </visual>
+    <collision>
+      <origin xyz="0 0 0"/>
+      <geometry>
+        <cylinder radius="0.0005" length="0.001"/>
+      </geometry>
+    </collision>
+  </link>
+  <joint name="base_link_to_foo_joint" type="continuous">
+    <origin xyz="0 0 0"/>
+    <axis xyz="1 0 0"/>
+    <parent link="base_link"/>
+    <child link="foo"/>
+  </joint>
+  <link name="bar">
+    <inertial>
+      <origin xyz="0 0 -${$(arg bar_l)/2}"/>
+      <mass value="0.005"/>
+      <inertia ixx="1e-06" ixy="0" ixz="0" iyy="1e-06" iyz="0" izz="9e-06"/>
+    </inertial>
+    <visual>
+      <origin xyz="0 0 -${$(arg bar_l)/2}"/>
+      <geometry>
+        <cylinder radius="0.0005" length="$(arg bar_l)"/>
+      </geometry>
+    </visual>
+    <collision>
+      <origin xyz="0 0 -${$(arg bar_l)/2}"/>
+      <geometry>
+        <cylinder radius="0.0005" length="$(arg bar_l)"/>
+      </geometry>
+    </collision>
+  </link>
+  <joint name="foo_to_bar_joint" type="continuous">
+    <origin xyz="0 0 0"/>
+    <axis xyz="1 0 0"/>
+    <parent link="foo"/>
+    <child link="bar"/>
+  </joint>
+  <link name="ball">
+    <inertial>
+      <origin xyz="0 0 0"/>
+      <mass value="0.005"/>
+      <inertia ixx="1e-06" ixy="0" ixz="0" iyy="1e-06" iyz="0" izz="9e-06"/>
+    </inertial>
+    <visual>
+      <origin xyz="0 0 0"/>
+      <geometry>
+        <sphere radius="$(arg ball_r)"/>
+      </geometry>
+    </visual>
+    <collision>
+      <origin xyz="0 0 0"/>
+      <geometry>
+        <sphere radius="$(arg ball_r)"/>
+      </geometry>
+    </collision>
+  </link>
+  <joint name="ball_joint" type="fixed">
+    <origin xyz="0 0 -${$(arg bar_l) + $(arg ball_r)}"/>
+    <parent link="bar"/>
+    <child link="ball"/>
+  </joint>
+  <gazebo reference="ball">
+    <material>$(arg ball_colour)</material>
+  </gazebo>
 </robot>

Commit message: Fixed Iris target drone xacro

File: mbzirc_gazebo_simulation/uavs_description/models/iris_target_drone/model.xacro (robot description, xacro)
@@ -1,90 +1,90 @@
 <?xml version="1.0"?>
-<robot name="iris" xmlns:xacro="http://ros.org/wiki/xacro">
-  <xacro:arg name="bar_l"           default="1.0"/>
-  <xacro:arg name="bar_r"           default="0.005"/>
-  <xacro:arg name="bar_mass"        default="0.005"/>
-  <xacro:arg name="ball_r"          default="0.07"/>
-  <xacro:arg name="ball_colour"     default="Gazebo/Red"/>
-  <xacro:arg name="ball_mass"       default="0.09"/>
-  <!-- Instantiate robots_description iris -->
-  <xacro:include filename="$(find robots_description)/models/iris/model.xacro" />
-  <!-- Bar-ball system -->
-  <link name="base_union">
-    <inertial>
+<robot name="iris"
+   xmlns:xacro="http://ros.org/wiki/xacro">
+   <xacro:arg name="bar_l" default="1.0"/>
+   <xacro:arg name="bar_r" default="0.005"/>
+   <xacro:arg name="bar_mass" default="0.005"/>
+   <xacro:arg name="ball_r" default="0.07"/>
+   <xacro:arg name="ball_colour" default="Gazebo/Red"/>
+   <xacro:arg name="ball_mass" default="0.09"/>
+   <!-- Instantiate robots_description iris -->
+   <xacro:include filename="$(find robots_description)/models/iris/model.xacro" />
+   <!-- Bar-ball system -->
+   <link name="base_union">
+      <inertial>
+         <origin xyz="0 0 0"/>
+         <mass value="0.005"/>
+         <inertia ixx="1e-06" ixy="0" ixz="0" iyy="1e-06" iyz="0" izz="9e-06"/>
+      </inertial>
+      <visual>
+         <origin xyz="0 0 0"/>
+         <geometry>
+            <cylinder radius="0.0005" length="0.001"/>
+         </geometry>
+      </visual>
+      <collision>
+         <origin xyz="0 0 0"/>
+         <geometry>
+            <cylinder radius="0.0005" length="0.001"/>
+         </geometry>
+      </collision>
+   </link>
+   <joint name="base_link_to_base_union_joint" type="continuous">
       <origin xyz="0 0 0"/>
-      <mass value="0.005"/>
-      <inertia ixx="1e-06" ixy="0" ixz="0" iyy="1e-06" iyz="0" izz="9e-06"/>
-    </inertial>
-    <visual>
+      <axis xyz="1 0 0"/>
+      <parent link="base_link"/>
+      <child link="base_union"/>
+   </joint>
+   <link name="bar">
+      <inertial>
+         <origin xyz="0 ${$(arg bar_l)/2} 0" rpy="1.5707963267948966 0 0"/>
+         <mass value="$(arg bar_mass)"/>
+         <inertia ixx="${(1/12)*$(arg bar_mass)*(3*$(arg bar_r)*$(arg bar_r)+$(arg bar_l)*$(arg bar_l)) }" ixy="0" ixz="0" iyy="${(1/12)*$(arg bar_mass)*(3*$(arg bar_r)*$(arg bar_r)+$(arg bar_l)*$(arg bar_l)) }" iyz="0" izz="${(1/12)*$(arg bar_mass)*(3*$(arg bar_r)*$(arg bar_r)+$(arg bar_l)*$(arg bar_l)) }"/>
+      </inertial>
+      <visual>
+         <origin xyz="0 ${$(arg bar_l)/2} 0" rpy="1.5707963267948966 0 0"/>
+         <geometry>
+            <cylinder radius="$(arg bar_r)" length="$(arg bar_l)"/>
+         </geometry>
+      </visual>
+      <collision>
+         <origin xyz="0 ${$(arg bar_l)/2} 0" rpy="1.5707963267948966 0 0"/>
+         <geometry>
+            <cylinder radius="$(arg bar_r)" length="$(arg bar_l)"/>
+         </geometry>
+      </collision>
+   </link>
+   <joint name="base_union_to_bar_joint" type="continuous">
       <origin xyz="0 0 0"/>
-      <geometry>
-        <cylinder radius="0.0005" length="0.001"/>
-      </geometry>
-    </visual>
-    <collision>
-      <origin xyz="0 0 0"/>
-      <geometry>
-        <cylinder radius="0.0005" length="0.001"/>
-      </geometry>
-    </collision>
-  </link>
-  <joint name="base_link_to_base_union_joint" type="continuous">
-    <origin xyz="0 0 0"/>
-    <axis xyz="1 0 0"/>
-    <parent link="base_link"/>
-    <child link="base_union"/>
-  </joint>
-  <link name="bar">
-    <inertial>
-      <origin xyz="0 ${$(arg bar_l)/2} 0" rpy="1.5707963267948966 0 0"/>
-      <mass value="${arg bar_mass}"/>
-      <inertia ixx="${(1/12)*${arg bar_mass}*(3*${arg bar_r}*${arg bar_r}+${arg bar_l}*${arg bar_l})}" ixy="0" ixz="0" iyy="${(1/12)*${arg bar_mass}*(3*${arg bar_r}*${arg bar_r}+${arg bar_l}*${arg bar_l})}" iyz="0" izz="${(1/12)*${arg bar_mass}*(3*${arg bar_r}*${arg bar_r}+${arg bar_l}*${arg bar_l})}"/>
-    </inertial>
-    <visual>
-      <origin xyz="0 ${$(arg bar_l)/2} 0" rpy="1.5707963267948966 0 0"/>
-      <geometry>
-        <cylinder radius="${arg bar_r}" length="$(arg bar_l)"/>
-      </geometry>
-    </visual>
-    <collision>
-      <origin xyz="0 ${$(arg bar_l)/2} 0" rpy="1.5707963267948966 0 0"/>
-      <geometry>
-        <cylinder radius="${arg bar_r}" length="$(arg bar_l)"/>
-      </geometry>
-    </collision>
-  </link>
-  <joint name="base_union_to_bar_joint" type="continuous">
-    <origin xyz="0 0 0"/>
-    <axis xyz="1 0 0"/>
-    <parent link="base_union"/>
-    <child link="bar"/>
-  </joint>
-  <link name="ball">
-    <inertial>
-      <origin xyz="0 0 0"/>
-      <mass value="${arg ball_mass}"/>
-      <inertia ixx="${(2/5)*${arg ball_mass}*${arg ball_r}*${arg ball_r}}" ixy="0" ixz="0"
-               iyy="${(2/5)*${arg ball_mass}*${arg ball_r}*${arg ball_r}}" iyz="0" izz="${(2/5)*${arg ball_mass}*${arg ball_r}*${arg ball_r}}"/>
-    </inertial>
-    <visual>
-      <origin xyz="0 0 0"/>
-      <geometry>
-        <sphere radius="$(arg ball_r)"/>
-      </geometry>
-    </visual>
-    <collision>
-      <origin xyz="0 0 0"/>
-      <geometry>
-        <sphere radius="$(arg ball_r)"/>
-      </geometry>
-    </collision>
-  </link>
-  <joint name="ball_joint" type="fixed">
-    <origin xyz="0 ${$(arg bar_l) + $(arg ball_r)} 0"/>
-    <parent link="bar"/>
-    <child link="ball"/>
-  </joint>
-  <gazebo reference="ball">
-    <material>$(arg ball_colour)</material>
-  </gazebo>
+      <axis xyz="1 0 0"/>
+      <parent link="base_union"/>
+      <child link="bar"/>
+   </joint>
+   <link name="ball">
+      <inertial>
+         <origin xyz="0 0 0"/>
+         <mass value="$(arg ball_mass)"/>
+         <inertia ixx="${(2/5)*$(arg ball_mass)*$(arg ball_r)*$(arg ball_r)}" ixy="0" ixz="0" iyy="${(2/5)*$(arg ball_mass)*$(arg ball_r)*$(arg ball_r)}" iyz="0" izz="${(2/5)*$(arg ball_mass)*$(arg ball_r)*$(arg ball_r)}"/>
+      </inertial>
+      <visual>
+         <origin xyz="0 0 0"/>
+         <geometry>
+            <sphere radius="$(arg ball_r)"/>
+         </geometry>
+      </visual>
+      <collision>
+         <origin xyz="0 0 0"/>
+         <geometry>
+            <sphere radius="$(arg ball_r)"/>
+         </geometry>
+      </collision>
+   </link>
+   <joint name="ball_joint" type="fixed">
+      <origin xyz="0 ${$(arg bar_l) + $(arg ball_r)} 0"/>
+      <parent link="bar"/>
+      <child link="ball"/>
+   </joint>
+   <gazebo reference="ball">
+      <material>$(arg ball_colour)</material>
+   </gazebo>
 </robot>
