Commit message: Added depth camera

File: mbzirc_gazebo_simulation/uavs_description/models/dji_f550_c1/geometry.xacro (robot description, xacro)
@@ -56,23 +56,80 @@
     <xacro:insert_block name="body_inertia" />
   </xacro:multirotor_base_macro>
-  <!-- Visual camera -->
-  <xacro:camera_macro
-    namespace="${namespace}"
-    parent_link="base_link"
-    camera_suffix="rgb"
-    frame_rate="30"
-    horizontal_fov="1.57108"
-    image_width="848"
-    image_height="480"
-    image_format="R8G8B8"
-    min_distance="0.01"
-    max_distance="100"
-    noise_mean="0"
-    noise_stddev="0"
-    enable_visual="true"
-    >
-    <box size="0.01 0.01 0.01"/>
-    <origin xyz="0.16 0 -0.04" rpy="0 0.41887902047863906 0" />
-  </xacro:camera_macro>
+<!-- Visual RGB-D camera -->
+<xacro:macro name="camera_macro"
+    params="namespace parent_link camera_suffix frame_rate
+      horizontal_fov focal_length image_width image_height image_format min_distance
+      max_distance baseline noise_mean noise_stddev *origin">
+<link name='camera_link'>
+    <xacro:insert_block name="origin" />
+    <collision>
+        <origin xyz="0 0 0" rpy="0 0 0" />
+        <geometry>
+          <cylinder radius="0.01" length="0.05"/>
+        </geometry>
+    </collision>
+    <inertial>
+      <mass value="1e-5" />
+      <origin xyz="0 0 0" rpy="0 0 0" />
+      <inertia ixx="1e-6" ixy="0" ixz="0" iyy="1e-6" iyz="0" izz="1e-6" />
+    </inertial>
+</link>
+  <gazebo reference="camera_link">
+    <sensor name='camera' type='depth'>
+      <update_rate>${frame_rate}</update_rate>
+      <camera name='intel_d435'>
+        <horizontal_fov>${horizontal_fov}</horizontal_fov> <!--1.57108-->
+        <image>
+          <width>${image_width}</width>
+          <height>${image_height}</height>
+          <format>${image_format}</format>
+        </image>
+        <clip>
+          <near>${min_distance}</near>
+          <far>${max_distance}</far>
+        </clip>
+        <noise>
+            <type>gaussian</type>
+            <!-- Noise is sampled independently per pixel on each frame.
+                 That pixel's noise value is added to each of its color
+                 channels, which at that point lie in the range [0,1]. -->
+            <mean>${noise_mean}</mean>
+            <stddev>${noise_stddev}</stddev>
+          </noise>
+      </camera>
+      <plugin name='intel_D435_plugin' filename='libgazebo_ros_openni_kinect.so'>
+        <baseline>${baseline}</baseline> <!--0.05-->
+        <alwaysOn>1</alwaysOn>
+        <updateRate>${frame_rate}</updateRate>
+        <cameraName>${namespace}_camera_${camera_suffix}</cameraName>
+        <imageTopicName>rgb/image_raw</imageTopicName>
+        <cameraInfoTopicName>rgb/camera_info</cameraInfoTopicName>
+        <depthImageTopicName>depth/image_raw</depthImageTopicName>
+        <depthImageInfoTopicName>depth/camera_info</depthImageInfoTopicName>
+        <pointCloudTopicName>depth/points</pointCloudTopicName>
+        <frameName>camera_link</frameName>
+        <pointCloudCutoff>0.15</pointCloudCutoff>
+        <pointCloudCutoffMax>10</pointCloudCutoffMax>
+        <distortionK1>0</distortionK1>
+        <distortionK2>0</distortionK2>
+        <distortionK3>0</distortionK3>
+        <distortionT1>0</distortionT1>
+        <distortionT2>0</distortionT2>
+        <CxPrime>0</CxPrime>
+        <Cx>0</Cx>
+        <Cy>0</Cy>
+        <!-- <focalLength>1.93</focalLength> -->
+        <!-- <focalLength>420.22</focalLength> -->
+        <focalLength>${focal_length}</focalLength>  <!-- 599.7654 -->
+        <hackBaseline>0</hackBaseline>
+      </plugin>
+    </sensor>
+  </gazebo>
+  <joint name="${namespace}/camera_joint" type="fixed">
+      <origin xyz="0.16 0 -0.04" rpy="0 0.41887902047863906 0" />
+      <parent link="${parent_link}" />
+      <child link="camera_link" />
+  </joint>
+  </xacro:macro>
   <!-- Instantiate rotors -->
   <xacro:vertical_rotor

File: mbzirc_gazebo_simulation/uavs_description/models/dji_f550_c1/model.xacro (robot description, xacro)
@@ -26,4 +26,22 @@
 		<origin xyz="0.5 0 -0.27" rpy="0 1.57 0" />
 </fake_camera-->
+  <xacro:camera_macro
+    namespace="dji_F550"
+    parent_link="base_link"
+    camera_suffix="$(arg robot_id)"
+    frame_rate="30"
+    horizontal_fov="1.57108"
+    focal_length="599.7654"
+    image_width="848"
+    image_height="480"
+    image_format="R8G8B8"
+    min_distance="0.01"
+    max_distance="100"
+    baseline="0.05"
+    noise_mean="0.1"
+    noise_stddev="0.001"
+    >
+  <origin xyz="0.16 0 -0.04" rpy="0 0.41887902047863906 0" />
+</xacro:camera_macro>
   <xacro:if value="$(arg enable_gps_plugin)">
     <!-- Instantiate gps plugin. -->

Commit message: Removed agent 1 task and renamed camera to dji_f550_camera_x

File: mbzirc_gazebo_simulation/uavs_description/models/dji_f550_c1/geometry.xacro (robot description, xacro)
@@ -1,4 +1,5 @@
 <?xml version="1.0"?>
-<robot name="dji_f550_c1" xmlns:xacro="http://ros.org/wiki/xacro">
+<robot name="dji_f550_c1"
+  xmlns:xacro="http://ros.org/wiki/xacro">
   <!-- Properties -->
   <xacro:property name="model_name" value="dji_f550_c1" />
@@ -9,15 +10,26 @@
   <xacro:property name="mesh_scale" value="1 1 1"/>
   <xacro:property name="mesh_scale_prop" value="1 1 1"/>
-  <xacro:property name="mass" value="5.850" /> <!-- [kg] -->
-  <xacro:property name="body_width" value="0.600" /> <!-- [m] -->
-  <xacro:property name="body_height" value="0.08" /> <!-- [m] -->
-  <xacro:property name="mass_rotor" value="0.005" /> <!-- [kg] -->
-  <xacro:property name="rotor_offset_top" value="0.0" /> <!-- [m] -->
-  <xacro:property name="radius_rotor" value="0.12" /> <!-- [m] -->
-  <xacro:property name="motor_constant" value="20.0e-06" /> <!-- [kg.m/s^2] -->
-  <xacro:property name="moment_constant" value="0.12" /> <!-- [m] -->
-  <xacro:property name="time_constant_up" value="0.0125" /> <!-- [s] -->
-  <xacro:property name="time_constant_down" value="0.025" /> <!-- [s] -->
-  <xacro:property name="max_rot_velocity" value="2100" /> <!-- [rad/s] -->
+  <xacro:property name="mass" value="5.850" />
+  <!-- [kg] -->
+  <xacro:property name="body_width" value="0.600" />
+  <!-- [m] -->
+  <xacro:property name="body_height" value="0.08" />
+  <!-- [m] -->
+  <xacro:property name="mass_rotor" value="0.005" />
+  <!-- [kg] -->
+  <xacro:property name="rotor_offset_top" value="0.0" />
+  <!-- [m] -->
+  <xacro:property name="radius_rotor" value="0.12" />
+  <!-- [m] -->
+  <xacro:property name="motor_constant" value="20.0e-06" />
+  <!-- [kg.m/s^2] -->
+  <xacro:property name="moment_constant" value="0.12" />
+  <!-- [m] -->
+  <xacro:property name="time_constant_up" value="0.0125" />
+  <!-- [s] -->
+  <xacro:property name="time_constant_down" value="0.025" />
+  <!-- [s] -->
+  <xacro:property name="max_rot_velocity" value="11000" />
+  <!-- [rad/s] -->
   <xacro:property name="sin30" value="0.5" />
   <xacro:property name="cos30" value="0.866025403784" />
@@ -28,13 +40,11 @@
   <!-- Property Blocks -->
   <xacro:property name="body_inertia">
-    <inertia ixx="0.287" ixy="0.0" ixz="0.0" iyy="0.287" iyz="0.0" izz="0.468" /> <!-- [kg.m^2] [kg.m^2] [kg.m^2] [kg.m^2] [kg.m^2] [kg.m^2] -->
+    <inertia ixx="0.287" ixy="0.0" ixz="0.0" iyy="0.287" iyz="0.0" izz="0.468" />
+    <!-- [kg.m^2] [kg.m^2] [kg.m^2] [kg.m^2] [kg.m^2] [kg.m^2] -->
   </xacro:property>
   <!-- inertia of a single rotor, copied from iris drone blades -->
   <xacro:property name="rotor_inertia">
-    <inertia
-    ixx="0.00000097"
-    iyy="0.00027310"
-    izz="0.00027310"
-    ixy="0.0" ixz="0.0"  iyz="0.0" /> <!-- [kg.m^2] [kg.m^2] [kg.m^2] [kg.m^2] [kg.m^2] [kg.m^2] -->
+    <inertia ixx="0.00000097" iyy="0.00027310" izz="0.00027310" ixy="0.0" ixz="0.0" iyz="0.0" />
+    <!-- [kg.m^2] [kg.m^2] [kg.m^2] [kg.m^2] [kg.m^2] [kg.m^2] -->
   </xacro:property>
   <!-- Included URDF Files -->
@@ -42,52 +52,40 @@
   <xacro:include filename="$(find robots_description)/urdf/component_snippets.xacro" />
   <!-- Instantiate multirotor_base_macro once -->
-  <xacro:multirotor_base_macro
-    description_package="${description_package}"
-    model_name="${model_name}"
-    robot_namespace="${namespace}"
-    mass="${mass}"
-    body_width="${body_width}"
-    body_height="${body_height}"
-    height_offset="0.0"
-    mesh_file="${mesh_file}"
-    mesh_scale="${mesh_scale}"
-    color=""
-    >
+  <xacro:multirotor_base_macro description_package="${description_package}" model_name="${model_name}" robot_namespace="${namespace}" mass="${mass}" body_width="${body_width}" body_height="${body_height}" height_offset="0.0" mesh_file="${mesh_file}" mesh_scale="${mesh_scale}" color="">
     <xacro:insert_block name="body_inertia" />
   </xacro:multirotor_base_macro>
-<!-- Visual RGB-D camera -->
-<xacro:macro name="camera_macro"
-    params="namespace parent_link camera_suffix frame_rate
+  <!-- Visual RGB-D camera -->
+  <xacro:macro name="rgbd_camera_macro" params="namespace parent_link camera_suffix frame_rate
       horizontal_fov focal_length image_width image_height image_format min_distance
       max_distance baseline noise_mean noise_stddev *origin">
-<link name='camera_link'>
-    <xacro:insert_block name="origin" />
-    <collision>
+    <link name='camera_link'>
+      <xacro:insert_block name="origin" />
+      <collision>
         <origin xyz="0 0 0" rpy="0 0 0" />
         <geometry>
           <cylinder radius="0.01" length="0.05"/>
         </geometry>
-    </collision>
-    <inertial>
-      <mass value="1e-5" />
-      <origin xyz="0 0 0" rpy="0 0 0" />
-      <inertia ixx="1e-6" ixy="0" ixz="0" iyy="1e-6" iyz="0" izz="1e-6" />
-    </inertial>
-</link>
-  <gazebo reference="camera_link">
-    <sensor name='camera' type='depth'>
-      <update_rate>${frame_rate}</update_rate>
-      <camera name='intel_d435'>
-        <horizontal_fov>${horizontal_fov}</horizontal_fov> <!--1.57108-->
-        <image>
-          <width>${image_width}</width>
-          <height>${image_height}</height>
-          <format>${image_format}</format>
-        </image>
-        <clip>
-          <near>${min_distance}</near>
-          <far>${max_distance}</far>
-        </clip>
-        <noise>
+      </collision>
+      <inertial>
+        <mass value="1e-5" />
+        <origin xyz="0 0 0" rpy="0 0 0" />
+        <inertia ixx="1e-6" ixy="0" ixz="0" iyy="1e-6" iyz="0" izz="1e-6" />
+      </inertial>
+    </link>
+    <gazebo reference="camera_link">
+      <sensor name='camera' type='depth'>
+        <update_rate>${frame_rate}</update_rate>
+        <camera name='intel_d435'>
+          <horizontal_fov>${horizontal_fov}</horizontal_fov>          <!--1.57108-->
+          <image>
+            <width>${image_width}</width>
+            <height>${image_height}</height>
+            <format>${image_format}</format>
+          </image>
+          <clip>
+            <near>${min_distance}</near>
+            <far>${max_distance}</far>
+          </clip>
+          <noise>
             <type>gaussian</type>
             <!-- Noise is sampled independently per pixel on each frame.
@@ -97,169 +95,61 @@
             <stddev>${noise_stddev}</stddev>
           </noise>
-      </camera>
-      <plugin name='intel_D435_plugin' filename='libgazebo_ros_openni_kinect.so'>
-        <baseline>${baseline}</baseline> <!--0.05-->
-        <alwaysOn>1</alwaysOn>
-        <updateRate>${frame_rate}</updateRate>
-        <cameraName>${namespace}_camera_${camera_suffix}</cameraName>
-        <imageTopicName>rgb/image_raw</imageTopicName>
-        <cameraInfoTopicName>rgb/camera_info</cameraInfoTopicName>
-        <depthImageTopicName>depth/image_raw</depthImageTopicName>
-        <depthImageInfoTopicName>depth/camera_info</depthImageInfoTopicName>
-        <pointCloudTopicName>depth/points</pointCloudTopicName>
-        <frameName>camera_link</frameName>
-        <pointCloudCutoff>0.15</pointCloudCutoff>
-        <pointCloudCutoffMax>10</pointCloudCutoffMax>
-        <distortionK1>0</distortionK1>
-        <distortionK2>0</distortionK2>
-        <distortionK3>0</distortionK3>
-        <distortionT1>0</distortionT1>
-        <distortionT2>0</distortionT2>
-        <CxPrime>0</CxPrime>
-        <Cx>0</Cx>
-        <Cy>0</Cy>
-        <!-- <focalLength>1.93</focalLength> -->
-        <!-- <focalLength>420.22</focalLength> -->
-        <focalLength>${focal_length}</focalLength>  <!-- 599.7654 -->
-        <hackBaseline>0</hackBaseline>
-      </plugin>
-    </sensor>
-  </gazebo>
-  <joint name="${namespace}/camera_joint" type="fixed">
+        </camera>
+        <plugin name='intel_D435_plugin' filename='libgazebo_ros_openni_kinect.so'>
+          <baseline>${baseline}</baseline>          <!--0.05-->
+          <alwaysOn>1</alwaysOn>
+          <updateRate>${frame_rate}</updateRate>
+          <cameraName>${namespace}_camera_${camera_suffix}</cameraName>
+          <imageTopicName>rgb/image_raw</imageTopicName>
+          <cameraInfoTopicName>rgb/camera_info</cameraInfoTopicName>
+          <depthImageTopicName>depth/image_raw</depthImageTopicName>
+          <depthImageInfoTopicName>depth/camera_info</depthImageInfoTopicName>
+          <pointCloudTopicName>depth/points</pointCloudTopicName>
+          <frameName>camera_link</frameName>
+          <pointCloudCutoff>0.15</pointCloudCutoff>
+          <pointCloudCutoffMax>10</pointCloudCutoffMax>
+          <distortionK1>0</distortionK1>
+          <distortionK2>0</distortionK2>
+          <distortionK3>0</distortionK3>
+          <distortionT1>0</distortionT1>
+          <distortionT2>0</distortionT2>
+          <CxPrime>0</CxPrime>
+          <Cx>0</Cx>
+          <Cy>0</Cy>
+          <!-- <focalLength>1.93</focalLength> -->
+          <!-- <focalLength>420.22</focalLength> -->
+          <focalLength>${focal_length}</focalLength>          <!-- 599.7654 -->
+          <hackBaseline>0</hackBaseline>
+        </plugin>
+      </sensor>
+    </gazebo>
+    <joint name="${namespace}/camera_joint" type="fixed">
       <origin xyz="0.16 0 -0.04" rpy="0 0.41887902047863906 0" />
       <parent link="${parent_link}" />
       <child link="camera_link" />
-  </joint>
+    </joint>
   </xacro:macro>
   <!-- Instantiate rotors -->
-  <xacro:vertical_rotor
-    description_package="${description_package}"
-    robot_namespace="${namespace}"
-    suffix="right"
-    direction="cw"
-    motor_constant="${motor_constant}"
-    moment_constant="${moment_constant}"
-    parent="base_link"
-    mass_rotor="${mass_rotor}"
-    radius_rotor="${radius_rotor}"
-    time_constant_up="${time_constant_up}"
-    time_constant_down="${time_constant_down}"
-    max_rot_velocity="${max_rot_velocity}"
-    motor_number="0"
-    rotor_drag_coefficient="${rotor_drag_coefficient}"
-    rolling_moment_coefficient="${rolling_moment_coefficient}"
-    mesh="prop"
-    mesh_scale="${mesh_scale_prop}"
-    color="DarkGrey">
+  <xacro:vertical_rotor description_package="${description_package}" robot_namespace="${namespace}" suffix="right" direction="cw" motor_constant="${motor_constant}" moment_constant="${moment_constant}" parent="base_link" mass_rotor="${mass_rotor}" radius_rotor="${radius_rotor}" time_constant_up="${time_constant_up}" time_constant_down="${time_constant_down}" max_rot_velocity="${max_rot_velocity}" motor_number="0" rotor_drag_coefficient="${rotor_drag_coefficient}" rolling_moment_coefficient="${rolling_moment_coefficient}" mesh="prop" mesh_scale="${mesh_scale_prop}" color="DarkGrey">
     <origin xyz="0 -0.272 0.074" rpy="0 0 0" />
     <xacro:insert_block name="rotor_inertia" />
   </xacro:vertical_rotor>
-  <xacro:vertical_rotor
-    description_package="${description_package}"
-    robot_namespace="${namespace}"
-    suffix="left"
-    direction="ccw"
-    motor_constant="${motor_constant}"
-    moment_constant="${moment_constant}"
-    parent="base_link"
-    mass_rotor="${mass_rotor}"
-    radius_rotor="${radius_rotor}"
-    time_constant_up="${time_constant_up}"
-    time_constant_down="${time_constant_down}"
-    max_rot_velocity="${max_rot_velocity}"
-    motor_number="1"
-    rotor_drag_coefficient="${rotor_drag_coefficient}"
-    rolling_moment_coefficient="${rolling_moment_coefficient}"
-    mesh="prop"
-    mesh_scale="${mesh_scale_prop}"
-    color="DarkGrey">
+  <xacro:vertical_rotor description_package="${description_package}" robot_namespace="${namespace}" suffix="left" direction="ccw" motor_constant="${motor_constant}" moment_constant="${moment_constant}" parent="base_link" mass_rotor="${mass_rotor}" radius_rotor="${radius_rotor}" time_constant_up="${time_constant_up}" time_constant_down="${time_constant_down}" max_rot_velocity="${max_rot_velocity}" motor_number="1" rotor_drag_coefficient="${rotor_drag_coefficient}" rolling_moment_coefficient="${rolling_moment_coefficient}" mesh="prop" mesh_scale="${mesh_scale_prop}" color="DarkGrey">
     <origin xyz="0 0.272 0.074" rpy="0 0 0" />
     <xacro:insert_block name="rotor_inertia" />
   </xacro:vertical_rotor>
-  <xacro:vertical_rotor
-    description_package="${description_package}"
-    robot_namespace="${namespace}"
-    suffix="front_left"
-    direction="cw"
-    motor_constant="${motor_constant}"
-    moment_constant="${moment_constant}"
-    parent="base_link"
-    mass_rotor="${mass_rotor}"
-    radius_rotor="${radius_rotor}"
-    time_constant_up="${time_constant_up}"
-    time_constant_down="${time_constant_down}"
-    max_rot_velocity="${max_rot_velocity}"
-    motor_number="2"
-    rotor_drag_coefficient="${rotor_drag_coefficient}"
-    rolling_moment_coefficient="${rolling_moment_coefficient}"
-    mesh="prop"
-    mesh_scale="${mesh_scale_prop}"
-    color="${color}">
+  <xacro:vertical_rotor description_package="${description_package}" robot_namespace="${namespace}" suffix="front_left" direction="cw" motor_constant="${motor_constant}" moment_constant="${moment_constant}" parent="base_link" mass_rotor="${mass_rotor}" radius_rotor="${radius_rotor}" time_constant_up="${time_constant_up}" time_constant_down="${time_constant_down}" max_rot_velocity="${max_rot_velocity}" motor_number="2" rotor_drag_coefficient="${rotor_drag_coefficient}" rolling_moment_coefficient="${rolling_moment_coefficient}" mesh="prop" mesh_scale="${mesh_scale_prop}" color="${color}">
     <origin xyz="0.23556 0.136 0.074" rpy="0 0 0" />
     <xacro:insert_block name="rotor_inertia" />
   </xacro:vertical_rotor>
-  <xacro:vertical_rotor
-    description_package="${description_package}"
-    robot_namespace="${namespace}"
-    suffix="back_right"
-    direction="ccw"
-    motor_constant="${motor_constant}"
-    moment_constant="${moment_constant}"
-    parent="base_link"
-    mass_rotor="${mass_rotor}"
-    radius_rotor="${radius_rotor}"
-    time_constant_up="${time_constant_up}"
-    time_constant_down="${time_constant_down}"
-    max_rot_velocity="${max_rot_velocity}"
-    motor_number="3"
-    rotor_drag_coefficient="${rotor_drag_coefficient}"
-    rolling_moment_coefficient="${rolling_moment_coefficient}"
-    mesh="prop"
-    mesh_scale="${mesh_scale_prop}"
-    color="DarkGrey">
+  <xacro:vertical_rotor description_package="${description_package}" robot_namespace="${namespace}" suffix="back_right" direction="ccw" motor_constant="${motor_constant}" moment_constant="${moment_constant}" parent="base_link" mass_rotor="${mass_rotor}" radius_rotor="${radius_rotor}" time_constant_up="${time_constant_up}" time_constant_down="${time_constant_down}" max_rot_velocity="${max_rot_velocity}" motor_number="3" rotor_drag_coefficient="${rotor_drag_coefficient}" rolling_moment_coefficient="${rolling_moment_coefficient}" mesh="prop" mesh_scale="${mesh_scale_prop}" color="DarkGrey">
     <origin xyz="-0.23556 -0.136 0.074" rpy="0 0 0" />
     <xacro:insert_block name="rotor_inertia" />
   </xacro:vertical_rotor>
-  <xacro:vertical_rotor
-    description_package="${description_package}"
-    robot_namespace="${namespace}"
-    suffix="front_right"
-    direction="ccw"
-    motor_constant="${motor_constant}"
-    moment_constant="${moment_constant}"
-    parent="base_link"
-    mass_rotor="${mass_rotor}"
-    radius_rotor="${radius_rotor}"
-    time_constant_up="${time_constant_up}"
-    time_constant_down="${time_constant_down}"
-    max_rot_velocity="${max_rot_velocity}"
-    motor_number="4"
-    rotor_drag_coefficient="${rotor_drag_coefficient}"
-    rolling_moment_coefficient="${rolling_moment_coefficient}"
-    mesh="prop"
-    mesh_scale="${mesh_scale_prop}"
-    color="${color}">
+  <xacro:vertical_rotor description_package="${description_package}" robot_namespace="${namespace}" suffix="front_right" direction="ccw" motor_constant="${motor_constant}" moment_constant="${moment_constant}" parent="base_link" mass_rotor="${mass_rotor}" radius_rotor="${radius_rotor}" time_constant_up="${time_constant_up}" time_constant_down="${time_constant_down}" max_rot_velocity="${max_rot_velocity}" motor_number="4" rotor_drag_coefficient="${rotor_drag_coefficient}" rolling_moment_coefficient="${rolling_moment_coefficient}" mesh="prop" mesh_scale="${mesh_scale_prop}" color="${color}">
     <origin xyz="0.23556 -0.136 0.074" rpy="0 0 0" />
     <xacro:insert_block name="rotor_inertia" />
   </xacro:vertical_rotor>
-  <xacro:vertical_rotor
-    description_package="${description_package}"
-    robot_namespace="${namespace}"
-    suffix="back_left"
-    direction="cw"
-    motor_constant="${motor_constant}"
-    moment_constant="${moment_constant}"
-    parent="base_link"
-    mass_rotor="${mass_rotor}"
-    radius_rotor="${radius_rotor}"
-    time_constant_up="${time_constant_up}"
-    time_constant_down="${time_constant_down}"
-    max_rot_velocity="${max_rot_velocity}"
-    motor_number="5"
-    rotor_drag_coefficient="${rotor_drag_coefficient}"
-    rolling_moment_coefficient="${rolling_moment_coefficient}"
-    mesh="prop"
-    mesh_scale="${mesh_scale_prop}"
-    color="DarkGrey">
+  <xacro:vertical_rotor description_package="${description_package}" robot_namespace="${namespace}" suffix="back_left" direction="cw" motor_constant="${motor_constant}" moment_constant="${moment_constant}" parent="base_link" mass_rotor="${mass_rotor}" radius_rotor="${radius_rotor}" time_constant_up="${time_constant_up}" time_constant_down="${time_constant_down}" max_rot_velocity="${max_rot_velocity}" motor_number="5" rotor_drag_coefficient="${rotor_drag_coefficient}" rolling_moment_coefficient="${rolling_moment_coefficient}" mesh="prop" mesh_scale="${mesh_scale_prop}" color="DarkGrey">
     <origin xyz="-0.23556 0.136 0.074" rpy="0 0 0" />
     <xacro:insert_block name="rotor_inertia" />
