Commit message: Add kinect plugin and test it

File: mbzirc_gazebo_simulation/uavs_description/models/mbzirc2020/component_snippets.xacro (robot description, xacro)
@@ -589,3 +589,258 @@
    </gazebo>
 </xacro:macro>
+<!-- KINECT -->
+<xacro:macro name='kinect_macro'
+  params="namespace parent_link camera_suffix">
+    <link name="${namespace}/kinect_${camera_suffix}_link">
+      <inertial>
+      <mass value="1e-5" />
+      <origin xyz="0 0 0" rpy="0 0 0"/>
+      <inertia ixx="1e-6" ixy="0" ixz="0" iyy="1e-6" iyz="0"      izz="1e-6" />
+    </inertial>
+      <self_collide>0</self_collide>
+      <enable_wind>0</enable_wind>
+      <kinematic>0</kinematic>
+      <pose frame=''>0 0 0 0 -0 0</pose>
+      <visual name='visual'>
+        <geometry>
+          <box size="0.01 0.01 0.01"/>
+          <!-- <mesh filename="package://uavs_description/models/mbzirc2020/meshes/kinect.dae" scale="0.01 0.01 0.01" /> -->
+          <!-- <mesh>
+            <uri>model://kinect/meshes/kinect.dae</uri>
+          </mesh> -->
+        </geometry>
+        <!-- <material>
+          <shader type='pixel'/>
+        </material> -->
+        <pose frame=''>0 0 0 0 -0 0</pose>
+        <transparency>0</transparency>
+        <cast_shadows>1</cast_shadows>
+      </visual>
+      <collision name='collision'>
+        <laser_retro>0</laser_retro>
+        <max_contacts>10</max_contacts>
+        <pose frame=''>0 0 0 0 -0 0</pose>
+        <geometry>
+           <box size="0.01 0.01 0.01"/>
+          <!-- <mesh filename="package://uavs_description/models/mbzirc2020/meshes/kinect.dae" scale="1 1 1" /> -->
+          <!-- <box>
+            <size>0.073 0.276 0.072</size>
+          </box> -->
+        </geometry>
+        <surface>
+          <friction>
+            <ode>
+              <mu>1</mu>
+              <mu2>1</mu2>
+              <fdir1>0 0 0</fdir1>
+              <slip1>0</slip1>
+              <slip2>0</slip2>
+            </ode>
+            <torsional>
+              <coefficient>1</coefficient>
+              <patch_radius>0</patch_radius>
+              <surface_radius>0</surface_radius>
+              <use_patch_radius>1</use_patch_radius>
+              <ode>
+                <slip>0</slip>
+              </ode>
+            </torsional>
+          </friction>
+          <bounce>
+            <restitution_coefficient>0</restitution_coefficient>
+            <threshold>1e+06</threshold>
+          </bounce>
+          <contact>
+            <collide_without_contact>0</collide_without_contact>
+            <collide_without_contact_bitmask>1</collide_without_contact_bitmask>
+            <collide_bitmask>1</collide_bitmask>
+            <ode>
+              <soft_cfm>0</soft_cfm>
+              <soft_erp>0.2</soft_erp>
+              <kp>1e+13</kp>
+              <kd>1</kd>
+              <max_vel>0.01</max_vel>
+              <min_depth>0</min_depth>
+            </ode>
+            <bullet>
+              <split_impulse>1</split_impulse>
+              <split_impulse_penetration_threshold>-0.01</split_impulse_penetration_threshold>
+              <soft_cfm>0</soft_cfm>
+              <soft_erp>0.2</soft_erp>
+              <kp>1e+13</kp>
+              <kd>1</kd>
+            </bullet>
+          </contact>
+        </surface>
+      </collision>
+    </link>
+    <static>0</static>
+    <allow_auto_disable>1</allow_auto_disable>
+    <joint name="${namespace}/kinect_${camera_suffix}_joint" type="fixed">
+      <axis xyz="0 1 0" />
+      <origin rpy="0 0 0" xyz="0.5 0 0" />
+      <parent link="${parent_link}"/>
+      <child link="${namespace}/kinect_${camera_suffix}_link"/>
+    </joint>
+    <gazebo reference="${namespace}/kinect_${camera_suffix}_link">
+      <sensor name='camera_kinect' type='depth'>
+          <update_rate>20</update_rate>
+          <camera name='__default__'>
+            <horizontal_fov>1.0472</horizontal_fov>
+            <image>
+              <width>8</width>
+              <height>8</height>
+              <format>R8G8B8</format>
+            </image>
+            <clip>
+              <near>0.1</near>
+              <far>5</far>
+            </clip>
+          </camera>
+          <plugin name='camera_plugin' filename='libgazebo_ros_openni_kinect.so'>
+            <baseline>0.2</baseline>
+            <alwaysOn>1</alwaysOn>
+            <updateRate>0.0</updateRate>
+            <cameraName>camera_kinect</cameraName>
+            <imageTopicName>/camera_kinect/depth/image_raw</imageTopicName>
+            <cameraInfoTopicName>/camera_kinect/depth/camera_info</cameraInfoTopicName>
+            <depthImageTopicName>/camera_kinect/depth/image_raw</depthImageTopicName>
+            <depthImageInfoTopicName>/camera_kinect/depth/camera_info</depthImageInfoTopicName>
+            <pointCloudTopicName>/camera_kinect/depth/points</pointCloudTopicName>
+            <frameName>uav_1</frameName>
+            <!-- <frameName>${namespace}/kinect_${camera_suffix}_link</frameName> -->
+            <pointCloudCutoff>0.05</pointCloudCutoff>
+            <distortionK1>0</distortionK1>
+            <distortionK2>0</distortionK2>
+            <distortionK3>0</distortionK3>
+            <distortionT1>0</distortionT1>
+            <distortionT2>0</distortionT2>
+            <CxPrime>0</CxPrime>
+            <Cx>0</Cx>
+            <Cy>0</Cy>
+            <focalLength>0</focalLength>
+            <hackBaseline>0</hackBaseline>
+          </plugin>
+        </sensor>
+      </gazebo>
+  </xacro:macro>
+<!-- MyraBot Kinect -->
+<xacro:macro name="kinect" params="parent_link *origin">
+  <joint name="base_camera_joint" type="fixed">
+	<xacro:insert_block name="origin" />
+    <parent link="${parent_link}" />
+    <child link="camera_link" />
+  </joint>
+  <link name="camera_link">
+    <inertial>
+      <mass value="0.01" />
+      <origin xyz="0 0 0" />
+      <inertia ixx="0.001" ixy="0.0" ixz="0.0"
+        iyy="0.001" iyz="0.0"
+        izz="0.001" />
+    </inertial>
+    <visual>
+      <origin xyz=" 0 0 0 " rpy="0 0 0" />
+      <geometry>
+        <box size="0.01 0.01 0.01"/>
+        <!-- <mesh filename="package://myrabot_fer_modelo/meshes/kinect.dae"/> -->
+      </geometry>
+    </visual>
+    <collision>
+      <origin xyz="0.0 0.0 0.0" rpy="0 0 0" />
+      <geometry>
+        <box size="0.01 0.01 0.01"/>
+        <!-- <mesh filename="package://myrabot_fer_modelo/meshes/kinect.dae"/> -->
+      </geometry>
+    </collision>
+  </link>
+  <joint name="camera_depth_joint" type="fixed">
+    <origin xyz="0 0.018 0" rpy="0 0 0" />
+    <parent link="camera_link" />
+    <child link="camera_depth_frame" />
+  </joint>
+  <link name="camera_depth_frame">
+    <inertial>
+      <mass value="0.01" />
+      <origin xyz="0 0 0" />
+      <inertia ixx="0.001" ixy="0.0" ixz="0.0"
+        iyy="0.001" iyz="0.0"
+        izz="0.001" />
+    </inertial>
+  </link>
+  <joint name="camera_depth_optical_joint" type="fixed">
+    <origin xyz="0 0 0" rpy="${-3.1416/2} 0 ${-3.1416/2}" />
+    <parent link="camera_depth_frame" />
+    <child link="camera_depth_optical_frame" />
+  </joint>
+  <link name="camera_depth_optical_frame">
+    <inertial>
+      <mass value="0.001" />
+      <origin xyz="0 0 0" />
+      <inertia ixx="0.0001" ixy="0.0" ixz="0.0"
+        iyy="0.0001" iyz="0.0"
+        izz="0.0001" />
+    </inertial>
+  </link>
+  <joint name="camera_rgb_joint" type="fixed">
+    <origin xyz="0 -0.005 0" rpy="0 0 0" />
+    <parent link="camera_link" />
+    <child link="camera_rgb_frame" />
+  </joint>
+  <link name="camera_rgb_frame">
+    <inertial>
+      <mass value="0.001" />
+      <origin xyz="0 0 0" />
+      <inertia ixx="0.0001" ixy="0.0" ixz="0.0"
+        iyy="0.0001" iyz="0.0"
+        izz="0.0001" />
+    </inertial>
+  </link>
+  <joint name="camera_rgb_optical_joint" type="fixed">
+    <origin xyz="0 0 0" rpy="${-3.1416/2} 0 ${-3.1416/2}" />
+    <parent link="camera_rgb_frame" />
+    <child link="camera_rgb_optical_frame" />
+  </joint>
+  <link name="camera_rgb_optical_frame">
+    <inertial>
+      <mass value="0.001" />
+      <origin xyz="0 0 0" />
+      <inertia ixx="0.0001" ixy="0.0" ixz="0.0"
+        iyy="0.0001" iyz="0.0"
+        izz="0.0001" />
+    </inertial>
+  </link>
+  <gazebo reference="camera_link">
+    <sensor name="camera" type="camera">
+      <update_rate>20</update_rate>
+      <camera name="myra">
+      <image>
+        <width>8</width>
+        <height>8</height>
+        <format>R8G8B8</format>
+      </image>
+      <horizontal_fov>1.0472</horizontal_fov>
+      <clip>
+        <near>0.05</near>
+        <far>5</far>
+      </clip>
+      </camera>
+      <plugin name="kinect_camera_controller" filename="libgazebo_ros_openni_kinect.so">
+        <baseline>0.1</baseline>
+        <alwaysOn>true</alwaysOn>
+        <updateRate>20</updateRate>
+        <robotNamespace>/</robotNamespace>
+        <imageTopicName>/camera/image_raw</imageTopicName>
+        <pointCloudTopicName>/camera/depth/points</pointCloudTopicName>
+        <cameraInfoTopicName>/camera/camera_info</cameraInfoTopicName>
+        <frameName>camera_depth_optical_frame</frameName>
+        <distortion_k1>0.0</distortion_k1>
+        <distortion_k2>0.0</distortion_k2>
+        <distortion_k3>0.0</distortion_k3>
+        <distortion_t1>0.0</distortion_t1>
+        <distortion_t2>0.0</distortion_t2>
+      </plugin>
+    </sensor>
+  </gazebo>
+</xacro:macro>
 </robot>

File: mbzirc_gazebo_simulation/uavs_description/models/mbzirc2020/geometry.xacro (robot description, xacro)
@@ -96,10 +96,22 @@
   </xacro:camera_macro>
 <!-- Installing Teraranger Evo frontal-->
-  <xacro:teraranger_macro
+  <!-- <xacro:teraranger_macro
     namespace="${model_name}"
     parent_link="base_link"
     teraranger_suffix="0"
   >
-  </xacro:teraranger_macro>
+  </xacro:teraranger_macro> -->
+<!-- Installing Kinect-->
+  <xacro:kinect_macro
+    namespace="${model_name}"
+    parent_link="base_link"
+    camera_suffix="0"
+  >
+  </xacro:kinect_macro>
+  <!-- Installing MyraBot Kinect -->
+  <xacro:kinect
+    parent_link="base_link">
+		<origin xyz="0.2 0.2 0.2" rpy="0 0 1.5" />
+	</xacro:kinect>
   <!-- Instantiate rotors -->
   <xacro:vertical_rotor

Commit message: Cleanup mbzirc2020 simulation model

File: mbzirc_gazebo_simulation/uavs_description/models/mbzirc2020/component_snippets.xacro (robot description, xacro)
@@ -46,5 +46,5 @@
       <xacro:if value="${enable_visual}">
         <visual>
-          <origin xyz="0 0 0" rpy="0 1.57079632679 0" />
+          <origin xyz="0 0 0" rpy="0 0 0" />
           <geometry>
             <xacro:insert_block name="cylinder" />

File: mbzirc_gazebo_simulation/uavs_description/models/mbzirc2020/geometry.xacro (robot description, xacro)
@@ -3,4 +3,5 @@
   <!-- Properties -->
   <xacro:property name="model_name" value="mbzirc2020" />
+  <xacro:property name="description_package" value="uavs_description" />
   <xacro:property name="namespace" value="" />
   <xacro:property name="rotor_velocity_slowdown_sim" value="10" />
@@ -37,13 +38,10 @@
     ixy="0.0" ixz="0.0"  iyz="0.0" /> <!-- [kg.m^2] [kg.m^2] [kg.m^2] [kg.m^2] [kg.m^2] [kg.m^2] -->
   </xacro:property>
-  <!--Property cylinder_camera-->
-  <xacro:property name="camera_cylinder">
-    <box size="0.1 0.025 0.02"/>
-  </xacro:property>
   <!-- Included URDF Files -->
-  <xacro:include filename="$(find uavs_description)/models/mbzirc2020/multirotor_base.xacro" />
-  <xacro:include filename="$(find uavs_description)/models/mbzirc2020/component_snippets.xacro" />
+  <xacro:include filename="$(find robots_description)/urdf/multirotor_base.xacro" />
+  <xacro:include filename="$(find robots_description)/urdf/component_snippets.xacro" />
   <!-- Instantiate multirotor_base_macro once -->
   <xacro:multirotor_base_macro
+    description_package="${description_package}"
     model_name="${model_name}"
     robot_namespace="${namespace}"
@@ -73,9 +71,9 @@
     enable_visual="true"
     >
-    <xacro:insert_block name="camera_cylinder"/>
-    <origin xyz="0 0.24 -0.24" rpy="0 1.57 0" />
+    <box size="0.01 0.01 0.01"/>
+    <origin xyz="0 0 -0.275" rpy="0 1.57079632679 0" />
   </xacro:camera_macro>
 <!-- Installing Camera 1 -->
-  <xacro:camera_macro
+  <!-- <xacro:camera_macro
     namespace="${namespace}"
     parent_link="base_link"
@@ -94,14 +92,15 @@
     <xacro:insert_block name="camera_cylinder"/>
     <origin xyz="0 0.24 -0.24" rpy="0 0 0" />
-  </xacro:camera_macro>
+  </xacro:camera_macro> -->
 <!-- Installing Teraranger Evo frontal-->
-  <xacro:teraranger_macro
+  <!-- <xacro:teraranger_macro
     namespace="${model_name}"
     parent_link="base_link"
     teraranger_suffix="0"
   >
-  </xacro:teraranger_macro>
+  </xacro:teraranger_macro> -->
   <!-- Instantiate rotors -->
   <xacro:vertical_rotor
+    description_package="${description_package}"
     robot_namespace="${namespace}"
     suffix="right"
@@ -125,4 +124,5 @@
   </xacro:vertical_rotor>
   <xacro:vertical_rotor
+    description_package="${description_package}"
     robot_namespace="${namespace}"
     suffix="left"
@@ -145,5 +145,7 @@
     <xacro:insert_block name="rotor_inertia" />
   </xacro:vertical_rotor>
-  <xacro:vertical_rotor robot_namespace="${namespace}"
+  <xacro:vertical_rotor
+    description_package="${description_package}"
+    robot_namespace="${namespace}"
     suffix="front_left"
     direction="cw"
@@ -165,5 +167,7 @@
     <xacro:insert_block name="rotor_inertia" />
   </xacro:vertical_rotor>
-  <xacro:vertical_rotor robot_namespace="${namespace}"
+  <xacro:vertical_rotor
+    description_package="${description_package}"
+    robot_namespace="${namespace}"
     suffix="back_right"
     direction="ccw"
@@ -185,5 +189,7 @@
     <xacro:insert_block name="rotor_inertia" />
   </xacro:vertical_rotor>
-  <xacro:vertical_rotor robot_namespace="${namespace}"
+  <xacro:vertical_rotor
+    description_package="${description_package}"
+    robot_namespace="${namespace}"
     suffix="front_right"
     direction="ccw"
@@ -205,5 +211,7 @@
     <xacro:insert_block name="rotor_inertia" />
   </xacro:vertical_rotor>
-  <xacro:vertical_rotor robot_namespace="${namespace}"
+  <xacro:vertical_rotor
+    description_package="${description_package}"
+    robot_namespace="${namespace}"
     suffix="back_left"
     direction="cw"

File: mbzirc_gazebo_simulation/uavs_description/models/mbzirc2020/model.xacro (robot description, xacro)
@@ -13,5 +13,5 @@
   <xacro:arg name='enable_logging' default='false' />
   <!-- macros for gazebo plugins, sensors -->
-  <xacro:include filename="$(find uavs_description)/models/mbzirc2020/component_snippets.xacro" />
+  <xacro:include filename="$(find robots_description)/urdf/component_snippets.xacro" />
   <!-- Instantiate mbzirc "mechanics" -->
   <xacro:include filename="$(find uavs_description)/models/mbzirc2020/geometry.xacro" />

Commit message: backup

File: mbzirc_gazebo_simulation/uavs_description/models/mbzirc2020/component_snippets.xacro (robot description, xacro)
@@ -702,11 +702,12 @@
             <alwaysOn>1</alwaysOn>
             <updateRate>0.0</updateRate>
+            <robotNamespace>${namespace}</robotNamespace>
             <cameraName>camera_kinect</cameraName>
-            <imageTopicName>/camera_kinect/depth/image_raw</imageTopicName>
-            <cameraInfoTopicName>/camera_kinect/depth/camera_info</cameraInfoTopicName>
-            <depthImageTopicName>/camera_kinect/depth/image_raw</depthImageTopicName>
-            <depthImageInfoTopicName>/camera_kinect/depth/camera_info</depthImageInfoTopicName>
-            <pointCloudTopicName>/camera_kinect/depth/points</pointCloudTopicName>
-            <frameName>uav_1</frameName>
+            <imageTopicName>camera_kinect/depth/image_raw</imageTopicName>
+            <cameraInfoTopicName>camera_kinect/depth/camera_info</cameraInfoTopicName>
+            <depthImageTopicName>camera_kinect/depth/depth_image_raw</depthImageTopicName>
+            <depthImageInfoTopicName>camera_kinect/depth/camera_info_depth</depthImageInfoTopicName>
+            <pointCloudTopicName>camera_kinect/depth/pointsCloud</pointCloudTopicName>
+            <frameName>/uav_1</frameName>
             <!-- <frameName>${namespace}/kinect_${camera_suffix}_link</frameName> -->
             <pointCloudCutoff>0.05</pointCloudCutoff>
@@ -830,5 +831,5 @@
         <alwaysOn>true</alwaysOn>
         <updateRate>20</updateRate>
-        <robotNamespace>/</robotNamespace>
+        <robotNamespace>${namespace}</robotNamespace>
         <imageTopicName>/camera/image_raw</imageTopicName>
         <pointCloudTopicName>/camera/depth/points</pointCloudTopicName>
@@ -844,3 +845,60 @@
   </gazebo>
 </xacro:macro>
+<!-- Installing Hokuyo-->
+<!-- Macro to add a laser Hokuyo. -->
+ <xacro:macro name="hokuyo" params="name namespace parent *origin ros_topic update_rate ray_count min_angle max_angle">
+   <link name="${namespace}_hokuyo_link">
+     <collision>
+       <origin xyz="0 0 0" rpy="0 0 0" />
+       <geometry>
+         <cylinder length="0.03" radius="0.015"/>
+       </geometry>
+     </collision>
+     <visual>
+       <origin xyz="0 0 0" rpy="0 0 0" />
+       <geometry>
+         <cylinder length="0.03" radius="0.015"/>
+         <!--mesh filename="package://home/agugrvc/catkin_ws/src/grvc-ual/ball_description/models/bola/meshes/hokuyo_utm_30lx.dae"/-->
+       </geometry>
+     </visual>
+     <inertial>
+       <mass value="1e-5" />
+       <origin xyz="0 0 0" rpy="0 0 0" />
+       <inertia ixx="1e-6" ixy="0" ixz="0" iyy="1e-6" iyz="0" izz="1e-6" />
+     </inertial>
+   </link>
+   <joint name="${namespace}_hokuyo_joint" type="fixed">
+     <xacro:insert_block name="origin" />
+     <parent link="${parent}" />
+     <child link="${namespace}_hokuyo_link" />
+   </joint>
+   <gazebo reference="${namespace}_hokuyo_link">
+     <sensor type="ray" name="laser">
+       <pose>0 0 0 0 0 0</pose>
+       <ray>
+         <scan>
+           <horizontal>
+             <samples>${ray_count}</samples>
+             <resolution>1</resolution>
+             <min_angle>${min_angle}</min_angle>
+             <max_angle>${max_angle}</max_angle>
+           </horizontal>
+         </scan>
+         <range>
+           <min>0.08</min>
+           <max>40</max>
+           <resolution>0.01</resolution>
+         </range>
+       </ray>
+           <plugin name="laser" filename="libgazebo_ros_laser.so">
+             <frameName>/hokuyo_frame</frameName>
+             <robotNamespace>${namespace}</robotNamespace>
+             <topicName>${ros_topic}</topicName>
+             <always_on>1</always_on>
+           <update_rate>${update_rate}</update_rate>
+           <visualize>true</visualize>
+       </plugin>
+     </sensor>
+   </gazebo>
+ </xacro:macro>
 </robot>

File: mbzirc_gazebo_simulation/uavs_description/models/mbzirc2020/geometry.xacro (robot description, xacro)
@@ -95,4 +95,16 @@
     <origin xyz="0 0.24 -0.24" rpy="0 0 0" />
   </xacro:camera_macro>
+<!--Installing Hokuyo-->
+  <xacro:hokuyo
+     name="laser0"
+     namespace="${namespace}"
+     parent="base_link"
+     ros_topic="hokuyo_laser"
+     update_rate="40"
+     ray_count="1080"
+     min_angle="-2.268899"
+     max_angle="2.268899">
+      <origin xyz="0 0 0.5" rpy="0 0 0.785"/>
+    </xacro:hokuyo>
 <!-- Installing Teraranger Evo frontal-->
   <!-- <xacro:teraranger_macro
