Commit message: Add laser scan sensor to challenge 3 uav

File: mbzirc_gazebo_simulation/uavs_description/models/mbzirc2020/model.xacro (robot description, xacro)
@@ -19,10 +19,10 @@
   <xacro:include filename="$(find uavs_description)/models/mbzirc2020/geometry.xacro" />
   <xacro:if value="${$(arg challenge) == 2}">
-    <!-- Installing magnetic gripper -->
+    <!-- Install magnetic gripper -->
     <xacro:include filename="$(find mbzirc_gazebo_plugins)/urdf/magnetic_gripper.xacro" />
     <xacro:magnetic_gripper parent="base_link" robot_name="mbzirc2020_$(arg robot_id)">
       <origin xyz="0 0 -0.275" rpy="0 0 0" />
     </xacro:magnetic_gripper>
-    <!-- Installing Camera 0 -->
+    <!-- Install camera facing down -->
     <xacro:camera_macro
       namespace="${namespace}"
@@ -44,35 +44,78 @@
     </xacro:camera_macro>
   </xacro:if>
-<!-- Installing Camera 1 -->
-  <!-- <xacro:camera_macro
-    namespace="${namespace}"
-    parent_link="base_link"
-    camera_suffix="1"
-    frame_rate="10"
-    horizontal_fov="1.07079633"
-    image_width="800"
-    image_height="600"
-    image_format="R8G8B8"
-    min_distance="0.01"
-    max_distance="100"
-    noise_mean="0"
-    noise_stddev="0"
-    enable_visual="true"
-    >
-    <xacro:insert_block name="camera_cylinder"/>
-    <origin xyz="0 0.24 -0.24" rpy="0 0 0" />
-  </xacro:camera_macro> -->
-<!-- Installing Teraranger Evo frontal-->
+<!-- Install Teraranger Evo frontal -->
   <!-- <xacro:teraranger_macro
     namespace="${model_name}"
     parent_link="base_link"
-    teraranger_suffix="0"
-  >
+    teraranger_suffix="0">
   </xacro:teraranger_macro> -->
-  <xacro:include filename="$(find mbzirc_gazebo_plugins)/urdf/fake_camera.xacro" />
   <xacro:if value="${$(arg challenge) == 3}">
+    <!-- Install fake camera for fire detection -->
+    <xacro:include filename="$(find mbzirc_gazebo_plugins)/urdf/fake_camera.xacro" />
     <xacro:fake_camera parent="base_link" robot_name="mbzirc2020_$(arg robot_id)">
       <origin xyz="0.5 0 -0.27" rpy="0 1.57 0" />
     </xacro:fake_camera>
+    <!-- Install laser scanner TODO: Move to snippets? -->
+    <joint name="laser_joint" type="fixed">
+      <axis xyz="0 1 0" />
+      <origin xyz="0 0 0.1" rpy="0 0 0"/>
+      <parent link="base_link"/>
+      <child link="laser_link"/>
+    </joint>
+    <link name="laser_link">
+      <collision>
+        <origin xyz="0 0 0" rpy="0 0 0"/>
+        <geometry>
+          <cylinder length="0.03" radius="0.04" />
+        </geometry>
+      </collision>
+      <visual>
+        <origin xyz="0 0 0" rpy="0 0 0"/>
+        <geometry>
+          <cylinder length="0.03" radius="0.04" />
+        </geometry>
+      </visual>
+      <inertial>
+        <mass value="1e-5" />
+        <origin xyz="0 0 0" rpy="0 0 0"/>
+        <inertia ixx="1e-6" ixy="0" ixz="0" iyy="1e-6" iyz="0" izz="1e-6" />
+      </inertial>
+    </link>
+    <gazebo reference="laser_link">
+      <sensor type="gpu_ray" name="laser_sensor">
+        <pose>0 0 0 0 0 0</pose>
+        <visualize>false</visualize>
+        <update_rate>40</update_rate>
+        <ray>
+          <scan>
+            <horizontal>
+              <samples>720</samples>
+              <resolution>1</resolution>
+              <min_angle>-1.570796</min_angle>
+              <max_angle>1.570796</max_angle>
+            </horizontal>
+          </scan>
+          <range>
+            <min>0.10</min>
+            <max>30.0</max>
+            <resolution>0.01</resolution>
+          </range>
+          <noise>
+            <type>gaussian</type>
+            <!-- Noise parameters based on published spec for Hokuyo laser
+                achieving "+-30mm" accuracy at range < 10m.  A mean of 0.0m and
+                stddev of 0.01m will put 99.7% of samples within 0.03m of the true
+                reading. -->
+            <mean>0.0</mean>
+            <stddev>0.01</stddev>
+          </noise>
+        </ray>
+        <plugin name="${namespace}_laser_controller" filename="libgazebo_ros_gpu_laser.so">
+          <robotNamespace>${namespace}</robotNamespace>
+          <topicName>scan</topicName>
+          <frameName>laser_link</frameName>
+        </plugin>
+      </sensor>
+    </gazebo>
   </xacro:if>
   <xacro:if value="$(arg enable_gps_plugin)">

Commit message: Adding depth camera c3

File: mbzirc_gazebo_simulation/uavs_description/models/mbzirc2020/model.xacro (robot description, xacro)
@@ -56,8 +56,142 @@
       <origin xyz="0.5 0 -0.27" rpy="0 1.57 0" />
     </xacro:fake_camera>
+<!-- KINECT -->
+    <link name="kinect_link">
+      <inertial>
+      <mass value="1e-5" />
+      <origin xyz="0 0 0" rpy="0 0 0"/>
+      <inertia ixx="1e-6" ixy="0" ixz="0" iyy="1e-6" iyz="0"      izz="1e-6" />
+    </inertial>
+      <self_collide>0</self_collide>
+      <enable_wind>0</enable_wind>
+      <kinematic>0</kinematic>
+      <pose frame=''>0 0 0 0 -0 0</pose>
+      <visual name='visual'>
+        <geometry>
+          <box size="0.01 0.01 0.01"/>
+          <!-- <mesh filename="package://uavs_description/models/mbzirc2020/meshes/kinect.dae" scale="0.01 0.01 0.01" /> -->
+          <!-- <mesh>
+            <uri>model://kinect/meshes/kinect.dae</uri>
+          </mesh> -->
+        </geometry>
+        <!-- <material>
+          <shader type='pixel'/>
+        </material> -->
+        <pose frame=''>0 0 0 0 -0 0</pose>
+        <transparency>0</transparency>
+        <cast_shadows>1</cast_shadows>
+      </visual>
+      <collision name='collision'>
+        <laser_retro>0</laser_retro>
+        <max_contacts>10</max_contacts>
+        <pose frame=''>0 0 0 0 -0 0</pose>
+        <geometry>
+           <box size="0.01 0.01 0.01"/>
+          <!-- <mesh filename="package://uavs_description/models/mbzirc2020/meshes/kinect.dae" scale="1 1 1" /> -->
+          <!-- <box>
+            <size>0.073 0.276 0.072</size>
+          </box> -->
+        </geometry>
+        <surface>
+          <friction>
+            <ode>
+              <mu>1</mu>
+              <mu2>1</mu2>
+              <fdir1>0 0 0</fdir1>
+              <slip1>0</slip1>
+              <slip2>0</slip2>
+            </ode>
+            <torsional>
+              <coefficient>1</coefficient>
+              <patch_radius>0</patch_radius>
+              <surface_radius>0</surface_radius>
+              <use_patch_radius>1</use_patch_radius>
+              <ode>
+                <slip>0</slip>
+              </ode>
+            </torsional>
+          </friction>
+          <bounce>
+            <restitution_coefficient>0</restitution_coefficient>
+            <threshold>1e+06</threshold>
+          </bounce>
+          <contact>
+            <collide_without_contact>0</collide_without_contact>
+            <collide_without_contact_bitmask>1</collide_without_contact_bitmask>
+            <collide_bitmask>1</collide_bitmask>
+            <ode>
+              <soft_cfm>0</soft_cfm>
+              <soft_erp>0.2</soft_erp>
+              <kp>1e+13</kp>
+              <kd>1</kd>
+              <max_vel>0.01</max_vel>
+              <min_depth>0</min_depth>
+            </ode>
+            <bullet>
+              <split_impulse>1</split_impulse>
+              <split_impulse_penetration_threshold>-0.01</split_impulse_penetration_threshold>
+              <soft_cfm>0</soft_cfm>
+              <soft_erp>0.2</soft_erp>
+              <kp>1e+13</kp>
+              <kd>1</kd>
+            </bullet>
+          </contact>
+        </surface>
+      </collision>
+    </link>
+    <static>0</static>
+    <allow_auto_disable>1</allow_auto_disable>
+    <joint name="kinect_joint" type="fixed">
+      <axis xyz="0 1 0" />
+      <origin rpy="0 0 0" xyz="0.5 0 0" />
+      <parent link="base_link"/>
+      <child link="kinect_link"/>
+    </joint>
+    <gazebo reference="kinect_link">
+      <sensor name='camera_kinect' type='depth'>
+          <update_rate>20</update_rate>
+          <camera name='__default__'>
+            <horizontal_fov>1.0472</horizontal_fov>
+            <image>
+              <width>1800</width>
+              <height>720</height>
+              <format>R8G8B8</format>
+            </image>
+            <clip>
+              <near>0.5</near>
+              <far>15</far>
+            </clip>
+          </camera>
+          <plugin name='camera_plugin' filename='libgazebo_ros_openni_kinect.so'>
+            <baseline>0.2</baseline>
+            <alwaysOn>1</alwaysOn>
+            <updateRate>0.0</updateRate>
+            <robotNamespace>${namespace}</robotNamespace>
+            <cameraName>camera_kinect</cameraName>
+            <imageTopicName>depth/image_raw</imageTopicName>
+            <cameraInfoTopicName>depth/camera_info</cameraInfoTopicName>
+            <depthImageTopicName>depth/depth_image_raw</depthImageTopicName>
+            <depthImageInfoTopicName>depth/camera_info_depth</depthImageInfoTopicName>
+            <pointCloudTopicName>depth/pointsCloud</pointCloudTopicName>
+            <frameName>/uav_1</frameName>
+            <!-- <frameName>${namespace}/kinect_${camera_suffix}_link</frameName> -->
+            <pointCloudCutoff>0.05</pointCloudCutoff>
+            <distortionK1>0</distortionK1>
+            <distortionK2>0</distortionK2>
+            <distortionK3>0</distortionK3>
+            <distortionT1>0</distortionT1>
+            <distortionT2>0</distortionT2>
+            <CxPrime>0</CxPrime>
+            <Cx>0</Cx>
+            <Cy>0</Cy>
+            <focalLength>0</focalLength>
+            <hackBaseline>0</hackBaseline>
+          </plugin>
+        </sensor>
+      </gazebo>
     <!-- Install laser scanner TODO: Move to snippets? -->
     <joint name="laser_joint" type="fixed">
-      <axis xyz="0 1 0" />
-      <origin xyz="0 0 0.1" rpy="0 0 0"/>
+      <axis xyz="0 0 0" />
+      <origin xyz="0 0 0.4" rpy="0 0 0"/>
       <parent link="base_link"/>
       <child link="laser_link"/>
@@ -65,5 +199,5 @@
     <link name="laser_link">
       <collision>
-        <origin xyz="0 0 0" rpy="0 0 0"/>
+        <origin xyz="0 0 0.4" rpy="0 0 0"/>
         <geometry>
           <cylinder length="0.03" radius="0.04" />
@@ -83,5 +217,5 @@
     </link>
     <gazebo reference="laser_link">
-      <sensor type="gpu_ray" name="laser_sensor">
+      <sensor type="ray" name="laser_sensor">
         <pose>0 0 0 0 0 0</pose>
         <visualize>false</visualize>
@@ -111,5 +245,5 @@
           </noise>
         </ray>
-        <plugin name="${namespace}_laser_controller" filename="libgazebo_ros_gpu_laser.so">
+        <plugin name="${namespace}_laser_controller" filename="libgazebo_ros_laser.so">
           <robotNamespace>${namespace}</robotNamespace>
           <topicName>scan</topicName>

Commit message: fixing UAV sensor position

File: mbzirc_gazebo_simulation/uavs_description/models/mbzirc2020/model.xacro (robot description, xacro)
@@ -50,9 +50,10 @@
     teraranger_suffix="0">
   </xacro:teraranger_macro> -->
+<!-- WATER C3 UAV -->
   <xacro:if value="${$(arg challenge) == 3}">
     <!-- Install fake camera for fire detection -->
     <xacro:include filename="$(find mbzirc_gazebo_plugins)/urdf/fake_camera.xacro" />
     <xacro:fake_camera parent="base_link" robot_name="mbzirc2020_$(arg robot_id)">
-      <origin xyz="0.5 0 -0.27" rpy="0 1.57 0" />
+      <origin xyz="0.25 0 -0.11" rpy="0 0 0" />
     </xacro:fake_camera>
     <!-- KINECT -->
@@ -144,5 +145,5 @@
     <joint name="kinect_joint" type="fixed">
       <axis xyz="0 1 0" />
-      <origin rpy="0 0 0" xyz="0.5 0 0" />
+      <origin rpy="0 0 0" xyz="0.23 0 -0.06" />
       <parent link="base_link"/>
       <child link="kinect_link"/>
@@ -206,5 +207,5 @@
       visualize="false"
       >
-      <origin xyz="0 0 0.05" rpy="0 0 0" />
+      <origin xyz="-0.19 0 0.17" rpy="0 0 0" />
     </xacro:laser_scanner>
     <!-- Install laser scanner: altimeter -->
@@ -224,5 +225,183 @@
       visualize="true"
       >
-      <origin xyz="-0.45 0 0.05" rpy="0 1.57 0" />
+      <origin xyz="-0.28 0.28 -0.05" rpy="0 1.57 0" />
+    </xacro:laser_scanner>
+  </xacro:if>
+<!-- BLANKET C3 UAV -->
+<xacro:if value="${$(arg challenge) == 3b}">
+    <!-- Install fake camera for fire detection -->
+    <xacro:include filename="$(find mbzirc_gazebo_plugins)/urdf/fake_camera.xacro" />
+    <xacro:fake_camera parent="base_link" robot_name="mbzirc2020_$(arg robot_id)">
+      <origin xyz="0.25 0 -0.11" rpy="0 1.57 0" />
+    </xacro:fake_camera>
+    <!-- KINECT -->
+    <link name="kinect_link">
+      <inertial>
+        <mass value="1e-5" />
+        <origin xyz="0 0 0" rpy="0 0 0"/>
+        <inertia ixx="1e-6" ixy="0" ixz="0" iyy="1e-6" iyz="0" izz="1e-6"/>
+      </inertial>
+      <self_collide>0</self_collide>
+      <enable_wind>0</enable_wind>
+      <kinematic>0</kinematic>
+      <pose frame=''>0 0 0 0 -0 0</pose>
+      <visual name='visual'>
+        <geometry>
+          <box size="0.01 0.01 0.01"/>
+          <!-- <mesh filename="package://uavs_description/models/mbzirc2020/meshes/kinect.dae" scale="0.01 0.01 0.01" /> -->
+          <!-- <mesh>
+            <uri>model://kinect/meshes/kinect.dae</uri>
+          </mesh> -->
+        </geometry>
+        <!-- <material>
+          <shader type='pixel'/>
+        </material> -->
+        <pose frame=''>0 0 0 0 -0 0</pose>
+        <transparency>0</transparency>
+        <cast_shadows>1</cast_shadows>
+      </visual>
+      <collision name='collision'>
+        <laser_retro>0</laser_retro>
+        <max_contacts>10</max_contacts>
+        <pose frame=''>0 0 0 0 -0 0</pose>
+        <geometry>
+           <box size="0.01 0.01 0.01"/>
+          <!-- <mesh filename="package://uavs_description/models/mbzirc2020/meshes/kinect.dae" scale="1 1 1" /> -->
+          <!-- <box>
+            <size>0.073 0.276 0.072</size>
+          </box> -->
+        </geometry>
+        <surface>
+          <friction>
+            <ode>
+              <mu>1</mu>
+              <mu2>1</mu2>
+              <fdir1>0 0 0</fdir1>
+              <slip1>0</slip1>
+              <slip2>0</slip2>
+            </ode>
+            <torsional>
+              <coefficient>1</coefficient>
+              <patch_radius>0</patch_radius>
+              <surface_radius>0</surface_radius>
+              <use_patch_radius>1</use_patch_radius>
+              <ode>
+                <slip>0</slip>
+              </ode>
+            </torsional>
+          </friction>
+          <bounce>
+            <restitution_coefficient>0</restitution_coefficient>
+            <threshold>1e+06</threshold>
+          </bounce>
+          <contact>
+            <collide_without_contact>0</collide_without_contact>
+            <collide_without_contact_bitmask>1</collide_without_contact_bitmask>
+            <collide_bitmask>1</collide_bitmask>
+            <ode>
+              <soft_cfm>0</soft_cfm>
+              <soft_erp>0.2</soft_erp>
+              <kp>1e+13</kp>
+              <kd>1</kd>
+              <max_vel>0.01</max_vel>
+              <min_depth>0</min_depth>
+            </ode>
+            <bullet>
+              <split_impulse>1</split_impulse>
+              <split_impulse_penetration_threshold>-0.01</split_impulse_penetration_threshold>
+              <soft_cfm>0</soft_cfm>
+              <soft_erp>0.2</soft_erp>
+              <kp>1e+13</kp>
+              <kd>1</kd>
+            </bullet>
+          </contact>
+        </surface>
+      </collision>
+    </link>
+    <static>0</static>
+    <allow_auto_disable>1</allow_auto_disable>
+    <joint name="kinect_joint" type="fixed">
+      <axis xyz="0 1 0" />
+      <origin rpy="0 0 0" xyz="0.23 0 -0.06" />
+      <parent link="base_link"/>
+      <child link="kinect_link"/>
+    </joint>
+    <gazebo reference="kinect_link">
+      <sensor name='camera_kinect' type='depth'>
+        <update_rate>20</update_rate>
+        <camera name='__default__'>
+          <horizontal_fov>1.0472</horizontal_fov>
+          <image>
+            <width>1280</width>
+            <height>720</height>
+            <format>R8G8B8</format>
+          </image>
+          <clip>
+            <near>0.5</near>
+            <far>15</far>
+          </clip>
+        </camera>
+        <plugin name='camera_plugin' filename='libgazebo_ros_openni_kinect.so'>
+          <baseline>0.2</baseline>
+          <alwaysOn>1</alwaysOn>
+          <updateRate>0.0</updateRate>
+          <robotNamespace>${namespace}</robotNamespace>
+          <cameraName>camera_kinect</cameraName>
+          <imageTopicName>depth/image_raw</imageTopicName>
+          <cameraInfoTopicName>depth/camera_info</cameraInfoTopicName>
+          <depthImageTopicName>depth/depth_image_raw</depthImageTopicName>
+          <depthImageInfoTopicName>depth/camera_info_depth</depthImageInfoTopicName>
+          <pointCloudTopicName>depth/pointsCloud</pointCloudTopicName>
+          <frameName>/uav_1</frameName>
+          <!-- <frameName>${namespace}/kinect_${camera_suffix}_link</frameName> -->
+          <pointCloudCutoff>0.05</pointCloudCutoff>
+          <distortionK1>0</distortionK1>
+          <distortionK2>0</distortionK2>
+          <distortionK3>0</distortionK3>
+          <distortionT1>0</distortionT1>
+          <distortionT2>0</distortionT2>
+          <CxPrime>0</CxPrime>
+          <Cx>0</Cx>
+          <Cy>0</Cy>
+          <focalLength>0</focalLength>
+          <hackBaseline>0</hackBaseline>
+        </plugin>
+      </sensor>
+    </gazebo>
+    <!-- Install laser scanner: rplidar -->
+    <xacro:laser_scanner
+      namespace="${namespace}"
+      id="0"
+      pub_topic="scan"
+      tf="laser_link"
+      parent_link="base_link"
+      update_rate="40"
+      sample_count="720"
+      angle_min="-1.570796"
+      angle_max="1.570796"
+      range_min="0.10"
+      range_max="30.0"
+      range_res="0.01"
+      visualize="false"
+      >
+      <origin xyz="-0.19 0 0.17" rpy="0 0 0" />
+    </xacro:laser_scanner>
+    <!-- Install laser scanner: altimeter -->
+    <xacro:laser_scanner
+      namespace="${namespace}"
+      id="1"
+      pub_topic="sf11_sim_as_scan"
+      tf="sf11_link"
+      parent_link="base_link"
+      update_rate="20"
+      sample_count="1"
+      angle_min="0"
+      angle_max="0"
+      range_min="0.10"
+      range_max="120.0"
+      range_res="0.01"
+      visualize="true"
+      >
+      <origin xyz="-0.28 0.28 -0.05" rpy="0 1.57 0" />
     </xacro:laser_scanner>
   </xacro:if>

Commit message: Test to pick with new tracking

File: mbzirc_gazebo_simulation/uavs_description/models/mbzirc2020/model.xacro (robot description, xacro)
@@ -22,5 +22,5 @@
     <xacro:include filename="$(find mbzirc_gazebo_plugins)/urdf/magnetic_gripper.xacro" />
     <xacro:magnetic_gripper parent="base_link" robot_name="mbzirc2020_$(arg robot_id)">
-      <origin xyz="0 0 -0.275" rpy="0 0 0" />
+      <origin xyz="0 0 -0.3" rpy="0 0 0" />
     </xacro:magnetic_gripper>
     <!-- Install camera facing down -->
@@ -41,6 +41,24 @@
       >
       <box size="0.01 0.01 0.01"/>
-      <origin xyz="0 0 -0.295" rpy="0 1.57079632679 0" />
+      <origin xyz="0.25 0 0.05" rpy="0 1.57079632679 0" />
     </xacro:camera_macro>
+    <!-- Install laser scanner: altimeter -->
+    <xacro:laser_scanner
+      namespace="${namespace}"
+      id="1"
+      pub_topic="sf11_sim_as_scan"
+      tf="sf11_link"
+      parent_link="base_link"
+      update_rate="20"
+      sample_count="1"
+      angle_min="0"
+      angle_max="0"
+      range_min="0.10"
+      range_max="120.0"
+      range_res="0.01"
+      visualize="true"
+      >
+      <origin xyz="-0.28 0.28 -0.05" rpy="0 1.57 0" />
+    </xacro:laser_scanner>
   </xacro:if>
 <!-- Install Teraranger Evo frontal -->

Commit message: Move and rotate camera

File: mbzirc_gazebo_simulation/uavs_description/models/mbzirc2020/model.xacro (robot description, xacro)
@@ -41,5 +41,5 @@
       >
       <box size="0.01 0.01 0.01"/>
-      <origin xyz="0.25 0 0.05" rpy="0 1.57079632679 0" />
+      <origin xyz="0.17 0 -0.16" rpy="0 1.57079632679 3.141592" />
     </xacro:camera_macro>
     <!-- Install laser scanner: altimeter -->

Commit message: Test to align to wall with rplidar

File: mbzirc_gazebo_simulation/uavs_description/models/mbzirc2020/model.xacro (robot description, xacro)
@@ -43,4 +43,22 @@
       <origin xyz="0.17 0 -0.16" rpy="0 1.57079632679 3.141592" />
     </xacro:camera_macro>
+    <!-- Install laser scanner: rplidar -->
+    <xacro:laser_scanner
+      namespace="${namespace}"
+      id="0"
+      pub_topic="scan"
+      tf="laser_link"
+      parent_link="base_link"
+      update_rate="40"
+      sample_count="720"
+      angle_min="-1.570796"
+      angle_max="1.570796"
+      range_min="0.10"
+      range_max="30.0"
+      range_res="0.01"
+      visualize="false"
+      >
+      <origin xyz="-0.19 0 0.17" rpy="0 0 0" />
+    </xacro:laser_scanner>
     <!-- Install laser scanner: altimeter -->
     <xacro:laser_scanner
