Commit message: replacing normal camera for kinect type in ch2

File: mbzirc_gazebo_simulation/uavs_description/models/mbzirc2020/model.xacro (robot description, xacro)
@@ -25,5 +25,5 @@
     </xacro:magnetic_gripper>
     <!-- Install camera facing down -->
-    <xacro:camera_macro
+    <!-- <xacro:camera_macro
       namespace="${namespace}"
       parent_link="base_link"
@@ -42,5 +42,141 @@
       <box size="0.01 0.01 0.01"/>
       <origin xyz="0.17 0 -0.16" rpy="0 1.57079632679 3.141592" />
-    </xacro:camera_macro>
+    </xacro:camera_macro> -->
+    <!-- KINECT -->
+    <link name="kinect_link">
+      <inertial>
+        <mass value="1e-5" />
+        <origin xyz="0 0 0" rpy="0 0 0"/>
+        <inertia ixx="1e-6" ixy="0" ixz="0" iyy="1e-6" iyz="0" izz="1e-6"/>
+      </inertial>
+      <self_collide>0</self_collide>
+      <enable_wind>0</enable_wind>
+      <kinematic>0</kinematic>
+      <pose frame=''>0 0 0 0 -0 0</pose>
+      <visual name='visual'>
+        <geometry>
+          <box size="0.01 0.01 0.01"/>
+          <!-- <mesh filename="package://uavs_description/models/mbzirc2020/meshes/kinect.dae" scale="0.01 0.01 0.01" /> -->
+          <!-- <mesh>
+            <uri>model://kinect/meshes/kinect.dae</uri>
+          </mesh> -->
+        </geometry>
+        <!-- <material>
+          <shader type='pixel'/>
+        </material> -->
+        <pose frame=''>0 0 0 0 -0 0</pose>
+        <transparency>0</transparency>
+        <cast_shadows>1</cast_shadows>
+      </visual>
+      <collision name='collision'>
+        <laser_retro>0</laser_retro>
+        <max_contacts>10</max_contacts>
+        <pose frame=''>0 0 0 0 -0 0</pose>
+        <geometry>
+           <box size="0.01 0.01 0.01"/>
+          <!-- <mesh filename="package://uavs_description/models/mbzirc2020/meshes/kinect.dae" scale="1 1 1" /> -->
+          <!-- <box>
+            <size>0.073 0.276 0.072</size>
+          </box> -->
+        </geometry>
+        <surface>
+          <friction>
+            <ode>
+              <mu>1</mu>
+              <mu2>1</mu2>
+              <fdir1>0 0 0</fdir1>
+              <slip1>0</slip1>
+              <slip2>0</slip2>
+            </ode>
+            <torsional>
+              <coefficient>1</coefficient>
+              <patch_radius>0</patch_radius>
+              <surface_radius>0</surface_radius>
+              <use_patch_radius>1</use_patch_radius>
+              <ode>
+                <slip>0</slip>
+              </ode>
+            </torsional>
+          </friction>
+          <bounce>
+            <restitution_coefficient>0</restitution_coefficient>
+            <threshold>1e+06</threshold>
+          </bounce>
+          <contact>
+            <collide_without_contact>0</collide_without_contact>
+            <collide_without_contact_bitmask>1</collide_without_contact_bitmask>
+            <collide_bitmask>1</collide_bitmask>
+            <ode>
+              <soft_cfm>0</soft_cfm>
+              <soft_erp>0.2</soft_erp>
+              <kp>1e+13</kp>
+              <kd>1</kd>
+              <max_vel>0.01</max_vel>
+              <min_depth>0</min_depth>
+            </ode>
+            <bullet>
+              <split_impulse>1</split_impulse>
+              <split_impulse_penetration_threshold>-0.01</split_impulse_penetration_threshold>
+              <soft_cfm>0</soft_cfm>
+              <soft_erp>0.2</soft_erp>
+              <kp>1e+13</kp>
+              <kd>1</kd>
+            </bullet>
+          </contact>
+        </surface>
+      </collision>
+    </link>
+    <static>0</static>
+    <allow_auto_disable>1</allow_auto_disable>
+    <joint name="kinect_joint" type="fixed">
+      <axis xyz="0 1 0" />
+      <origin rpy="0 1.57079632679 3.141592" xyz="0.17 0 -0.16" />
+      <parent link="base_link"/>
+      <child link="kinect_link"/>
+    </joint>
+    <gazebo reference="kinect_link">
+      <sensor name='camera_kinect' type='depth'>
+        <update_rate>20</update_rate>
+        <camera name='__default__'>
+          <horizontal_fov>1.0472</horizontal_fov>
+          <image>
+            <width>1280</width>
+            <height>720</height>
+            <format>R8G8B8</format>
+          </image>
+          <clip>
+            <near>0.5</near>
+            <far>15</far>
+          </clip>
+        </camera>
+        <plugin name='camera_plugin' filename='libgazebo_ros_openni_kinect.so'>
+          <baseline>0.2</baseline>
+          <alwaysOn>1</alwaysOn>
+          <updateRate>0.0</updateRate>
+          <robotNamespace>${namespace}</robotNamespace>
+          <cameraName>camera</cameraName>
+          <imageTopicName>color/image_rect_color</imageTopicName>
+          <!-- <cameraInfoTopicName>color/camera_info</cameraInfoTopicName> -->
+          <cameraInfoTopicName>aligned_depth_to_color/camera_info</cameraInfoTopicName>
+          <depthImageTopicName>aligned_depth_to_color/image_raw</depthImageTopicName>
+          <!-- <depthImageInfoTopicName>aligned_depth_to_color/camera_info</depthImageInfoTopicName> -->
+          <depthImageInfoTopicName>dummy/camera_info</depthImageInfoTopicName>
+          <pointCloudTopicName>depth/pointsCloud</pointCloudTopicName>
+          <frameName>camera_color_optical_frame</frameName>
+          <!-- <frameName>${namespace}/kinect_${camera_suffix}_link</frameName> -->
+          <pointCloudCutoff>0.05</pointCloudCutoff>
+          <distortionK1>0</distortionK1>
+          <distortionK2>0</distortionK2>
+          <distortionK3>0</distortionK3>
+          <distortionT1>0</distortionT1>
+          <distortionT2>0</distortionT2>
+          <CxPrime>0</CxPrime>
+          <Cx>0</Cx>
+          <Cy>0</Cy>
+          <focalLength>0</focalLength>
+          <hackBaseline>0</hackBaseline>
+        </plugin>
+      </sensor>
+    </gazebo>
     <!-- Install laser scanner: rplidar -->
     <xacro:laser_scanner

Commit message: Change sim model to fix take off issue

File: mbzirc_gazebo_simulation/uavs_description/models/mbzirc2020/model.xacro (robot description, xacro)
@@ -22,5 +22,5 @@
     <xacro:include filename="$(find mbzirc_gazebo_plugins)/urdf/magnetic_gripper.xacro" />
     <xacro:magnetic_gripper parent="base_link" robot_name="mbzirc2020_$(arg robot_id)">
-      <origin xyz="0 0 -0.3" rpy="0 0 0" />
+      <origin xyz="0 0 -0.275" rpy="0 0 0" />
     </xacro:magnetic_gripper>
     <!-- Install camera facing down -->

Commit message: fixing c31 uav model kinect orientation

File: mbzirc_gazebo_simulation/uavs_description/models/mbzirc2020/model.xacro (robot description, xacro)
@@ -496,5 +496,5 @@
     <joint name="kinect_joint" type="fixed">
       <axis xyz="0 1 0" />
-      <origin rpy="0 0 0" xyz="0.23 0 -0.06" />
+      <origin rpy="0 1.57 0" xyz="0.23 0 -0.06" />
       <parent link="base_link"/>
       <child link="kinect_link"/>
@@ -521,10 +521,12 @@
           <robotNamespace>${namespace}</robotNamespace>
           <cameraName>camera</cameraName>
-          <imageTopicName>color/image_rect_color</imageTopicName>
-          <cameraInfoTopicName>color/camera_info</cameraInfoTopicName>
-          <depthImageTopicName>depth/depth_image_raw</depthImageTopicName>
-          <depthImageInfoTopicName>depth/camera_info</depthImageInfoTopicName>
+          <imageTopicName>color/image_raw</imageTopicName>
+          <!-- <cameraInfoTopicName>color/camera_info</cameraInfoTopicName> -->
+          <cameraInfoTopicName>aligned_depth_to_color/camera_info</cameraInfoTopicName>
+          <depthImageTopicName>aligned_depth_to_color/image_raw</depthImageTopicName>
+          <!-- <depthImageInfoTopicName>aligned_depth_to_color/camera_info</depthImageInfoTopicName> -->
+          <depthImageInfoTopicName>dummy/camera_info</depthImageInfoTopicName>
           <pointCloudTopicName>depth/pointsCloud</pointCloudTopicName>
-          <frameName>/uav_1</frameName>
+          <frameName>camera_color_optical_frame</frameName>
           <!-- <frameName>${namespace}/kinect_${camera_suffix}_link</frameName> -->
           <pointCloudCutoff>0.05</pointCloudCutoff>
@@ -539,4 +541,21 @@
           <focalLength>0</focalLength>
           <hackBaseline>0</hackBaseline>
+          <!-- <imageTopicName>color/image_rect_color</imageTopicName>
+          <cameraInfoTopicName>color/camera_info</cameraInfoTopicName>
+          <depthImageTopicName>depth/depth_image_raw</depthImageTopicName>
+          <depthImageInfoTopicName>depth/camera_info</depthImageInfoTopicName>
+          <pointCloudTopicName>depth/pointsCloud</pointCloudTopicName>
+          <frameName>/uav_1</frameName>
+          <pointCloudCutoff>0.05</pointCloudCutoff>
+          <distortionK1>0</distortionK1>
+          <distortionK2>0</distortionK2>
+          <distortionK3>0</distortionK3>
+          <distortionT1>0</distortionT1>
+          <distortionT2>0</distortionT2>
+          <CxPrime>0</CxPrime>
+          <Cx>0</Cx>
+          <Cy>0</Cy>
+          <focalLength>0</focalLength>
+          <hackBaseline>0</hackBaseline> -->
         </plugin>
       </sensor>
