Commit message: Update gazebo simulation to include magnetic gripper

File: mbzirc_gazebo_simulation/uavs_description/models/mbzirc2020/geometry.xacro (robot description, xacro)
@@ -72,5 +72,5 @@
     >
     <box size="0.01 0.01 0.01"/>
-    <origin xyz="0 0 -0.275" rpy="0 1.57079632679 0" />
+    <origin xyz="0 0 -0.295" rpy="0 1.57079632679 0" />
   </xacro:camera_macro>
 <!-- Installing Camera 1 -->

File: mbzirc_gazebo_simulation/uavs_description/models/mbzirc2020/model.xacro (robot description, xacro)
@@ -4,4 +4,5 @@
   Is there a reason not to make all properties arguments?
   -->
+  <xacro:arg name='robot_id' default='1' />
   <xacro:arg name='mavlink_addr' default='INADDR_ANY' />
   <xacro:arg name='mavlink_udp_port' default='14560' />
@@ -16,4 +17,8 @@
   <!-- Instantiate mbzirc "mechanics" -->
   <xacro:include filename="$(find uavs_description)/models/mbzirc2020/geometry.xacro" />
+  <xacro:include filename="$(find mbzirc_gazebo_plugins)/urdf/magnetic_gripper.xacro" />
+  <xacro:magnetic_gripper parent="base_link" robot_name="mbzirc2020_$(arg robot_id)">
+    <origin xyz="0 0 -0.275" rpy="0 0 0" />
+  </xacro:magnetic_gripper>
   <xacro:if value="$(arg enable_gps_plugin)">
     <!-- Instantiate gps plugin. -->

Commit message: Use laser snippet and add simulated altimeter

File: mbzirc_gazebo_simulation/uavs_description/models/mbzirc2020/geometry.xacro (robot description, xacro)
@@ -11,5 +11,6 @@
   <xacro:property name="mass" value="5.850" /> <!-- [kg] -->
   <xacro:property name="body_width" value="0.8" /> <!-- [m] -->
-  <xacro:property name="body_height" value="0.6" /> <!-- [m] -->
+  <xacro:property name="body_height" value="0.3" /> <!-- [m] -->
+  <xacro:property name="height_offset" value="-0.15" /> <!-- [m] -->
   <xacro:property name="mass_rotor" value="0.005" /> <!-- [kg] -->
   <xacro:property name="rotor_offset_top" value="0.0" /> <!-- [m] -->
@@ -48,4 +49,5 @@
     body_width="${body_width}"
     body_height="${body_height}"
+    height_offset="${height_offset}"
     mesh_file="${mesh_file}"
     mesh_scale="${mesh_scale}"

File: mbzirc_gazebo_simulation/uavs_description/models/mbzirc2020/model.xacro (robot description, xacro)
@@ -56,11 +56,11 @@
       <origin xyz="0.5 0 -0.27" rpy="0 1.57 0" />
     </xacro:fake_camera>
-<!-- KINECT -->
+    <!-- KINECT -->
     <link name="kinect_link">
       <inertial>
-      <mass value="1e-5" />
-      <origin xyz="0 0 0" rpy="0 0 0"/>
-      <inertia ixx="1e-6" ixy="0" ixz="0" iyy="1e-6" iyz="0"      izz="1e-6" />
-    </inertial>
+        <mass value="1e-5" />
+        <origin xyz="0 0 0" rpy="0 0 0"/>
+        <inertia ixx="1e-6" ixy="0" ixz="0" iyy="1e-6" iyz="0" izz="1e-6"/>
+      </inertial>
       <self_collide>0</self_collide>
       <enable_wind>0</enable_wind>
@@ -150,106 +150,76 @@
     <gazebo reference="kinect_link">
       <sensor name='camera_kinect' type='depth'>
-          <update_rate>20</update_rate>
-          <camera name='__default__'>
-            <horizontal_fov>1.0472</horizontal_fov>
-            <image>
-              <width>1800</width>
-              <height>720</height>
-              <format>R8G8B8</format>
-            </image>
-            <clip>
-              <near>0.5</near>
-              <far>15</far>
-            </clip>
-          </camera>
-          <plugin name='camera_plugin' filename='libgazebo_ros_openni_kinect.so'>
-            <baseline>0.2</baseline>
-            <alwaysOn>1</alwaysOn>
-            <updateRate>0.0</updateRate>
-            <robotNamespace>${namespace}</robotNamespace>
-            <cameraName>camera_kinect</cameraName>
-            <imageTopicName>depth/image_raw</imageTopicName>
-            <cameraInfoTopicName>depth/camera_info</cameraInfoTopicName>
-            <depthImageTopicName>depth/depth_image_raw</depthImageTopicName>
-            <depthImageInfoTopicName>depth/camera_info_depth</depthImageInfoTopicName>
-            <pointCloudTopicName>depth/pointsCloud</pointCloudTopicName>
-            <frameName>/uav_1</frameName>
-            <!-- <frameName>${namespace}/kinect_${camera_suffix}_link</frameName> -->
-            <pointCloudCutoff>0.05</pointCloudCutoff>
-            <distortionK1>0</distortionK1>
-            <distortionK2>0</distortionK2>
-            <distortionK3>0</distortionK3>
-            <distortionT1>0</distortionT1>
-            <distortionT2>0</distortionT2>
-            <CxPrime>0</CxPrime>
-            <Cx>0</Cx>
-            <Cy>0</Cy>
-            <focalLength>0</focalLength>
-            <hackBaseline>0</hackBaseline>
-          </plugin>
-        </sensor>
-      </gazebo>
-    <!-- Install laser scanner TODO: Move to snippets? -->
-    <joint name="laser_joint" type="fixed">
-      <axis xyz="0 0 0" />
-      <origin xyz="0 0 0.4" rpy="0 0 0"/>
-      <parent link="base_link"/>
-      <child link="laser_link"/>
-    </joint>
-    <link name="laser_link">
-      <collision>
-        <origin xyz="0 0 0.4" rpy="0 0 0"/>
-        <geometry>
-          <cylinder length="0.03" radius="0.04" />
-        </geometry>
-      </collision>
-      <visual>
-        <origin xyz="0 0 0" rpy="0 0 0"/>
-        <geometry>
-          <cylinder length="0.03" radius="0.04" />
-        </geometry>
-      </visual>
-      <inertial>
-        <mass value="1e-5" />
-        <origin xyz="0 0 0" rpy="0 0 0"/>
-        <inertia ixx="1e-6" ixy="0" ixz="0" iyy="1e-6" iyz="0" izz="1e-6" />
-      </inertial>
-    </link>
-    <gazebo reference="laser_link">
-      <sensor type="ray" name="laser_sensor">
-        <pose>0 0 0 0 0 0</pose>
-        <visualize>false</visualize>
-        <update_rate>40</update_rate>
-        <ray>
-          <scan>
-            <horizontal>
-              <samples>720</samples>
-              <resolution>1</resolution>
-              <min_angle>-1.570796</min_angle>
-              <max_angle>1.570796</max_angle>
-            </horizontal>
-          </scan>
-          <range>
-            <min>0.10</min>
-            <max>30.0</max>
-            <resolution>0.01</resolution>
-          </range>
-          <noise>
-            <type>gaussian</type>
-            <!-- Noise parameters based on published spec for Hokuyo laser
-                achieving "+-30mm" accuracy at range < 10m.  A mean of 0.0m and
-                stddev of 0.01m will put 99.7% of samples within 0.03m of the true
-                reading. -->
-            <mean>0.0</mean>
-            <stddev>0.01</stddev>
-          </noise>
-        </ray>
-        <plugin name="${namespace}_laser_controller" filename="libgazebo_ros_laser.so">
+        <update_rate>20</update_rate>
+        <camera name='__default__'>
+          <horizontal_fov>1.0472</horizontal_fov>
+          <image>
+            <width>1800</width>
+            <height>720</height>
+            <format>R8G8B8</format>
+          </image>
+          <clip>
+            <near>0.5</near>
+            <far>15</far>
+          </clip>
+        </camera>
+        <plugin name='camera_plugin' filename='libgazebo_ros_openni_kinect.so'>
+          <baseline>0.2</baseline>
+          <alwaysOn>1</alwaysOn>
+          <updateRate>0.0</updateRate>
           <robotNamespace>${namespace}</robotNamespace>
-          <topicName>scan</topicName>
-          <frameName>laser_link</frameName>
+          <cameraName>camera_kinect</cameraName>
+          <imageTopicName>depth/image_raw</imageTopicName>
+          <cameraInfoTopicName>depth/camera_info</cameraInfoTopicName>
+          <depthImageTopicName>depth/depth_image_raw</depthImageTopicName>
+          <depthImageInfoTopicName>depth/camera_info_depth</depthImageInfoTopicName>
+          <pointCloudTopicName>depth/pointsCloud</pointCloudTopicName>
+          <frameName>/uav_1</frameName>
+          <!-- <frameName>${namespace}/kinect_${camera_suffix}_link</frameName> -->
+          <pointCloudCutoff>0.05</pointCloudCutoff>
+          <distortionK1>0</distortionK1>
+          <distortionK2>0</distortionK2>
+          <distortionK3>0</distortionK3>
+          <distortionT1>0</distortionT1>
+          <distortionT2>0</distortionT2>
+          <CxPrime>0</CxPrime>
+          <Cx>0</Cx>
+          <Cy>0</Cy>
+          <focalLength>0</focalLength>
+          <hackBaseline>0</hackBaseline>
         </plugin>
       </sensor>
     </gazebo>
+    <!-- Install laser scanner: rplidar -->
+    <xacro:laser_scanner
+      namespace="${namespace}"
+      id="0"
+      parent_link="base_link"
+      update_rate="40"
+      sample_count="720"
+      angle_min="-1.570796"
+      angle_max="1.570796"
+      range_min="0.10"
+      range_max="30.0"
+      range_res="0.01"
+      visualize="false"
+      >
+      <origin xyz="0 0 0.05" rpy="0 0 0" />
+    </xacro:laser_scanner>
+    <!-- Install laser scanner: altimeter -->
+    <xacro:laser_scanner
+      namespace="${namespace}"
+      id="1"
+      parent_link="base_link"
+      update_rate="20"
+      sample_count="1"
+      angle_min="0"
+      angle_max="0"
+      range_min="0.10"
+      range_max="120.0"
+      range_res="0.01"
+      visualize="true"
+      >
+      <origin xyz="-0.45 0 0.05" rpy="0 1.57 0" />
+    </xacro:laser_scanner>
   </xacro:if>
   <xacro:if value="$(arg enable_gps_plugin)">

Commit message: Fix self-or-brick altimeter detection

File: mbzirc_gazebo_simulation/uavs_description/models/mbzirc2020/geometry.xacro (robot description, xacro)
@@ -10,5 +10,5 @@
   <xacro:property name="mesh_scale_prop" value=".001 .001 .001"/>
   <xacro:property name="mass" value="5.850" /> <!-- [kg] -->
-  <xacro:property name="body_width" value="0.8" /> <!-- [m] -->
+  <xacro:property name="body_width" value="0.6" /> <!-- [m] -->
   <xacro:property name="body_height" value="0.3" /> <!-- [m] -->
   <xacro:property name="height_offset" value="-0.15" /> <!-- [m] -->
