Commit message: pcl segmentations + laser brick detection + pan joint limit + realsense calib

File: realsense/realsense2_camera/urdf/_d435.urdf.xacro (robot description, xacro)
@@ -32,5 +32,5 @@
     <joint name="camera_joint" type="fixed">
       <!-- <xacro:insert_block name="origin" /> -->
-      <origin xyz="0 -0.03 0.15" rpy="0 -0.1 1.57"/>
+      <origin xyz="-0.035 0.04 0.20" rpy="0 -0.23 1.57"/>
 <!--       pus a camara mais abaixo do que a realidade para nao afetar o costmap -->
       <parent link="${parent}"/>

File: universal_robot-ur_e_fix/ur_e_description/urdf/ur5e.urdf.xacro (robot description, xacro)
@@ -103,10 +103,11 @@
       <axis xyz="0 0 1" />
       <xacro:unless value="${joint_limited}">
-        <limit lower="${-2.0 * pi}" upper="${2.0 * pi}" effort="150.0" velocity="3.14"/>
-      </xacro:unless>
-      <xacro:if value="${joint_limited}">
-        <limit lower="${shoulder_pan_lower_limit}" upper="${shoulder_pan_upper_limit}" effort="150.0" velocity="3.14"/>
-      </xacro:if>
-      <dynamics damping="0.0" friction="0.0"/>
+        <limit lower="-3" upper="0.1" effort="150.0" velocity="3.14"/>
+      </xacro:unless>
+      <xacro:if value="${joint_limited}">
+        <limit lower="-3" upper="0.1" effort="150.0" velocity="3.14"/>
+      </xacro:if>
+      <dynamics damping="0.0" friction="0.0"/>
+      <safety_controller k_position="100" k_velocity="1.5" soft_lower_limit="-3" soft_upper_limit="0.1"/>    <!-- check what are these k_position and k_velocity -->
     </joint>
     <link name="${prefix}shoulder_link">
