Commit message: UGV+UAVs sim working with gotoaction, pickupaction, better arm controller, footprint modified

File: universal_robot-ur_e_fix/ur_e_description/urdf/ur5e.urdf.xacro (robot description, xacro)
@@ -320,4 +320,10 @@
     </joint>
     <link name="${prefix}ee_link">
+      <visual>
+        <geometry>
+          <box size="0.06 0.13 0.06"/>
+        </geometry>
+        <origin rpy="0 0 0" xyz="0 0 0"/>
+      </visual>
       <collision>
         <geometry>
