Commit message: adding xacro for generating c3 world

File: mbzirc_gazebo_simulation/challenge_worlds/worlds/challenge3.world.xacro (robot description, xacro)
@@ -1,12 +1,19 @@
 <?xml version="1.0" ?>
-<!-- =================================================================================== -->
-<!-- |    This document was autogenerated by xacro from challenge3.world.xacro         | -->
-<!-- |    EDITING THIS FILE BY HAND IS NOT RECOMMENDED                                 | -->
-<!-- =================================================================================== -->
 <sdf version="1.4" xmlns:xacro="http://www.ros.org/wiki/xacro">
-  <env name="GAZEBO_RESOURCE_PATH" value="/home/alex/catkin_ws/src/mbzirc2020/mbzirc_gazebo_simulation/challenge_worlds"/>
-  <!-- The following is the geometric expresion for an axis rotation -->
-  <!-- X'= X*cos(yaw)-Y*sin(yaw) -->
-  <!-- Y'= X*sin(yaw)+Y*cos(yaw)  -->
+    <env name="GAZEBO_RESOURCE_PATH" value="$(find challenge_worlds)" />
+<!-- Global yaw: to change the global position of all the objects in the world -->
+<xacro:property name="yaw" value="0.0"/>
+<!-- Properties for every object in the world -->
+ <!-- 0 => X position , 1 => Y position , 2 => Z position , 3 => Item yaw -->
+<xacro:property name="f1" value="${[15,27,0,0]}"/>
+<xacro:property name="f2" value="${[33,16,0,0]}"/>
+<xacro:property name="f3" value="${[32,50,0,0]}"/>
+<xacro:property name="f4" value="${[26,31,0,0]}"/>
+<xacro:property name="f5" value="${[25,31,15,0]}"/>
+<xacro:property name="b" value="${[25,30,0,0]}"/>
+<xacro:property name="g" value="${[25,30,0,0]}"/>
+   <!-- The following is the geometric expresion for an axis rotation -->
+   <!-- X'= X*cos(yaw)-Y*sin(yaw) -->
+   <!-- Y'= X*sin(yaw)+Y*cos(yaw)  -->
   <world name="default">
     <model name="ground_plane_asfalt">
@@ -14,5 +21,5 @@
         <uri>model://ground_plane_asfalt</uri>
       </include>
-      <pose frame="">25.0 30.0 0 0 0 0.0 </pose>
+      <pose frame=''>${g[0]*cos(yaw)-g[1]*sin(yaw)} ${g[0]*sin(yaw)+g[1]*cos(yaw)} ${g[2]} 0 0 ${g[3]+yaw} </pose>
     </model>
     <model name="cubewithflames_1">
@@ -20,11 +27,11 @@
         <uri>model://cubewithflames</uri>
       </include>
-      <pose frame="">15.0 27.0 0 0 0 0.0 </pose>
+      <pose frame=''>${f1[0]*cos(yaw)-f1[1]*sin(yaw)} ${f1[0]*sin(yaw)+f1[1]*cos(yaw)} ${f1[2]} 0 0 ${f1[3]+yaw} </pose>
     </model>
     <model name="cubewithflames_2">
       <include>
-        <uri>model://cubewithflames</uri>
+      <uri>model://cubewithflames</uri>
       </include>
-      <pose frame="">33.0 16.0 0 0 0 0.0 </pose>
+      <pose frame=''>${f2[0]*cos(yaw)-f2[1]*sin(yaw)} ${f2[0]*sin(yaw)+f2[1]*cos(yaw)} ${f2[2]} 0 0 ${f2[3]+yaw} </pose>
     </model>
     <model name="cubewithflames_3">
@@ -32,5 +39,5 @@
         <uri>model://cubewithflames</uri>
       </include>
-      <pose frame="">32.0 50.0 0 0 0 0.0 </pose>
+      <pose frame=''>${f3[0]*cos(yaw)-f3[1]*sin(yaw)} ${f3[0]*sin(yaw)+f3[1]*cos(yaw)} ${f3[2]} 0 0 ${f3[3]+yaw} </pose>
     </model>
     <model name="cubewithflames_4">
@@ -38,5 +45,5 @@
         <uri>model://cubewithflames</uri>
       </include>
-      <pose frame="">26.0 31.0 0 0 0 0.0 </pose>
+      <pose frame=''>${f4[0]*cos(yaw)-f4[1]*sin(yaw)} ${f4[0]*sin(yaw)+f4[1]*cos(yaw)} ${f4[2]} 0 0 ${f4[3]+yaw} </pose>
     </model>
     <model name="cubewithflames_5">
@@ -44,5 +51,5 @@
         <uri>model://cubewithflames</uri>
       </include>
-      <pose frame="">25.0 31.0 15 0 0 0.0 </pose>
+      <pose frame=''>${f5[0]*cos(yaw)-f5[1]*sin(yaw)} ${f5[0]*sin(yaw)+f5[1]*cos(yaw)} ${f5[2]} 0 0 ${f5[3]+yaw} </pose>
     </model>
     <model name="building">
@@ -50,9 +57,9 @@
         <uri>model://BuildingC3</uri>
       </include>
-      <pose frame="">25.0 30.0 0 0 0 0.0 </pose>
+      <pose frame=''>${b[0]*cos(yaw)-b[1]*sin(yaw)} ${b[0]*sin(yaw)+b[1]*cos(yaw)} ${b[2]} 0 0 ${b[3]+yaw} </pose>
     </model>
-    <light name="sun" type="directional">
+    <light name='sun' type='directional'>
       <cast_shadows>1</cast_shadows>
-      <pose frame="">0 0 10 0 -0 0</pose>
+      <pose frame=''>0 0 10 0 -0 0</pose>
       <diffuse>0.8 0.8 0.8 1</diffuse>
       <specular>0.1 0.1 0.1 1</specular>
@@ -65,7 +72,7 @@
       <direction>-0.5 0.5 -1</direction>
     </light>
-    <gui fullscreen="0">
-      <camera name="user_camera">
-        <pose frame="">-4.01588 -6.89701 14.3505 -0 0.40453 0.863487</pose>
+    <gui fullscreen='0'>
+      <camera name='user_camera'>
+        <pose frame=''>-4.01588 -6.89701 14.3505 -0 0.40453 0.863487</pose>
         <view_controller>orbit</view_controller>
         <projection_type>perspective</projection_type>
@@ -74,9 +81,9 @@
     <gravity>0 0 -9.8</gravity>
     <magnetic_field>6e-06 2.3e-05 -4.2e-05</magnetic_field>
-    <atmosphere type="adiabatic"/>
+    <atmosphere type='adiabatic'/>
     <wind>
       <linear_velocity>0.1 0.1 0</linear_velocity>
     </wind>
-    <physics default="0" name="default_physics" type="ode">
+    <physics name='default_physics' default='0' type='ode'>
       <max_step_size>0.004</max_step_size>
       <real_time_factor>1</real_time_factor>
@@ -101,5 +108,5 @@
       <heading_deg>0</heading_deg>
     </spherical_coordinates>
-    <plugin filename="libWindPlugin.so" name="wind">
+    <plugin name='wind' filename='libWindPlugin.so'>
       <horizontal>
         <magnitude>
@@ -109,5 +116,5 @@
             <period>60</period>
           </sin>
-          <noise type="gaussian">
+          <noise type='gaussian'>
             <mean>0</mean>
             <stddev>0.0002</stddev>
@@ -120,5 +127,5 @@
             <period>20</period>
           </sin>
-          <noise type="gaussian">
+          <noise type='gaussian'>
             <mean>0</mean>
             <stddev>0.03</stddev>
@@ -127,5 +134,5 @@
       </horizontal>
       <vertical>
-        <noise type="gaussian">
+        <noise type='gaussian'>
           <mean>0</mean>
           <stddev>0.03</stddev>
@@ -133,4 +140,4 @@
       </vertical>
     </plugin>
-  </world>
+   </world>
 </sdf>

Commit message: adding arena_yaw as argument in C3

File: mbzirc_gazebo_simulation/challenge_worlds/worlds/challenge3.world.xacro (robot description, xacro)
@@ -1,16 +1,16 @@
 <?xml version="1.0" ?>
 <sdf version="1.4" xmlns:xacro="http://www.ros.org/wiki/xacro">
-    <env name="GAZEBO_RESOURCE_PATH" value="$(find challenge_worlds)" />
 <!-- Global yaw: to change the global position of all the objects in the world -->
-<xacro:property name="yaw" value="0.0"/>
+<xacro:arg name="arena_yaw" default="0"/>
+<xacro:property name="yaw" value="$(arg arena_yaw)"/>
 <!-- Properties for every object in the world -->
  <!-- 0 => X position , 1 => Y position , 2 => Z position , 3 => Item yaw -->
-<xacro:property name="f1" value="${[15,27,0,0]}"/>
-<xacro:property name="f2" value="${[33,16,0,0]}"/>
-<xacro:property name="f3" value="${[32,50,0,0]}"/>
-<xacro:property name="f4" value="${[26,31,0,0]}"/>
-<xacro:property name="f5" value="${[25,31,15,0]}"/>
-<xacro:property name="b" value="${[25,30,0,0]}"/>
-<xacro:property name="g" value="${[25,30,0,0]}"/>
+<xacro:property name="f1" value="${[15,27,0,1.570795]}"/>
+<xacro:property name="f2" value="${[33,16,0,1.570795]}"/>
+<xacro:property name="f3" value="${[32,45,0,1.570795]}"/>
+<xacro:property name="f4" value="${[31,25,0,1.570795]}"/>
+<xacro:property name="f5" value="${[31,25,15,1.570795]}"/>
+<xacro:property name="b" value="${[30,25,0,3.14159]}"/>
+<xacro:property name="g" value="${[30,25,0,0]}"/>
    <!-- The following is the geometric expresion for an axis rotation -->
    <!-- X'= X*cos(yaw)-Y*sin(yaw) -->

Commit message: Adding new building and fires in CH3 world

File: mbzirc_gazebo_simulation/challenge_worlds/worlds/challenge3.world.xacro (robot description, xacro)
@@ -7,9 +7,9 @@
  <!-- 0 => X position , 1 => Y position , 2 => Z position , 3 => Item yaw -->
 <xacro:property name="f1" value="${[15,27,0,1.570795]}"/>
-<xacro:property name="f2" value="${[33,16,0,1.570795]}"/>
+<xacro:property name="f2" value="${[36,17,0,0]}"/>
 <xacro:property name="f3" value="${[32,45,0,1.570795]}"/>
-<xacro:property name="f4" value="${[31,25,0,1.570795]}"/>
-<xacro:property name="f5" value="${[31,25,15,1.570795]}"/>
-<xacro:property name="b" value="${[30,25,0,3.14159]}"/>
+<xacro:property name="f4" value="${[43,22,0,0]}"/>
+<xacro:property name="f5" value="${[33,22,10.5,1.570795]}"/>
+<xacro:property name="b" value="${[30,25,0,4.7124]}"/>
 <xacro:property name="g" value="${[30,25,0,0]}"/>
    <!-- The following is the geometric expresion for an axis rotation -->

Commit message: Add vertical fire holder model in c3 simulation

File: mbzirc_gazebo_simulation/challenge_worlds/worlds/challenge3.world.xacro (robot description, xacro)
@@ -9,5 +9,5 @@
 <xacro:property name="f2" value="${[36,17,0,0]}"/>
 <xacro:property name="f3" value="${[32,45,0,1.570795]}"/>
-<xacro:property name="f4" value="${[43,22,0,0]}"/>
+<xacro:property name="f4a" value="${[35, 15, 2, 0]}"/>
 <xacro:property name="f5" value="${[33,22,10.5,1.570795]}"/>
 <xacro:property name="b" value="${[30,25,0,4.7124]}"/>
@@ -41,9 +41,10 @@
       <pose frame=''>${f3[0]*cos(yaw)-f3[1]*sin(yaw)} ${f3[0]*sin(yaw)+f3[1]*cos(yaw)} ${f3[2]} 0 0 ${f3[3]+yaw} </pose>
     </model>
-    <model name="cubewithflames_4">
+    <model name="f4a">
       <include>
-        <uri>model://cubewithflames</uri>
+        <uri>model://vertical_fire_holder</uri>
       </include>
-      <pose frame=''>${f4[0]*cos(yaw)-f4[1]*sin(yaw)} ${f4[0]*sin(yaw)+f4[1]*cos(yaw)} ${f4[2]} 0 0 ${f4[3]+yaw} </pose>
+      <pose frame=''>${f4a[0]*cos(yaw)-f4a[1]*sin(yaw)} ${f4a[0]*sin(yaw)+f4a[1]*cos(yaw)} ${f4a[2]} 0 0 ${f4a[3]+yaw} </pose>
+      <static>true</static>
     </model>
     <model name="cubewithflames_5">

Commit message: fixing non-axis rotation in C3 world

File: mbzirc_gazebo_simulation/challenge_worlds/worlds/challenge3.world.xacro (robot description, xacro)
@@ -7,25 +7,39 @@
 <!-- Properties for every object in the world -->
  <!-- 0 => X position , 1 => Y position , 2 => Z position , 3 => Item yaw -->
-<xacro:property name="f1" value="${[15,27,0,1.570795]}"/>
+<!-- <xacro:property name="f1" value="${[15,27,0,1.570795]}"/>
 <xacro:property name="f2" value="${[36,17,0,0]}"/>
 <xacro:property name="f3" value="${[32,45,0,1.570795]}"/>
-<xacro:property name="f5" value="${[33,22,10.5,1.570795]}"/>
-<xacro:property name="f4a" value="${[37.5,25,5.3, 3.1416]}"/>
-<xacro:property name="f4b" value="${[36, 15, 5.3, 0]}"/>
-<xacro:property name="f4c" value="${[30, 20.5, 5.3, -1.570795]}"/>
-<xacro:property name="f4d" value="${[40, 20.3, 5.5, 1.570795]}"/>
-<xacro:property name="f4e" value="${[41.3, 25, 2, 3.1416]}"/>
-<xacro:property name="f5a" value="${[35, 25, 7.5, 3.1416]}"/>
-<xacro:property name="f5b" value="${[38.7, 15, 8.25, 0]}"/>
-<xacro:property name="f5c" value="${[30, 23, 9.2, -1.570795]}"/>
-<xacro:property name="f5d" value="${[40, 23.5, 9.2, 1.570795]}"/>
-<xacro:property name="f6a" value="${[36.5, 25, 10.3, 3.1416]}"/>
-<xacro:property name="f6b" value="${[31.3, 15, 11.25, 0]}"/>
-<xacro:property name="f6c" value="${[30, 16.3, 12, -1.570795]}"/>
-<xacro:property name="f6d" value="${[40, 16.3, 12.5, 1.570795]}"/>
+<xacro:property name="f5" value="${[33,22,10.5,1.570795]}"/> -->
+<xacro:property name="f4ap" value="${[b[0]+0,b[1]+7.5,b[2]+5.3, -1.57]}"/>
+<xacro:property name="f4a" value="${[(f4ap[0]-b[0])*cos(b[3])-(f4ap[1]-b[1])*sin(b[3])+b[0],(f4ap[0]-b[0])*sin(b[3])+(f4ap[1]-b[1])*cos(b[3])+b[1],f4ap[2],f4ap[3]+b[3]]}"/>
+<xacro:property name="f4bp" value="${[b[0]+10, b[1]+6, b[2]+5.3, 1.57]}"/>
+<xacro:property name="f4b" value="${[(f4bp[0]-b[0])*cos(b[3])-(f4bp[1]-b[1])*sin(b[3])+b[0],(f4bp[0]-b[0])*sin(b[3])+(f4bp[1]-b[1])*cos(b[3])+b[1],f4bp[2],f4bp[3]+b[3]]}"/>
+<xacro:property name="f4cp" value="${[b[0]+4.5, b[1]+0, b[2]+5.3, 0]}"/>
+<xacro:property name="f4c" value="${[(f4cp[0]-b[0])*cos(b[3])-(f4cp[1]-b[1])*sin(b[3])+b[0],(f4cp[0]-b[0])*sin(b[3])+(f4cp[1]-b[1])*cos(b[3])+b[1],f4cp[2],f4cp[3]+b[3]]}"/>
+<xacro:property name="f4dp" value="${[b[0]+4.7, b[1]+10, b[2]+5.5, -3.1416]}"/>
+<xacro:property name="f4d" value="${[(f4dp[0]-b[0])*cos(b[3])-(f4dp[1]-b[1])*sin(b[3])+b[0],(f4dp[0]-b[0])*sin(b[3])+(f4dp[1]-b[1])*cos(b[3])+b[1],f4dp[2],f4dp[3]+b[3]]}"/>
+<xacro:property name="f4ep" value="${[b[0]+0, b[1]+11.3, b[2]+2, -1.57]}"/>
+<xacro:property name="f4e" value="${[(f4ep[0]-b[0])*cos(b[3])-(f4ep[1]-b[1])*sin(b[3])+b[0],(f4ep[0]-b[0])*sin(b[3])+(f4ep[1]-b[1])*cos(b[3])+b[1],f4ep[2],f4ep[3]+b[3]]}"/>
+<xacro:property name="f5ap" value="${[b[0]+0, b[1]+5, b[2]+7.5, -1.57]}"/>
+<xacro:property name="f5a" value="${[(f5ap[0]-b[0])*cos(b[3])-(f5ap[1]-b[1])*sin(b[3])+b[0],(f5ap[0]-b[0])*sin(b[3])+(f5ap[1]-b[1])*cos(b[3])+b[1],f5ap[2],f5ap[3]+b[3]]}"/>
+<xacro:property name="f5bp" value="${[b[0]+10, b[1]+8.7, b[2]+8.25, 1.57]}"/>
+<xacro:property name="f5b" value="${[(f5bp[0]-b[0])*cos(b[3])-(f5bp[1]-b[1])*sin(b[3])+b[0],(f5bp[0]-b[0])*sin(b[3])+(f5bp[1]-b[1])*cos(b[3])+b[1],f5bp[2],f5bp[3]+b[3]]}"/>
+<xacro:property name="f5cp" value="${[b[0]+2, b[1]+0, b[2]+9.2, 0]}"/>
+<xacro:property name="f5c" value="${[(f5cp[0]-b[0])*cos(b[3])-(f5cp[1]-b[1])*sin(b[3])+b[0],(f5cp[0]-b[0])*sin(b[3])+(f5cp[1]-b[1])*cos(b[3])+b[1],f5cp[2],f5cp[3]+b[3]]}"/>
+<xacro:property name="f5dp" value="${[b[0]+1.5, b[1]+10, b[2]+9.2, 3.1416]}"/>
+<xacro:property name="f5d" value="${[(f5dp[0]-b[0])*cos(b[3])-(f5dp[1]-b[1])*sin(b[3])+b[0],(f5dp[0]-b[0])*sin(b[3])+(f5dp[1]-b[1])*cos(b[3])+b[1],f5dp[2],f5dp[3]+b[3]]}"/>
+<xacro:property name="f6ap" value="${[b[0]+0, b[1]+6.5, b[2]+10.3, -1.57]}"/>
+<xacro:property name="f6a" value="${[(f6ap[0]-b[0])*cos(b[3])-(f6ap[1]-b[1])*sin(b[3])+b[0],(f6ap[0]-b[0])*sin(b[3])+(f6ap[1]-b[1])*cos(b[3])+b[1],f6ap[2],f6ap[3]+b[3]]}"/>
+<xacro:property name="f6bp" value="${[b[0]+10, b[1]+1.3, b[2]+11.25, 1.57]}"/>
+<xacro:property name="f6b" value="${[(f6bp[0]-b[0])*cos(b[3])-(f6bp[1]-b[1])*sin(b[3])+b[0],(f6bp[0]-b[0])*sin(b[3])+(f6bp[1]-b[1])*cos(b[3])+b[1],f6bp[2],f6bp[3]+b[3]]}"/>
+<xacro:property name="f6cp" value="${[b[0]+8.7, b[1]+0, b[2]+12, 0]}"/>
+<xacro:property name="f6c" value="${[(f6cp[0]-b[0])*cos(b[3])-(f6cp[1]-b[1])*sin(b[3])+b[0],(f6cp[0]-b[0])*sin(b[3])+(f6cp[1]-b[1])*cos(b[3])+b[1],f6cp[2],f6cp[3]+b[3]]}"/>
+<xacro:property name="f6dp" value="${[b[0]+8.7, b[1]+10, b[2]+12.5, 3.1416]}"/>
+<xacro:property name="f6d" value="${[(f6dp[0]-b[0])*cos(b[3])-(f6dp[1]-b[1])*sin(b[3])+b[0],(f6dp[0]-b[0])*sin(b[3])+(f6dp[1]-b[1])*cos(b[3])+b[1],f6dp[2],f6dp[3]+b[3]]}"/>
 <xacro:property name="f7" value="${[15,10,0,0]}"/>
 <xacro:property name="f8" value="${[20,40,0,-1.570795]}"/>
-<xacro:property name="b" value="${[30,25,0,4.7124]}"/>
+<xacro:property name="b" value="${[30,25,0,0]}"/>
 <xacro:property name="g" value="${[30,25,0,0]}"/>
+<!-- 4.7124 -->
    <!-- The following is the geometric expresion for an axis rotation -->
    <!-- X'= X*cos(yaw)-Y*sin(yaw) -->
@@ -69,10 +83,10 @@
       <pose frame=''>${f1[0]*cos(yaw)-f1[1]*sin(yaw)} ${f1[0]*sin(yaw)+f1[1]*cos(yaw)} ${f1[2]} 0 0 ${f1[3]+yaw} </pose>
     </model> -->
-    <model name="cubewithflames_2">
+    <!-- <model name="cubewithflames_2">
       <include>
       <uri>model://cubewithflames</uri>
       </include>
       <pose frame=''>${f2[0]*cos(yaw)-f2[1]*sin(yaw)} ${f2[0]*sin(yaw)+f2[1]*cos(yaw)} ${f2[2]} 0 0 ${f2[3]+yaw} </pose>
-    </model>
+    </model> -->
     <!-- <model name="cubewithflames_3">
       <include>
@@ -88,10 +102,10 @@
       <static>true</static>
     </model> -->
-    <model name="cubewithflames_5">
+    <!-- <model name="cubewithflames_5">
       <include>
         <uri>model://cubewithflames</uri>
       </include>
       <pose frame=''>${f5[0]*cos(yaw)-f5[1]*sin(yaw)} ${f5[0]*sin(yaw)+f5[1]*cos(yaw)} ${f5[2]} 0 0 ${f5[3]+yaw} </pose>
-    </model>
+    </model> -->
     <model name="building">
       <include>
