Commit message: Adding Base and Walls to C2 world

File: mbzirc_gazebo_simulation/challenge_worlds/worlds/challenge2.world.xacro (robot description, xacro)
@@ -6,4 +6,5 @@
 <xacro:include filename="$(find challenge_worlds)/urdf/single_green_brick.xacro" />
 <xacro:include filename="$(find challenge_worlds)/urdf/single_orange_brick.xacro" />
+<xacro:include filename="$(find challenge_worlds)/urdf/BaseBricks.xacro" />
 <!-- Global yaw: to change the global position of all the objects in the world -->
 <xacro:arg name="arena_yaw" default="0"/>
@@ -12,21 +13,85 @@
  <!-- 0 => X position , 1 => Y position , 2 => Z position , 3 => Item yaw -->
 <xacro:property name="ground" value="${[30,25,0,0]}"/>
-<xacro:property name="red01" value="${[30.5,14.5,0,0]}"/>
-<xacro:property name="red02" value="${[29.5,14.5,0,0]}"/>
-<xacro:property name="red03" value="${[29.5,15.5,0,0]}"/>
-<xacro:property name="red04" value="${[30.5,15.5,0,0]}"/>
-<xacro:property name="blue01" value="${[19,26,0,0]}"/>
-<xacro:property name="blue02" value="${[19,24,0,0]}"/>
-<xacro:property name="blue03" value="${[21,26,0,0]}"/>
-<xacro:property name="blue04" value="${[21,24,0,0]}"/>
-<xacro:property name="green01" value="${[30.5,35.5,0,0]}"/>
-<xacro:property name="green02" value="${[29.5,35.5,0,0]}"/>
-<xacro:property name="green03" value="${[30.5,34.5,0,0]}"/>
-<xacro:property name="green04" value="${[29.5,34.5,0,0]}"/>
-<xacro:property name="orange01" value="${[41,26,0,0]}"/>
-<xacro:property name="orange02" value="${[41,24,0,0]}"/>
-<xacro:property name="orange03" value="${[39,26,0,0]}"/>
-<xacro:property name="orange04" value="${[39,24,0,0]}"/>
-<xacro:property name="L_frame" value="${[30,25,0.005,0.0]}"/>
+<xacro:property name="basebrick" value="${[15,30,0,0]}"/>
+<xacro:property name="red01" value="${[basebrick[0]+1.17,basebrick[1]-3,basebrick[2]+0.03,basebrick[3]]}"/>
+<xacro:property name="red02" value="${[basebrick[0]+1.17,basebrick[1]-2.5,basebrick[2]+0.03,basebrick[3]]}"/>
+<xacro:property name="red03" value="${[basebrick[0]+1.17,basebrick[1]-2,basebrick[2]+0.03,basebrick[3]]}"/>
+<xacro:property name="red04" value="${[basebrick[0]+1.17,basebrick[1]-1.5,basebrick[2]+0.03,basebrick[3]]}"/>
+<xacro:property name="red05" value="${[basebrick[0]+1.17,basebrick[1]-1,basebrick[2]+0.03,basebrick[3]]}"/>
+<xacro:property name="red06" value="${[basebrick[0]+1.17,basebrick[1]-0.5,basebrick[2]+0.03,basebrick[3]]}"/>
+<xacro:property name="red07" value="${[basebrick[0]+1.17,basebrick[1]+0,basebrick[2]+0.03,basebrick[3]]}"/>
+<xacro:property name="red08" value="${[basebrick[0]+1.17,basebrick[1]+3,basebrick[2]+0.03,basebrick[3]]}"/>
+<xacro:property name="red09" value="${[basebrick[0]+1.17,basebrick[1]+2.5,basebrick[2]+0.03,basebrick[3]]}"/>
+<xacro:property name="red20" value="${[basebrick[0]+1.17,basebrick[1]+2,basebrick[2]+0.03,basebrick[3]]}"/>
+<xacro:property name="red21" value="${[basebrick[0]+1.17,basebrick[1]+1.5,basebrick[2]+0.03,basebrick[3]]}"/>
+<xacro:property name="red22" value="${[basebrick[0]+1.17,basebrick[1]+1,basebrick[2]+0.03,basebrick[3]]}"/>
+<xacro:property name="red23" value="${[basebrick[0]+1.17,basebrick[1]+0.5,basebrick[2]+0.03,basebrick[3]]}"/>
+<xacro:property name="blue01" value="${[basebrick[0]-0.39,basebrick[1]-1,basebrick[2]+0.03,basebrick[3]]}"/>
+<xacro:property name="blue02" value="${[basebrick[0]-0.39,basebrick[1]-3,basebrick[2]+0.03,basebrick[3]]}"/>
+<xacro:property name="blue03" value="${[basebrick[0]-0.39,basebrick[1]+1,basebrick[2]+0.03,basebrick[3]]}"/>
+<xacro:property name="blue04" value="${[basebrick[0]-0.39,basebrick[1]+3,basebrick[2]+0.03,basebrick[3]]}"/>
+<xacro:property name="green01" value="${[basebrick[0]+0.39,basebrick[1]-1,basebrick[2]+0.03,basebrick[3]]}"/>
+<xacro:property name="green02" value="${[basebrick[0]+0.39,basebrick[1]-3,basebrick[2]+0.03,basebrick[3]]}"/>
+<xacro:property name="green03" value="${[basebrick[0]+0.39,basebrick[1]+1,basebrick[2]+0.03,basebrick[3]]}"/>
+<xacro:property name="green04" value="${[basebrick[0]+0.39,basebrick[1]+3,basebrick[2]+0.03,basebrick[3]]}"/>
+<xacro:property name="green05" value="${[basebrick[0]+0.39,basebrick[1]-2,basebrick[2]+0.03,basebrick[3]]}"/>
+<xacro:property name="green06" value="${[basebrick[0]+0.39,basebrick[1]+2,basebrick[2]+0.03,basebrick[3]]}"/>
+<xacro:property name="green07" value="${[basebrick[0]+0.39,basebrick[1]+0,basebrick[2]+0.03,basebrick[3]]}"/>
+<xacro:property name="orange01" value="${[basebrick[0]-1.17,basebrick[1]-1,basebrick[2]+0.03,basebrick[3]]}"/>
+<xacro:property name="orange02" value="${[basebrick[0]-1.17,basebrick[1]-3,basebrick[2]+0.03,basebrick[3]]}"/>
+<xacro:property name="orange03" value="${[basebrick[0]-1.17,basebrick[1]+1,basebrick[2]+0.03,basebrick[3]]}"/>
+<xacro:property name="orange04" value="${[basebrick[0]-1.17,basebrick[1]+3,basebrick[2]+0.03,basebrick[3]]}"/>
+<xacro:property name="L_frame" value="${[41,15,0.005,3.1416]}"/>
+<xacro:property name="dropwall_center" value="${[40,30,0,0]}"/>
+<xacro:property name="dropwall01" value="${[dropwall_center[0]-0.9,dropwall_center[1]+1.2,dropwall_center[2],dropwall_center[3]+1.570795]}"/>
+<xacro:property name="dropwall02" value="${[dropwall_center[0]+0,dropwall_center[1]+0,dropwall_center[2],dropwall_center[3]+0.0]}"/>
+<xacro:property name="dropwall03" value="${[dropwall_center[0]+1.2,dropwall_center[1]-0.9,dropwall_center[2],dropwall_center[3]+1.570795]}"/>
+<xacro:property name="dropwall04" value="${[dropwall_center[0]+2.1,dropwall_center[1]-2.1,dropwall_center[2],dropwall_center[3]+0.0]}"/>
+<!-- UGV Bricks -->
+<xacro:property name="ugvbricks" value="${[15,15,0,0]}"/>
+<xacro:property name="ugv_orange_center" value="${[ugvbricks[0],ugvbricks[1]-3.1,ugvbricks[2],ugvbricks[3]]}"/>
+<xacro:property name="ugv_blue_center" value="${[ugvbricks[0],ugvbricks[1]+0.6,ugvbricks[2],ugvbricks[3]]}"/>
+<xacro:property name="ugv_green_center" value="${[ugvbricks[0],ugvbricks[1]+3.1,ugvbricks[2],ugvbricks[3]]}"/>
+<xacro:property name="ugv_red_center" value="${[ugvbricks[0],ugvbricks[1]+4.6,ugvbricks[2],ugvbricks[3]]}"/>
+<xacro:property name="red10" value="${[ugv_red_center[0]-0.3,ugv_red_center[1]-0.2,ugv_red_center[2],ugv_red_center[3]]}"/>
+<xacro:property name="red11" value="${[ugv_red_center[0],ugv_red_center[1]-0.2,ugv_red_center[2],ugv_red_center[3]]}"/>
+<xacro:property name="red12" value="${[ugv_red_center[0]-0.3,ugv_red_center[1]+0.2,ugv_red_center[2],ugv_red_center[3]]}"/>
+<xacro:property name="red13" value="${[ugv_red_center[0],ugv_red_center[1]+0.2,ugv_red_center[2],ugv_red_center[3]]}"/>
+<xacro:property name="red14" value="${[ugv_red_center[0]-0.3,ugv_red_center[1]-0.2,ugv_red_center[2]+0.25,ugv_red_center[3]]}"/>
+<xacro:property name="red15" value="${[ugv_red_center[0],ugv_red_center[1]-0.2,ugv_red_center[2]+0.25,ugv_red_center[3]]}"/>
+<xacro:property name="red16" value="${[ugv_red_center[0]-0.3,ugv_red_center[1]+0.2,ugv_red_center[2]+0.25,ugv_red_center[3]]}"/>
+<xacro:property name="red17" value="${[ugv_red_center[0],ugv_red_center[1]+0.2,ugv_red_center[2]+0.25,ugv_red_center[3]]}"/>
+<xacro:property name="red18" value="${[ugv_red_center[0]+0.3,ugv_red_center[1]-0.2,ugv_red_center[2],ugv_red_center[3]]}"/>
+<xacro:property name="red19" value="${[ugv_red_center[0]+0.3,ugv_red_center[1]+0.2,ugv_red_center[2],ugv_red_center[3]]}"/>
+<xacro:property name="green10" value="${[ugv_green_center[0]-0.3,ugv_green_center[1]+0.35,ugv_green_center[2],ugv_green_center[3]]}"/>
+<xacro:property name="green11" value="${[ugv_green_center[0]-0.3,ugv_green_center[1]+0.35,ugv_green_center[2]+0.25,ugv_green_center[3]]}"/>
+<xacro:property name="green12" value="${[ugv_green_center[0]-0.3,ugv_green_center[1]-0.35,ugv_green_center[2],ugv_green_center[3]]}"/>
+<xacro:property name="green13" value="${[ugv_green_center[0]-0.3,ugv_green_center[1]-0.35,ugv_green_center[2]+0.25,ugv_green_center[3]]}"/>
+<xacro:property name="green14" value="${[ugv_green_center[0],ugv_green_center[1]+0.35,ugv_green_center[2],ugv_green_center[3]]}"/>
+<xacro:property name="green15" value="${[ugv_green_center[0],ugv_green_center[1]+0.35,ugv_green_center[2]+0.25,ugv_green_center[3]]}"/>
+<xacro:property name="green16" value="${[ugv_green_center[0],ugv_green_center[1]-0.35,ugv_green_center[2],ugv_green_center[3]]}"/>
+<xacro:property name="green17" value="${[ugv_green_center[0],ugv_green_center[1]-0.35,ugv_green_center[2]+0.25,ugv_green_center[3]]}"/>
+<xacro:property name="green18" value="${[ugv_green_center[0]+0.3,ugv_green_center[1]+0.35,ugv_green_center[2],ugv_green_center[3]]}"/>
+<xacro:property name="green19" value="${[ugv_green_center[0]+0.3,ugv_green_center[1]-0.35,ugv_green_center[2],ugv_green_center[3]]}"/>
+<xacro:property name="blue10" value="${[ugv_blue_center[0]-0.3,ugv_blue_center[1]+0.65,ugv_blue_center[2],ugv_blue_center[3]]}"/>
+<xacro:property name="blue11" value="${[ugv_blue_center[0]-0.3,ugv_blue_center[1]+0.65,ugv_blue_center[2]+0.25,ugv_blue_center[3]]}"/>
+<xacro:property name="blue12" value="${[ugv_blue_center[0]-0.3,ugv_blue_center[1]-0.65,ugv_blue_center[2],ugv_blue_center[3]]}"/>
+<xacro:property name="blue13" value="${[ugv_blue_center[0]-0.3,ugv_blue_center[1]-0.65,ugv_blue_center[2]+0.25,ugv_blue_center[3]]}"/>
+<xacro:property name="blue14" value="${[ugv_blue_center[0],ugv_blue_center[1]+0.65,ugv_blue_center[2],ugv_blue_center[3]]}"/>
+<xacro:property name="blue15" value="${[ugv_blue_center[0],ugv_blue_center[1]+0.65,ugv_blue_center[2]+0.25,ugv_blue_center[3]]}"/>
+<xacro:property name="blue16" value="${[ugv_blue_center[0],ugv_blue_center[1]-0.65,ugv_blue_center[2],ugv_blue_center[3]]}"/>
+<xacro:property name="blue17" value="${[ugv_blue_center[0],ugv_blue_center[1]-0.65,ugv_blue_center[2]+0.25,ugv_blue_center[3]]}"/>
+<xacro:property name="blue18" value="${[ugv_blue_center[0]+0.3,ugv_blue_center[1]+0.65,ugv_blue_center[2],ugv_blue_center[3]]}"/>
+<xacro:property name="blue19" value="${[ugv_blue_center[0]+0.3,ugv_blue_center[1]-0.65,ugv_blue_center[2],ugv_blue_center[3]]}"/>
+<xacro:property name="orange10" value="${[ugv_orange_center[0]-0.3,ugv_orange_center[1]+0.95,ugv_orange_center[2],ugv_orange_center[3]]}"/>
+<xacro:property name="orange11" value="${[ugv_orange_center[0]-0.3,ugv_orange_center[1]+0.95,ugv_orange_center[2]+0.25,ugv_orange_center[3]]}"/>
+<xacro:property name="orange12" value="${[ugv_orange_center[0]-0.3,ugv_orange_center[1]-0.95,ugv_orange_center[2],ugv_orange_center[3]]}"/>
+<xacro:property name="orange13" value="${[ugv_orange_center[0]-0.3,ugv_orange_center[1]-0.95,ugv_orange_center[2]+0.25,ugv_orange_center[3]]}"/>
+<xacro:property name="orange14" value="${[ugv_orange_center[0],ugv_orange_center[1]+0.95,ugv_orange_center[2],ugv_orange_center[3]]}"/>
+<xacro:property name="orange15" value="${[ugv_orange_center[0],ugv_orange_center[1]+0.95,ugv_orange_center[2]+0.25,ugv_orange_center[3]]}"/>
+<xacro:property name="orange16" value="${[ugv_orange_center[0],ugv_orange_center[1]-0.95,ugv_orange_center[2],ugv_orange_center[3]]}"/>
+<xacro:property name="orange17" value="${[ugv_orange_center[0],ugv_orange_center[1]-0.95,ugv_orange_center[2]+0.25,ugv_orange_center[3]]}"/>
+<xacro:property name="orange18" value="${[ugv_orange_center[0]+0.3,ugv_orange_center[1]+0.95,ugv_orange_center[2],ugv_orange_center[3]]}"/>
+<xacro:property name="orange19" value="${[ugv_orange_center[0]+0.3,ugv_orange_center[1]-0.95,ugv_orange_center[2],ugv_orange_center[3]]}"/>
   <world name="default">
     <!-- GRIPPER PLUGIN TO AVOID THE NEED OF COLLISIONS -->
@@ -43,4 +108,13 @@
     <single_red_brick id="Red_brick_03" pose="${red03[0]*cos(yaw)-red03[1]*sin(yaw)} ${red03[0]*sin(yaw)+red03[1]*cos(yaw)} ${red03[2]} 0 0 ${red03[3]+yaw}" sx="0.2" sy="0.3" sz="0.2" mass="1.0" mat="Gazebo/Red" />
     <single_red_brick id="Red_brick_04" pose="${red04[0]*cos(yaw)-red04[1]*sin(yaw)} ${red04[0]*sin(yaw)+red04[1]*cos(yaw)} ${red04[2]} 0 0 ${red04[3]+yaw}" sx="0.2" sy="0.3" sz="0.2" mass="1.0" mat="Gazebo/Red" />
+    <single_red_brick id="Red_brick_05" pose="${red05[0]*cos(yaw)-red05[1]*sin(yaw)} ${red05[0]*sin(yaw)+red05[1]*cos(yaw)} ${red05[2]} 0 0 ${red05[3]+yaw}" sx="0.2" sy="0.3" sz="0.2" mass="1.0" mat="Gazebo/Red" />
+    <single_red_brick id="Red_brick_06" pose="${red06[0]*cos(yaw)-red06[1]*sin(yaw)} ${red06[0]*sin(yaw)+red06[1]*cos(yaw)} ${red06[2]} 0 0 ${red06[3]+yaw}" sx="0.2" sy="0.3" sz="0.2" mass="1.0" mat="Gazebo/Red" />
+    <single_red_brick id="Red_brick_07" pose="${red07[0]*cos(yaw)-red07[1]*sin(yaw)} ${red07[0]*sin(yaw)+red07[1]*cos(yaw)} ${red07[2]} 0 0 ${red07[3]+yaw}" sx="0.2" sy="0.3" sz="0.2" mass="1.0" mat="Gazebo/Red" />
+    <single_red_brick id="Red_brick_08" pose="${red08[0]*cos(yaw)-red08[1]*sin(yaw)} ${red08[0]*sin(yaw)+red08[1]*cos(yaw)} ${red08[2]} 0 0 ${red08[3]+yaw}" sx="0.2" sy="0.3" sz="0.2" mass="1.0" mat="Gazebo/Red" />
+    <single_red_brick id="Red_brick_09" pose="${red09[0]*cos(yaw)-red09[1]*sin(yaw)} ${red09[0]*sin(yaw)+red09[1]*cos(yaw)} ${red09[2]} 0 0 ${red09[3]+yaw}" sx="0.2" sy="0.3" sz="0.2" mass="1.0" mat="Gazebo/Red" />
+    <single_red_brick id="Red_brick_20" pose="${red20[0]*cos(yaw)-red20[1]*sin(yaw)} ${red20[0]*sin(yaw)+red20[1]*cos(yaw)} ${red20[2]} 0 0 ${red20[3]+yaw}" sx="0.2" sy="0.3" sz="0.2" mass="1.0" mat="Gazebo/Red" />
+    <single_red_brick id="Red_brick_21" pose="${red21[0]*cos(yaw)-red21[1]*sin(yaw)} ${red21[0]*sin(yaw)+red21[1]*cos(yaw)} ${red21[2]} 0 0 ${red21[3]+yaw}" sx="0.2" sy="0.3" sz="0.2" mass="1.0" mat="Gazebo/Red" />
+    <single_red_brick id="Red_brick_22" pose="${red22[0]*cos(yaw)-red22[1]*sin(yaw)} ${red22[0]*sin(yaw)+red22[1]*cos(yaw)} ${red22[2]} 0 0 ${red22[3]+yaw}" sx="0.2" sy="0.3" sz="0.2" mass="1.0" mat="Gazebo/Red" />
+    <single_red_brick id="Red_brick_23" pose="${red23[0]*cos(yaw)-red23[1]*sin(yaw)} ${red23[0]*sin(yaw)+red23[1]*cos(yaw)} ${red23[2]} 0 0 ${red23[3]+yaw}" sx="0.2" sy="0.3" sz="0.2" mass="1.0" mat="Gazebo/Red" />
     <single_blue_brick id="Blue_brick_01" pose="${blue01[0]*cos(yaw)-blue01[1]*sin(yaw)} ${blue01[0]*sin(yaw)+blue01[1]*cos(yaw)} ${blue01[2]} 0 0 ${blue01[3]+yaw}" sx="0.2" sy="1.2" sz="0.2" mass="1.5" mat="Gazebo/Blue" />
     <single_blue_brick id="Blue_brick_02" pose="${blue02[0]*cos(yaw)-blue02[1]*sin(yaw)} ${blue02[0]*sin(yaw)+blue02[1]*cos(yaw)} ${blue02[2]} 0 0 ${blue02[3]+yaw}" sx="0.2" sy="1.2" sz="0.2" mass="1.5" mat="Gazebo/Blue" />
@@ -51,8 +125,53 @@
     <single_green_brick id="Green_brick_03" pose="${green03[0]*cos(yaw)-green03[1]*sin(yaw)} ${green03[0]*sin(yaw)+green03[1]*cos(yaw)} ${green03[2]} 0 0 ${green03[3]+yaw}" sx="0.2" sy="0.6" sz="0.2" mass="1.0" mat="Gazebo/Green" />
     <single_green_brick id="Green_brick_04" pose="${green04[0]*cos(yaw)-green04[1]*sin(yaw)} ${green04[0]*sin(yaw)+green04[1]*cos(yaw)} ${green04[2]} 0 0 ${green04[3]+yaw}" sx="0.2" sy="0.6" sz="0.2" mass="1.0" mat="Gazebo/Green" />
+    <single_green_brick id="Green_brick_04" pose="${green05[0]*cos(yaw)-green05[1]*sin(yaw)} ${green05[0]*sin(yaw)+green05[1]*cos(yaw)} ${green05[2]} 0 0 ${green05[3]+yaw}" sx="0.2" sy="0.6" sz="0.2" mass="1.0" mat="Gazebo/Green" />
+    <single_green_brick id="Green_brick_04" pose="${green06[0]*cos(yaw)-green06[1]*sin(yaw)} ${green06[0]*sin(yaw)+green06[1]*cos(yaw)} ${green06[2]} 0 0 ${green06[3]+yaw}" sx="0.2" sy="0.6" sz="0.2" mass="1.0" mat="Gazebo/Green" />
+    <single_green_brick id="Green_brick_04" pose="${green07[0]*cos(yaw)-green07[1]*sin(yaw)} ${green07[0]*sin(yaw)+green07[1]*cos(yaw)} ${green07[2]} 0 0 ${green07[3]+yaw}" sx="0.2" sy="0.6" sz="0.2" mass="1.0" mat="Gazebo/Green" />
     <single_orange_brick id="Orange_brick_01" pose="${orange01[0]*cos(yaw)-orange01[1]*sin(yaw)} ${orange01[0]*sin(yaw)+orange01[1]*cos(yaw)} ${orange01[2]} 0 0 ${orange01[3]+yaw}" sx="0.2" sy="1.8" sz="0.2" mass="2.0" mat="Gazebo/Orange" />
     <single_orange_brick id="Orange_brick_02" pose="${orange02[0]*cos(yaw)-orange02[1]*sin(yaw)} ${orange02[0]*sin(yaw)+orange02[1]*cos(yaw)} ${orange02[2]} 0 0 ${orange02[3]+yaw}" sx="0.2" sy="1.8" sz="0.2" mass="2.0" mat="Gazebo/Orange" />
     <single_orange_brick id="Orange_brick_03" pose="${orange03[0]*cos(yaw)-orange03[1]*sin(yaw)} ${orange03[0]*sin(yaw)+orange03[1]*cos(yaw)} ${orange03[2]} 0 0 ${orange03[3]+yaw}" sx="0.2" sy="1.8" sz="0.2" mass="2.0" mat="Gazebo/Orange" />
     <single_orange_brick id="Orange_brick_04" pose="${orange04[0]*cos(yaw)-orange04[1]*sin(yaw)} ${orange04[0]*sin(yaw)+orange04[1]*cos(yaw)} ${orange04[2]} 0 0 ${orange04[3]+yaw}" sx="0.2" sy="1.8" sz="0.2" mass="2.0" mat="Gazebo/Orange" />
+    <!-- UGV Bricks -->
+    <single_red_brick id="Red_brick_10" pose="${red10[0]*cos(yaw)-red10[1]*sin(yaw)} ${red10[0]*sin(yaw)+red10[1]*cos(yaw)} ${red10[2]} 0 0 ${red10[3]+yaw}" sx="0.2" sy="0.3" sz="0.2" mass="1.0" mat="Gazebo/Red" />
+    <single_red_brick id="Red_brick_11" pose="${red11[0]*cos(yaw)-red11[1]*sin(yaw)} ${red11[0]*sin(yaw)+red11[1]*cos(yaw)} ${red11[2]} 0 0 ${red11[3]+yaw}" sx="0.2" sy="0.3" sz="0.2" mass="1.0" mat="Gazebo/Red" />
+    <single_red_brick id="Red_brick_12" pose="${red12[0]*cos(yaw)-red12[1]*sin(yaw)} ${red12[0]*sin(yaw)+red12[1]*cos(yaw)} ${red12[2]} 0 0 ${red12[3]+yaw}" sx="0.2" sy="0.3" sz="0.2" mass="1.0" mat="Gazebo/Red" />
+    <single_red_brick id="Red_brick_13" pose="${red13[0]*cos(yaw)-red13[1]*sin(yaw)} ${red13[0]*sin(yaw)+red13[1]*cos(yaw)} ${red13[2]} 0 0 ${red13[3]+yaw}" sx="0.2" sy="0.3" sz="0.2" mass="1.0" mat="Gazebo/Red" />
+    <single_red_brick id="Red_brick_14" pose="${red14[0]*cos(yaw)-red14[1]*sin(yaw)} ${red14[0]*sin(yaw)+red14[1]*cos(yaw)} ${red14[2]} 0 0 ${red14[3]+yaw}" sx="0.2" sy="0.3" sz="0.2" mass="1.0" mat="Gazebo/Red" />
+    <single_red_brick id="Red_brick_15" pose="${red15[0]*cos(yaw)-red15[1]*sin(yaw)} ${red15[0]*sin(yaw)+red15[1]*cos(yaw)} ${red15[2]} 0 0 ${red15[3]+yaw}" sx="0.2" sy="0.3" sz="0.2" mass="1.0" mat="Gazebo/Red" />
+    <single_red_brick id="Red_brick_16" pose="${red16[0]*cos(yaw)-red16[1]*sin(yaw)} ${red16[0]*sin(yaw)+red16[1]*cos(yaw)} ${red16[2]} 0 0 ${red16[3]+yaw}" sx="0.2" sy="0.3" sz="0.2" mass="1.0" mat="Gazebo/Red" />
+    <single_red_brick id="Red_brick_17" pose="${red17[0]*cos(yaw)-red17[1]*sin(yaw)} ${red17[0]*sin(yaw)+red17[1]*cos(yaw)} ${red17[2]} 0 0 ${red17[3]+yaw}" sx="0.2" sy="0.3" sz="0.2" mass="1.0" mat="Gazebo/Red" />
+    <single_red_brick id="Red_brick_18" pose="${red18[0]*cos(yaw)-red18[1]*sin(yaw)} ${red18[0]*sin(yaw)+red18[1]*cos(yaw)} ${red18[2]} 0 0 ${red18[3]+yaw}" sx="0.2" sy="0.3" sz="0.2" mass="1.0" mat="Gazebo/Red" />
+    <single_red_brick id="Red_brick_19" pose="${red19[0]*cos(yaw)-red19[1]*sin(yaw)} ${red19[0]*sin(yaw)+red19[1]*cos(yaw)} ${red19[2]} 0 0 ${red19[3]+yaw}" sx="0.2" sy="0.3" sz="0.2" mass="1.0" mat="Gazebo/Red" />
+    <single_green_brick id="Green_brick_10" pose="${green10[0]*cos(yaw)-green10[1]*sin(yaw)} ${green10[0]*sin(yaw)+green10[1]*cos(yaw)} ${green10[2]} 0 0 ${green10[3]+yaw}" sx="0.2" sy="0.6" sz="0.2" mass="1.0" mat="Gazebo/Green" />
+    <single_green_brick id="Green_brick_11" pose="${green11[0]*cos(yaw)-green11[1]*sin(yaw)} ${green11[0]*sin(yaw)+green11[1]*cos(yaw)} ${green11[2]} 0 0 ${green11[3]+yaw}" sx="0.2" sy="0.6" sz="0.2" mass="1.0" mat="Gazebo/Green" />
+    <single_green_brick id="Green_brick_12" pose="${green12[0]*cos(yaw)-green12[1]*sin(yaw)} ${green12[0]*sin(yaw)+green12[1]*cos(yaw)} ${green12[2]} 0 0 ${green12[3]+yaw}" sx="0.2" sy="0.6" sz="0.2" mass="1.0" mat="Gazebo/Green" />
+    <single_green_brick id="Green_brick_13" pose="${green13[0]*cos(yaw)-green13[1]*sin(yaw)} ${green13[0]*sin(yaw)+green13[1]*cos(yaw)} ${green13[2]} 0 0 ${green13[3]+yaw}" sx="0.2" sy="0.6" sz="0.2" mass="1.0" mat="Gazebo/Green" />
+    <single_green_brick id="Green_brick_14" pose="${green14[0]*cos(yaw)-green14[1]*sin(yaw)} ${green14[0]*sin(yaw)+green14[1]*cos(yaw)} ${green14[2]} 0 0 ${green14[3]+yaw}" sx="0.2" sy="0.6" sz="0.2" mass="1.0" mat="Gazebo/Green" />
+    <single_green_brick id="Green_brick_15" pose="${green15[0]*cos(yaw)-green15[1]*sin(yaw)} ${green15[0]*sin(yaw)+green15[1]*cos(yaw)} ${green15[2]} 0 0 ${green15[3]+yaw}" sx="0.2" sy="0.6" sz="0.2" mass="1.0" mat="Gazebo/Green" />
+    <single_green_brick id="Green_brick_16" pose="${green16[0]*cos(yaw)-green16[1]*sin(yaw)} ${green16[0]*sin(yaw)+green16[1]*cos(yaw)} ${green16[2]} 0 0 ${green16[3]+yaw}" sx="0.2" sy="0.6" sz="0.2" mass="1.0" mat="Gazebo/Green" />
+    <single_green_brick id="Green_brick_17" pose="${green17[0]*cos(yaw)-green17[1]*sin(yaw)} ${green17[0]*sin(yaw)+green17[1]*cos(yaw)} ${green17[2]} 0 0 ${green17[3]+yaw}" sx="0.2" sy="0.6" sz="0.2" mass="1.0" mat="Gazebo/Green" />
+    <single_green_brick id="Green_brick_18" pose="${green18[0]*cos(yaw)-green18[1]*sin(yaw)} ${green18[0]*sin(yaw)+green18[1]*cos(yaw)} ${green18[2]} 0 0 ${green18[3]+yaw}" sx="0.2" sy="0.6" sz="0.2" mass="1.0" mat="Gazebo/Green" />
+    <single_green_brick id="Green_brick_19" pose="${green19[0]*cos(yaw)-green19[1]*sin(yaw)} ${green19[0]*sin(yaw)+green19[1]*cos(yaw)} ${green19[2]} 0 0 ${green19[3]+yaw}" sx="0.2" sy="0.6" sz="0.2" mass="1.0" mat="Gazebo/Green" />
+    <single_blue_brick id="Blue_brick_10" pose="${blue10[0]*cos(yaw)-blue10[1]*sin(yaw)} ${blue10[0]*sin(yaw)+blue10[1]*cos(yaw)} ${blue10[2]} 0 0 ${blue10[3]+yaw}" sx="0.2" sy="1.2" sz="0.2" mass="1.5" mat="Gazebo/Blue" />
+    <single_blue_brick id="Blue_brick_11" pose="${blue11[0]*cos(yaw)-blue11[1]*sin(yaw)} ${blue11[0]*sin(yaw)+blue11[1]*cos(yaw)} ${blue11[2]} 0 0 ${blue11[3]+yaw}" sx="0.2" sy="1.2" sz="0.2" mass="1.5" mat="Gazebo/Blue" />
+    <single_blue_brick id="Blue_brick_12" pose="${blue12[0]*cos(yaw)-blue12[1]*sin(yaw)} ${blue12[0]*sin(yaw)+blue12[1]*cos(yaw)} ${blue12[2]} 0 0 ${blue12[3]+yaw}" sx="0.2" sy="1.2" sz="0.2" mass="1.5" mat="Gazebo/Blue" />
+    <single_blue_brick id="Blue_brick_13" pose="${blue13[0]*cos(yaw)-blue13[1]*sin(yaw)} ${blue13[0]*sin(yaw)+blue13[1]*cos(yaw)} ${blue13[2]} 0 0 ${blue13[3]+yaw}" sx="0.2" sy="1.2" sz="0.2" mass="1.5" mat="Gazebo/Blue" />
+    <single_blue_brick id="Blue_brick_14" pose="${blue14[0]*cos(yaw)-blue14[1]*sin(yaw)} ${blue14[0]*sin(yaw)+blue14[1]*cos(yaw)} ${blue14[2]} 0 0 ${blue14[3]+yaw}" sx="0.2" sy="1.2" sz="0.2" mass="1.5" mat="Gazebo/Blue" />
+    <single_blue_brick id="Blue_brick_15" pose="${blue15[0]*cos(yaw)-blue15[1]*sin(yaw)} ${blue15[0]*sin(yaw)+blue15[1]*cos(yaw)} ${blue15[2]} 0 0 ${blue15[3]+yaw}" sx="0.2" sy="1.2" sz="0.2" mass="1.5" mat="Gazebo/Blue" />
+    <single_blue_brick id="Blue_brick_16" pose="${blue16[0]*cos(yaw)-blue16[1]*sin(yaw)} ${blue16[0]*sin(yaw)+blue16[1]*cos(yaw)} ${blue16[2]} 0 0 ${blue16[3]+yaw}" sx="0.2" sy="1.2" sz="0.2" mass="1.5" mat="Gazebo/Blue" />
+    <single_blue_brick id="Blue_brick_17" pose="${blue17[0]*cos(yaw)-blue17[1]*sin(yaw)} ${blue17[0]*sin(yaw)+blue17[1]*cos(yaw)} ${blue17[2]} 0 0 ${blue17[3]+yaw}" sx="0.2" sy="1.2" sz="0.2" mass="1.5" mat="Gazebo/Blue" />
+    <single_blue_brick id="Blue_brick_18" pose="${blue18[0]*cos(yaw)-blue18[1]*sin(yaw)} ${blue18[0]*sin(yaw)+blue18[1]*cos(yaw)} ${blue18[2]} 0 0 ${blue18[3]+yaw}" sx="0.2" sy="1.2" sz="0.2" mass="1.5" mat="Gazebo/Blue" />
+    <single_blue_brick id="Blue_brick_19" pose="${blue19[0]*cos(yaw)-blue19[1]*sin(yaw)} ${blue19[0]*sin(yaw)+blue19[1]*cos(yaw)} ${blue19[2]} 0 0 ${blue19[3]+yaw}" sx="0.2" sy="1.2" sz="0.2" mass="1.5" mat="Gazebo/Blue" />
+    <single_orange_brick id="Orange_brick_10" pose="${orange10[0]*cos(yaw)-orange10[1]*sin(yaw)} ${orange10[0]*sin(yaw)+orange10[1]*cos(yaw)} ${orange10[2]} 0 0 ${orange10[3]+yaw}" sx="0.2" sy="1.8" sz="0.2" mass="2" mat="Gazebo/Orange" />
+    <single_orange_brick id="Orange_brick_11" pose="${orange11[0]*cos(yaw)-orange11[1]*sin(yaw)} ${orange11[0]*sin(yaw)+orange11[1]*cos(yaw)} ${orange11[2]} 0 0 ${orange11[3]+yaw}" sx="0.2" sy="1.8" sz="0.2" mass="2" mat="Gazebo/Orange" />
+    <single_orange_brick id="Orange_brick_12" pose="${orange12[0]*cos(yaw)-orange12[1]*sin(yaw)} ${orange12[0]*sin(yaw)+orange12[1]*cos(yaw)} ${orange12[2]} 0 0 ${orange12[3]+yaw}" sx="0.2" sy="1.8" sz="0.2" mass="2" mat="Gazebo/Orange" />
+    <single_orange_brick id="Orange_brick_13" pose="${orange13[0]*cos(yaw)-orange13[1]*sin(yaw)} ${orange13[0]*sin(yaw)+orange13[1]*cos(yaw)} ${orange13[2]} 0 0 ${orange13[3]+yaw}" sx="0.2" sy="1.8" sz="0.2" mass="2" mat="Gazebo/Orange" />
+    <single_orange_brick id="Orange_brick_14" pose="${orange14[0]*cos(yaw)-orange14[1]*sin(yaw)} ${orange14[0]*sin(yaw)+orange14[1]*cos(yaw)} ${orange14[2]} 0 0 ${orange14[3]+yaw}" sx="0.2" sy="1.8" sz="0.2" mass="2" mat="Gazebo/Orange" />
+    <single_orange_brick id="Orange_brick_15" pose="${orange15[0]*cos(yaw)-orange15[1]*sin(yaw)} ${orange15[0]*sin(yaw)+orange15[1]*cos(yaw)} ${orange15[2]} 0 0 ${orange15[3]+yaw}" sx="0.2" sy="1.8" sz="0.2" mass="2" mat="Gazebo/Orange" />
+    <single_orange_brick id="Orange_brick_16" pose="${orange16[0]*cos(yaw)-orange16[1]*sin(yaw)} ${orange16[0]*sin(yaw)+orange16[1]*cos(yaw)} ${orange16[2]} 0 0 ${orange16[3]+yaw}" sx="0.2" sy="1.8" sz="0.2" mass="2" mat="Gazebo/Orange" />
+    <single_orange_brick id="Orange_brick_17" pose="${orange17[0]*cos(yaw)-orange17[1]*sin(yaw)} ${orange17[0]*sin(yaw)+orange17[1]*cos(yaw)} ${orange17[2]} 0 0 ${orange17[3]+yaw}" sx="0.2" sy="1.8" sz="0.2" mass="2" mat="Gazebo/Orange" />
+    <single_orange_brick id="Orange_brick_18" pose="${orange18[0]*cos(yaw)-orange18[1]*sin(yaw)} ${orange18[0]*sin(yaw)+orange18[1]*cos(yaw)} ${orange18[2]} 0 0 ${orange18[3]+yaw}" sx="0.2" sy="1.8" sz="0.2" mass="2" mat="Gazebo/Orange" />
+    <single_orange_brick id="Orange_brick_19" pose="${orange19[0]*cos(yaw)-orange19[1]*sin(yaw)} ${orange19[0]*sin(yaw)+orange19[1]*cos(yaw)} ${orange19[2]} 0 0 ${orange19[3]+yaw}" sx="0.2" sy="1.8" sz="0.2" mass="2" mat="Gazebo/Orange" />
+    <BaseBricks pose="${basebrick[0]*cos(yaw)-basebrick[1]*sin(yaw)} ${basebrick[0]*sin(yaw)+basebrick[1]*cos(yaw)} ${basebrick[2]} 0 0 ${basebrick[3]+yaw}" />
     <model name="L_wooden_frame">
       <include>
@@ -60,4 +179,28 @@
       </include>
       <pose frame=''>${L_frame[0]*cos(yaw)-L_frame[1]*sin(yaw)} ${L_frame[0]*sin(yaw)+L_frame[1]*cos(yaw)} ${L_frame[2]} 0 0 ${L_frame[3]+yaw} </pose>
+    </model>
+    <model name="DropWall01">
+      <include>
+        <uri>model://DropWall</uri>
+      </include>
+      <pose frame=''>${dropwall01[0]*cos(yaw)-dropwall01[1]*sin(yaw)} ${dropwall01[0]*sin(yaw)+dropwall01[1]*cos(yaw)} ${dropwall01[2]} 0 0 ${dropwall01[3]+yaw} </pose>
+    </model>
+    <model name="DropWall02">
+      <include>
+        <uri>model://DropWall</uri>
+      </include>
+      <pose frame=''>${dropwall02[0]*cos(yaw)-dropwall02[1]*sin(yaw)} ${dropwall02[0]*sin(yaw)+dropwall02[1]*cos(yaw)} ${dropwall02[2]} 0 0 ${dropwall02[3]+yaw} </pose>
+    </model>
+    <model name="DropWall03">
+      <include>
+        <uri>model://DropWall</uri>
+      </include>
+      <pose frame=''>${dropwall03[0]*cos(yaw)-dropwall03[1]*sin(yaw)} ${dropwall03[0]*sin(yaw)+dropwall03[1]*cos(yaw)} ${dropwall03[2]} 0 0 ${dropwall03[3]+yaw} </pose>
+    </model>
+    <model name="DropWall04">
+      <include>
+        <uri>model://DropWall</uri>
+      </include>
+      <pose frame=''>${dropwall04[0]*cos(yaw)-dropwall04[1]*sin(yaw)} ${dropwall04[0]*sin(yaw)+dropwall04[1]*cos(yaw)} ${dropwall04[2]} 0 0 ${dropwall04[3]+yaw} </pose>
     </model>
   </world>
