Commit message: resize wall2 CH2

File: mbzirc_gazebo_simulation/challenge_worlds/worlds/challenge2.world.xacro (robot description, xacro)
@@ -81,11 +81,11 @@
 <!-- Change "dropwall_center" to modify location and yaw -->
 <xacro:property name="dropwall_center" value="${[40,30,0,0]}"/>
-<xacro:property name="dropwall01p" value="${[dropwall_center[0]-0.9,dropwall_center[1]+1.2,dropwall_center[2],1.570795]}"/>
+<xacro:property name="dropwall01p" value="${[dropwall_center[0]-1.9,dropwall_center[1]+2.2,dropwall_center[2],1.570795]}"/>
 <xacro:property name="dropwall01" value="${[(dropwall01p[0]-dropwall_center[0])*cos(dropwall_center[3])-(dropwall01p[1]-dropwall_center[1])*sin(dropwall_center[3])+dropwall_center[0],(dropwall01p[0]-dropwall_center[0])*sin(dropwall_center[3])+(dropwall01p[1]-dropwall_center[1])*cos(dropwall_center[3])+dropwall_center[1],dropwall01p[2],dropwall01p[3]+dropwall_center[3]]}"/>
 <xacro:property name="dropwall02p" value="${[dropwall_center[0]+0,dropwall_center[1]+0,dropwall_center[2],0.0]}"/>
 <xacro:property name="dropwall02" value="${[(dropwall02p[0]-dropwall_center[0])*cos(dropwall_center[3])-(dropwall02p[1]-dropwall_center[1])*sin(dropwall_center[3])+dropwall_center[0],(dropwall02p[0]-dropwall_center[0])*sin(dropwall_center[3])+(dropwall02p[1]-dropwall_center[1])*cos(dropwall_center[3])+dropwall_center[1],dropwall02p[2],dropwall02p[3]+dropwall_center[3]]}"/>
-<xacro:property name="dropwall03p" value="${[dropwall_center[0]+1.2,dropwall_center[1]-0.9,dropwall_center[2],1.570795]}"/>
+<xacro:property name="dropwall03p" value="${[dropwall_center[0]+2.2,dropwall_center[1]-1.9,dropwall_center[2],1.570795]}"/>
 <xacro:property name="dropwall03" value="${[(dropwall03p[0]-dropwall_center[0])*cos(dropwall_center[3])-(dropwall03p[1]-dropwall_center[1])*sin(dropwall_center[3])+dropwall_center[0],(dropwall03p[0]-dropwall_center[0])*sin(dropwall_center[3])+(dropwall03p[1]-dropwall_center[1])*cos(dropwall_center[3])+dropwall_center[1],dropwall03p[2],dropwall03p[3]+dropwall_center[3]]}"/>
-<xacro:property name="dropwall04p" value="${[dropwall_center[0]+2.1,dropwall_center[1]-2.1,dropwall_center[2],0.0]}"/>
+<xacro:property name="dropwall04p" value="${[dropwall_center[0]+4.1,dropwall_center[1]-4.1,dropwall_center[2],0.0]}"/>
 <xacro:property name="dropwall04" value="${[(dropwall04p[0]-dropwall_center[0])*cos(dropwall_center[3])-(dropwall04p[1]-dropwall_center[1])*sin(dropwall_center[3])+dropwall_center[0],(dropwall04p[0]-dropwall_center[0])*sin(dropwall_center[3])+(dropwall04p[1]-dropwall_center[1])*cos(dropwall_center[3])+dropwall_center[1],dropwall04p[2],dropwall04p[3]+dropwall_center[3]]}"/>
 <!-- UGV Bricks Location-->

Commit message: re-locating arena and building in ch2 and ch3 after visiting real arena

File: mbzirc_gazebo_simulation/challenge_worlds/worlds/challenge2.world.xacro (robot description, xacro)
@@ -15,5 +15,5 @@
     <!-- X'-x= (X-x)*cos(yaw)-(Y-y)*sin(yaw) -->
     <!-- Y'-y= (X-x)*sin(yaw)+(Y-y)*cos(yaw)  -->
-<xacro:property name="ground" value="${[25,30,0,0]}"/>
+<xacro:property name="ground" value="${[30,25,0,0]}"/>
 <!-- UAV BRICKS Location -->
 <!-- Change "basebrick" to modify location and yaw for the entire pile-->

File: mbzirc_gazebo_simulation/challenge_worlds/worlds/challenge3.world.xacro (robot description, xacro)
@@ -39,6 +39,6 @@
 <xacro:property name="f7" value="${[30,10,0,0]}"/>
 <xacro:property name="f8" value="${[10,40,0,-1.570795]}"/>
-<xacro:property name="b" value="${[20,23,0,0]}"/>
-<xacro:property name="g" value="${[25,30,0,0]}"/>
+<xacro:property name="b" value="${[40,20,0,1.57]}"/>
+<xacro:property name="g" value="${[30,25,0,0]}"/>
 <!-- 4.7124 -->
    <!-- The following is the geometric expresion for an axis rotation -->
