Commit message: modifying arena origin in ch2 and ch3

File: mbzirc_gazebo_simulation/challenge_worlds/worlds/challenge2.world.xacro (robot description, xacro)
@@ -15,8 +15,8 @@
     <!-- X'-x= (X-x)*cos(yaw)-(Y-y)*sin(yaw) -->
     <!-- Y'-y= (X-x)*sin(yaw)+(Y-y)*cos(yaw)  -->
-<xacro:property name="ground" value="${[30,25,0,0]}"/>
+<xacro:property name="ground" value="${[8,17,0,0]}"/>
 <!-- UAV BRICKS Location -->
 <!-- Change "basebrick" to modify location and yaw for the entire pile-->
-<xacro:property name="basebrick" value="${[41,15,0,0]}"/>
+<xacro:property name="basebrick" value="${[14,7,0,-1.57]}"/>
 <xacro:property name="red01p" value="${[basebrick[0]+1.95,basebrick[1]-3.3,basebrick[2]+0.03,0]}"/>
 <xacro:property name="red01" value="${[(red01p[0]-basebrick[0])*cos(basebrick[3])-(red01p[1]-basebrick[1])*sin(basebrick[3])+basebrick[0],(red01p[0]-basebrick[0])*sin(basebrick[3])+(red01p[1]-basebrick[1])*cos(basebrick[3])+basebrick[1],red01p[2],red01p[3]+basebrick[3]]}"/>
@@ -113,8 +113,8 @@
 <!-- WALL 1 Location (L-SHAPE FRAME) -->
 <!-- Change "L_frame" to modify location and yaw -->
-<xacro:property name="L_frame" value="${[17,32,0.005,3.1416]}"/>
+<xacro:property name="L_frame" value="${[-14,28,0.005,-1.57]}"/>
 <!-- WALL 2 Location-->
 <!-- Change "dropwall_center" to modify location and yaw -->
-<xacro:property name="dropwall_center" value="${[40,30,0,0]}"/>
+<xacro:property name="dropwall_center" value="${[14,28,0,3.9278]}"/>
 <xacro:property name="dropwall01p" value="${[dropwall_center[0]-1.9,dropwall_center[1]+2.2,dropwall_center[2],1.570795]}"/>
 <xacro:property name="dropwall01" value="${[(dropwall01p[0]-dropwall_center[0])*cos(dropwall_center[3])-(dropwall01p[1]-dropwall_center[1])*sin(dropwall_center[3])+dropwall_center[0],(dropwall01p[0]-dropwall_center[0])*sin(dropwall_center[3])+(dropwall01p[1]-dropwall_center[1])*cos(dropwall_center[3])+dropwall_center[1],dropwall01p[2],dropwall01p[3]+dropwall_center[3]]}"/>
@@ -127,5 +127,5 @@
 <!-- UGV Bricks Location-->
 <!-- Change ugvbricks to modify location and yaw for the entire pile-->
-<xacro:property name="ugvbricks" value="${[15,12,0,0]}"/>
+<xacro:property name="ugvbricks" value="${[-14,7,0,-1.57]}"/>
 <xacro:property name="ugv_orange_centerp" value="${[ugvbricks[0]+0.1,ugvbricks[1]+0.9,ugvbricks[2],0]}"/>
 <xacro:property name="ugv_orange_center" value="${[(ugv_orange_centerp[0]-ugvbricks[0])*cos(ugvbricks[3])-(ugv_orange_centerp[1]-ugvbricks[1])*sin(ugvbricks[3])+ugvbricks[0],(ugv_orange_centerp[0]-ugvbricks[0])*sin(ugvbricks[3])+(ugv_orange_centerp[1]-ugvbricks[1])*cos(ugvbricks[3])+ugvbricks[1],ugv_orange_centerp[2],ugv_orange_centerp[3]+ugvbricks[3]]}"/>

File: mbzirc_gazebo_simulation/challenge_worlds/worlds/challenge3.world.xacro (robot description, xacro)
@@ -63,8 +63,8 @@
 <xacro:property name="f52c" value="${[(f52cp[0]-b[0])*cos(b[3])-(f52cp[1]-b[1])*sin(b[3])+b[0],(f52cp[0]-b[0])*sin(b[3])+(f52cp[1]-b[1])*cos(b[3])+b[1],f52cp[2],f52cp[3]+b[3]]}"/> -->
 <!-- OUTDOOR FIRES -->
-<xacro:property name="f7" value="${[5,17,0,0]}"/>
-<xacro:property name="f8" value="${[15,11,0,-1.570795]}"/>
-<xacro:property name="b" value="${[26,22.,0,-1.57]}"/>
-<xacro:property name="g" value="${[30,25,0,0]}"/>
+<xacro:property name="f7" value="${[-25,17,0,0]}"/>
+<xacro:property name="f8" value="${[-15,11,0,-1.570795]}"/>
+<xacro:property name="b" value="${[-4.1,21.93,0,-1.57]}"/>
+<xacro:property name="g" value="${[0,25,0,0]}"/>
    <!-- The following is the geometric expresion for an axis rotation -->
    <!-- X'= X*cos(yaw)-Y*sin(yaw) -->

Commit message: placing dropwall closer to uav bricks in ch2

File: mbzirc_gazebo_simulation/challenge_worlds/worlds/challenge2.world.xacro (robot description, xacro)
@@ -18,5 +18,5 @@
 <!-- UAV BRICKS Location -->
 <!-- Change "basebrick" to modify location and yaw for the entire pile-->
-<xacro:property name="basebrick" value="${[14,7,0,-1.57]}"/>
+<xacro:property name="basebrick" value="${[14,10,0,-1.57]}"/>
 <xacro:property name="red01p" value="${[basebrick[0]+1.95,basebrick[1]-3.3,basebrick[2]+0.03,0]}"/>
 <xacro:property name="red01" value="${[(red01p[0]-basebrick[0])*cos(basebrick[3])-(red01p[1]-basebrick[1])*sin(basebrick[3])+basebrick[0],(red01p[0]-basebrick[0])*sin(basebrick[3])+(red01p[1]-basebrick[1])*cos(basebrick[3])+basebrick[1],red01p[2],red01p[3]+basebrick[3]]}"/>
@@ -116,5 +116,5 @@
 <!-- WALL 2 Location-->
 <!-- Change "dropwall_center" to modify location and yaw -->
-<xacro:property name="dropwall_center" value="${[14,28,0,3.9278]}"/>
+<xacro:property name="dropwall_center" value="${[14,22,0,3.9278]}"/>
 <xacro:property name="dropwall01p" value="${[dropwall_center[0]-1.9,dropwall_center[1]+2.2,dropwall_center[2],1.570795]}"/>
 <xacro:property name="dropwall01" value="${[(dropwall01p[0]-dropwall_center[0])*cos(dropwall_center[3])-(dropwall01p[1]-dropwall_center[1])*sin(dropwall_center[3])+dropwall_center[0],(dropwall01p[0]-dropwall_center[0])*sin(dropwall_center[3])+(dropwall01p[1]-dropwall_center[1])*cos(dropwall_center[3])+dropwall_center[1],dropwall01p[2],dropwall01p[3]+dropwall_center[3]]}"/>

File: mbzirc_gazebo_simulation/uavs_description/models/mbzirc2020/model.xacro (robot description, xacro)
@@ -521,5 +521,5 @@
           <robotNamespace>${namespace}</robotNamespace>
           <cameraName>camera</cameraName>
-          <imageTopicName>color/image_raw</imageTopicName>
+          <imageTopicName>color/image_rect_color</imageTopicName>
           <!-- <cameraInfoTopicName>color/camera_info</cameraInfoTopicName> -->
           <cameraInfoTopicName>aligned_depth_to_color/camera_info</cameraInfoTopicName>

Commit message: moving piles for trial 2

File: mbzirc_gazebo_simulation/challenge_worlds/worlds/challenge2.world.xacro (robot description, xacro)
@@ -18,5 +18,5 @@
 <!-- UAV BRICKS Location -->
 <!-- Change "basebrick" to modify location and yaw for the entire pile-->
-<xacro:property name="basebrick" value="${[14,10,0,-1.57]}"/>
+<xacro:property name="basebrick" value="${[-11,12,0,-1.57]}"/>
 <xacro:property name="red01p" value="${[basebrick[0]+1.95,basebrick[1]-3.3,basebrick[2]+0.03,0]}"/>
 <xacro:property name="red01" value="${[(red01p[0]-basebrick[0])*cos(basebrick[3])-(red01p[1]-basebrick[1])*sin(basebrick[3])+basebrick[0],(red01p[0]-basebrick[0])*sin(basebrick[3])+(red01p[1]-basebrick[1])*cos(basebrick[3])+basebrick[1],red01p[2],red01p[3]+basebrick[3]]}"/>
@@ -113,8 +113,8 @@
 <!-- WALL 1 Location (L-SHAPE FRAME) -->
 <!-- Change "L_frame" to modify location and yaw -->
-<xacro:property name="L_frame" value="${[-14,28,0.005,-1.57]}"/>
+<xacro:property name="L_frame" value="${[14,22,0.005,-1.57]}"/>
 <!-- WALL 2 Location-->
 <!-- Change "dropwall_center" to modify location and yaw -->
-<xacro:property name="dropwall_center" value="${[14,22,0,3.9278]}"/>
+<xacro:property name="dropwall_center" value="${[-10.26,22.28,0,3.9278-0.25]}"/>
 <xacro:property name="dropwall01p" value="${[dropwall_center[0]-1.9,dropwall_center[1]+2.2,dropwall_center[2],1.570795]}"/>
 <xacro:property name="dropwall01" value="${[(dropwall01p[0]-dropwall_center[0])*cos(dropwall_center[3])-(dropwall01p[1]-dropwall_center[1])*sin(dropwall_center[3])+dropwall_center[0],(dropwall01p[0]-dropwall_center[0])*sin(dropwall_center[3])+(dropwall01p[1]-dropwall_center[1])*cos(dropwall_center[3])+dropwall_center[1],dropwall01p[2],dropwall01p[3]+dropwall_center[3]]}"/>
@@ -127,5 +127,5 @@
 <!-- UGV Bricks Location-->
 <!-- Change ugvbricks to modify location and yaw for the entire pile-->
-<xacro:property name="ugvbricks" value="${[-14,7,0,-1.57]}"/>
+<xacro:property name="ugvbricks" value="${[14,7,0,-1.57]}"/>
 <xacro:property name="ugv_orange_centerp" value="${[ugvbricks[0]+0.1,ugvbricks[1]+0.9,ugvbricks[2],0]}"/>
 <xacro:property name="ugv_orange_center" value="${[(ugv_orange_centerp[0]-ugvbricks[0])*cos(ugvbricks[3])-(ugv_orange_centerp[1]-ugvbricks[1])*sin(ugvbricks[3])+ugvbricks[0],(ugv_orange_centerp[0]-ugvbricks[0])*sin(ugvbricks[3])+(ugv_orange_centerp[1]-ugvbricks[1])*cos(ugvbricks[3])+ugvbricks[1],ugv_orange_centerp[2],ugv_orange_centerp[3]+ugvbricks[3]]}"/>

Commit message: Adapt sim to grand challenge layout

File: mbzirc_gazebo_simulation/challenge_worlds/worlds/challenge2.world.xacro (robot description, xacro)
@@ -18,5 +18,6 @@
 <!-- UAV BRICKS Location -->
 <!-- Change "basebrick" to modify location and yaw for the entire pile-->
-<xacro:property name="basebrick" value="${[-11,12,0,-1.57]}"/>
+<xacro:property name="basebrick" value="${[-6,12,0,-1.57]}"/>
+<xacro:property name="dropwall_center" value="${[-5,22.28,0,3.9278-0.25]}"/>
 <xacro:property name="red01p" value="${[basebrick[0]+1.95,basebrick[1]-3.3,basebrick[2]+0.03,0]}"/>
 <xacro:property name="red01" value="${[(red01p[0]-basebrick[0])*cos(basebrick[3])-(red01p[1]-basebrick[1])*sin(basebrick[3])+basebrick[0],(red01p[0]-basebrick[0])*sin(basebrick[3])+(red01p[1]-basebrick[1])*cos(basebrick[3])+basebrick[1],red01p[2],red01p[3]+basebrick[3]]}"/>
@@ -116,5 +117,4 @@
 <!-- WALL 2 Location-->
 <!-- Change "dropwall_center" to modify location and yaw -->
-<xacro:property name="dropwall_center" value="${[-10.26,22.28,0,3.9278-0.25]}"/>
 <xacro:property name="dropwall01p" value="${[dropwall_center[0]-1.9,dropwall_center[1]+2.2,dropwall_center[2],1.570795]}"/>
 <xacro:property name="dropwall01" value="${[(dropwall01p[0]-dropwall_center[0])*cos(dropwall_center[3])-(dropwall01p[1]-dropwall_center[1])*sin(dropwall_center[3])+dropwall_center[0],(dropwall01p[0]-dropwall_center[0])*sin(dropwall_center[3])+(dropwall01p[1]-dropwall_center[1])*cos(dropwall_center[3])+dropwall_center[1],dropwall01p[2],dropwall01p[3]+dropwall_center[3]]}"/>

Commit message: Last changes for Grand Challenge

File: mbzirc_gazebo_simulation/challenge_worlds/worlds/challenge2.world.xacro (robot description, xacro)
@@ -18,6 +18,6 @@
 <!-- UAV BRICKS Location -->
 <!-- Change "basebrick" to modify location and yaw for the entire pile-->
-<xacro:property name="basebrick" value="${[-6,12,0,-1.57]}"/>
-<xacro:property name="dropwall_center" value="${[-5,22.28,0,3.9278-0.25]}"/>
+<xacro:property name="basebrick" value="${[-10.17,14.37,0,-1.57]}"/>
+<xacro:property name="dropwall_center" value="${[-9.075,23.42,0,3.9278-0.25]}"/>
 <xacro:property name="red01p" value="${[basebrick[0]+1.95,basebrick[1]-3.3,basebrick[2]+0.03,0]}"/>
 <xacro:property name="red01" value="${[(red01p[0]-basebrick[0])*cos(basebrick[3])-(red01p[1]-basebrick[1])*sin(basebrick[3])+basebrick[0],(red01p[0]-basebrick[0])*sin(basebrick[3])+(red01p[1]-basebrick[1])*cos(basebrick[3])+basebrick[1],red01p[2],red01p[3]+basebrick[3]]}"/>

Commit message: Use new predefined paths, move asphalt to the left

File: mbzirc_gazebo_simulation/challenge_worlds/worlds/challenge2.world.xacro (robot description, xacro)
@@ -15,5 +15,5 @@
     <!-- X'-x= (X-x)*cos(yaw)-(Y-y)*sin(yaw) -->
     <!-- Y'-y= (X-x)*sin(yaw)+(Y-y)*cos(yaw)  -->
-<xacro:property name="ground" value="${[8,17,0,0]}"/>
+<xacro:property name="ground" value="${[3,17,0,0]}"/>
 <!-- UAV BRICKS Location -->
 <!-- Change "basebrick" to modify location and yaw for the entire pile-->
