Commit message: changing to single bricks in C2

File: mbzirc_gazebo_simulation/challenge_worlds/models/ground_plane_asfalt/ground_plane_asfalt.xacro (robot description, xacro)
@@ -40,7 +40,8 @@
           <material>
             <script>
-              <uri>model://ground_plane_asfalt/materials/scripts</uri>
-              <uri>model://ground_plane_asfalt/materials/textures</uri>
-		      <name>${material}</name>
+              <uri>file://materials/mbzirc.material</uri>
+              <!-- <uri>model://ground_plane_asfalt/materials/scripts</uri>
+              <uri>model://ground_plane_asfalt/materials/textures</uri> -->
+		          <name>${material}</name>
             </script>
           </material>

File: mbzirc_gazebo_simulation/challenge_worlds/worlds/challenge2.world.xacro (robot description, xacro)
@@ -1,30 +1,66 @@
 <?xml version="1.0" ?>
 <sdf version="1.4" xmlns:xacro="http://www.ros.org/wiki/xacro">
-<xacro:include filename="$(find challenge_worlds)/urdf/orange_pile.xacro" />
+<!-- <xacro:include filename="$(find challenge_worlds)/urdf/orange_pile.xacro" />
 <xacro:include filename="$(find challenge_worlds)/urdf/blue_pile.xacro" />
 <xacro:include filename="$(find challenge_worlds)/urdf/red_pile.xacro" />
-<xacro:include filename="$(find challenge_worlds)/urdf/green_pile.xacro" />
+<xacro:include filename="$(find challenge_worlds)/urdf/green_pile.xacro" /> -->
+<xacro:include filename="$(find challenge_worlds)/models/ground_plane_asfalt/ground_plane_asfalt.xacro" />
+<xacro:include filename="$(find challenge_worlds)/urdf/single_colored_brick.xacro" />
 <!-- Global yaw: to change the global position of all the objects in the world -->
 <xacro:property name="yaw" value="0"/>
 <!-- Properties for every object in the world -->
  <!-- 0 => X position , 1 => Y position , 2 => Z position , 3 => Item yaw -->
-<xacro:property name="orange" value="${[10,0,0,0]}"/>
+<!-- <xacro:property name="orange" value="${[10,0,0,0]}"/>
 <xacro:property name="blue" value="${[-10,0,0,0]}"/>
 <xacro:property name="green" value="${[0,10,0,0]}"/>
-<xacro:property name="red" value="${[0,-10,0,0]}"/>
+<xacro:property name="red" value="${[0,-10,0,0]}"/>  -->
+<xacro:property name="ground" value="${[0,0,0,0]}"/>
+<xacro:property name="red01" value="${[0.5,-10.5,0,0]}"/>
+<xacro:property name="red02" value="${[-0.5,-10.5,0,0]}"/>
+<xacro:property name="red03" value="${[-0.5,-9.5,0,0]}"/>
+<xacro:property name="red04" value="${[0.5,-9.5,0,0]}"/>
+<xacro:property name="blue01" value="${[-11,0.5,0,0]}"/>
+<xacro:property name="blue02" value="${[-11,-0.5,0,0]}"/>
+<xacro:property name="blue03" value="${[-9,0.5,0,0]}"/>
+<xacro:property name="blue04" value="${[-9,-0.5,0,0]}"/>
+<xacro:property name="green01" value="${[0.5,10.5,0,0]}"/>
+<xacro:property name="green02" value="${[-0.5,10.5,0,0]}"/>
+<xacro:property name="green03" value="${[0.5,9.5,0,0]}"/>
+<xacro:property name="green04" value="${[-0.5,9.5,0,0]}"/>
+<xacro:property name="orange01" value="${[11,0.5,0,0]}"/>
+<xacro:property name="orange02" value="${[11,-0.5,0,0]}"/>
+<xacro:property name="orange03" value="${[9,0.5,0,0]}"/>
+<xacro:property name="orange04" value="${[9,-0.5,0,0]}"/>
   <world name="default">
-    <include>
+    <!-- <include>
       <uri>model://ground_plane</uri>
-    </include>
+    </include> -->
     <include>
       <uri>model://sun</uri>
     </include>
+    <ground_plane_asfalt arena_yaw="${yaw}" pose="${ground[0]*cos(yaw)-ground[1]*sin(yaw)} ${ground[0]*sin(yaw)+ground[1]*cos(yaw)} ${ground[2]} 0 0 ${ground[3]+yaw}" material="mbzirc/Asfalt" />
     <!-- The following is the geometric expresion for an axis rotation -->
     <!-- X'= X*cos(yaw)-Y*sin(yaw) -->
     <!-- Y'= X*sin(yaw)+Y*cos(yaw)  -->
-    <orange_pile id="1" pose="${orange[0]*cos(yaw)-orange[1]*sin(yaw)} ${orange[0]*sin(yaw)+orange[1]*cos(yaw)} ${orange[2]} 0 0 ${orange[3]+yaw}" />
+    <!-- <orange_pile id="1" pose="${orange[0]*cos(yaw)-orange[1]*sin(yaw)} ${orange[0]*sin(yaw)+orange[1]*cos(yaw)} ${orange[2]} 0 0 ${orange[3]+yaw}" />
     <blue_pile id="2" pose="${blue[0]*cos(yaw)-blue[1]*sin(yaw)} ${blue[0]*sin(yaw)+blue[1]*cos(yaw)} ${blue[2]} 0 0 ${yaw+blue[3]}" />
     <green_pile id="3" pose="${green[0]*cos(yaw)-green[1]*sin(yaw)} ${green[0]*sin(yaw)+green[1]*cos(yaw)} ${green[2]} 0 0 ${yaw+green[3]}" />
-    <red_pile id="4" pose="${red[0]*cos(yaw)-red[1]*sin(yaw)} ${red[0]*sin(yaw)+red[1]*cos(yaw)} ${red[2]} 0 0 ${yaw+red[3]}" />
+    <red_pile id="4" pose="${red[0]*cos(yaw)-red[1]*sin(yaw)} ${red[0]*sin(yaw)+red[1]*cos(yaw)} ${red[2]} 0 0 ${yaw+red[3]}" /> -->
+    <single_colored_brick id="Red_brick_01" pose="${red01[0]*cos(yaw)-red01[1]*sin(yaw)} ${red01[0]*sin(yaw)+red01[1]*cos(yaw)} ${red01[2]} 0 0 ${red01[3]+yaw}" sx="0.3" sy="0.2" sz="0.2" mass="1.0" mat="Gazebo/Red" />
+    <single_colored_brick id="Red_brick_02" pose="${red02[0]*cos(yaw)-red02[1]*sin(yaw)} ${red02[0]*sin(yaw)+red02[1]*cos(yaw)} ${red02[2]} 0 0 ${red02[3]+yaw}" sx="0.3" sy="0.2" sz="0.2" mass="1.0" mat="Gazebo/Red" />
+    <single_colored_brick id="Red_brick_03" pose="${red03[0]*cos(yaw)-red03[1]*sin(yaw)} ${red03[0]*sin(yaw)+red03[1]*cos(yaw)} ${red03[2]} 0 0 ${red03[3]+yaw}" sx="0.3" sy="0.2" sz="0.2" mass="1.0" mat="Gazebo/Red" />
+    <single_colored_brick id="Red_brick_04" pose="${red04[0]*cos(yaw)-red04[1]*sin(yaw)} ${red04[0]*sin(yaw)+red04[1]*cos(yaw)} ${red04[2]} 0 0 ${red04[3]+yaw}" sx="0.3" sy="0.2" sz="0.2" mass="1.0" mat="Gazebo/Red" />
+    <single_colored_brick id="Blue_brick_01" pose="${blue01[0]*cos(yaw)-blue01[1]*sin(yaw)} ${blue01[0]*sin(yaw)+blue01[1]*cos(yaw)} ${blue01[2]} 0 0 ${blue01[3]+yaw}" sx="1.2" sy="0.2" sz="0.2" mass="1.0" mat="Gazebo/Blue" />
+    <single_colored_brick id="Blue_brick_02" pose="${blue02[0]*cos(yaw)-blue02[1]*sin(yaw)} ${blue02[0]*sin(yaw)+blue02[1]*cos(yaw)} ${blue02[2]} 0 0 ${blue02[3]+yaw}" sx="1.2" sy="0.2" sz="0.2" mass="1.0" mat="Gazebo/Blue" />
+    <single_colored_brick id="Blue_brick_03" pose="${blue03[0]*cos(yaw)-blue03[1]*sin(yaw)} ${blue03[0]*sin(yaw)+blue03[1]*cos(yaw)} ${blue03[2]} 0 0 ${blue03[3]+yaw}" sx="1.2" sy="0.2" sz="0.2" mass="1.0" mat="Gazebo/Blue" />
+    <single_colored_brick id="Blue_brick_04" pose="${blue04[0]*cos(yaw)-blue04[1]*sin(yaw)} ${blue04[0]*sin(yaw)+blue04[1]*cos(yaw)} ${blue04[2]} 0 0 ${blue04[3]+yaw}" sx="1.2" sy="0.2" sz="0.2" mass="1.0" mat="Gazebo/Blue" />
+    <single_colored_brick id="Green_brick_01" pose="${green01[0]*cos(yaw)-green01[1]*sin(yaw)} ${green01[0]*sin(yaw)+green01[1]*cos(yaw)} ${green01[2]} 0 0 ${green01[3]+yaw}" sx="0.6" sy="0.2" sz="0.2" mass="1.0" mat="Gazebo/Green" />
+    <single_colored_brick id="Green_brick_02" pose="${green02[0]*cos(yaw)-green02[1]*sin(yaw)} ${green02[0]*sin(yaw)+green02[1]*cos(yaw)} ${green02[2]} 0 0 ${green02[3]+yaw}" sx="0.6" sy="0.2" sz="0.2" mass="1.0" mat="Gazebo/Green" />
+    <single_colored_brick id="Green_brick_03" pose="${green03[0]*cos(yaw)-green03[1]*sin(yaw)} ${green03[0]*sin(yaw)+green03[1]*cos(yaw)} ${green03[2]} 0 0 ${green03[3]+yaw}" sx="0.6" sy="0.2" sz="0.2" mass="1.0" mat="Gazebo/Green" />
+    <single_colored_brick id="Green_brick_04" pose="${green04[0]*cos(yaw)-green04[1]*sin(yaw)} ${green04[0]*sin(yaw)+green04[1]*cos(yaw)} ${green04[2]} 0 0 ${green04[3]+yaw}" sx="0.6" sy="0.2" sz="0.2" mass="1.0" mat="Gazebo/Green" />
+    <single_colored_brick id="Orange_brick_01" pose="${orange01[0]*cos(yaw)-orange01[1]*sin(yaw)} ${orange01[0]*sin(yaw)+orange01[1]*cos(yaw)} ${orange01[2]} 0 0 ${orange01[3]+yaw}" sx="1.8" sy="0.2" sz="0.2" mass="1.0" mat="Gazebo/Orange" />
+    <single_colored_brick id="Orange_brick_02" pose="${orange02[0]*cos(yaw)-orange02[1]*sin(yaw)} ${orange02[0]*sin(yaw)+orange02[1]*cos(yaw)} ${orange02[2]} 0 0 ${orange02[3]+yaw}" sx="1.8" sy="0.2" sz="0.2" mass="1.0" mat="Gazebo/Orange" />
+    <single_colored_brick id="Orange_brick_03" pose="${orange03[0]*cos(yaw)-orange03[1]*sin(yaw)} ${orange03[0]*sin(yaw)+orange03[1]*cos(yaw)} ${orange03[2]} 0 0 ${orange03[3]+yaw}" sx="1.8" sy="0.2" sz="0.2" mass="1.0" mat="Gazebo/Orange" />
+    <single_colored_brick id="Orange_brick_04" pose="${orange04[0]*cos(yaw)-orange04[1]*sin(yaw)} ${orange04[0]*sin(yaw)+orange04[1]*cos(yaw)} ${orange04[2]} 0 0 ${orange04[3]+yaw}" sx="1.8" sy="0.2" sz="0.2" mass="1.0" mat="Gazebo/Orange" />
   </world>
 </sdf>

Commit message: Standardize challenge 2 arena simulation

File: mbzirc_gazebo_simulation/challenge_worlds/models/ground_plane_asfalt/ground_plane_asfalt.xacro (robot description, xacro)
@@ -10,5 +10,5 @@
             <plane>
               <normal>0 0 1</normal>
-              <size>100 60</size>
+              <size>100 100</size>
             </plane>
           </geometry>
@@ -35,5 +35,5 @@
             <plane>
               <normal>0 0 1</normal>
-              <size>50 60</size>
+              <size>60 50</size>
             </plane>
           </geometry>

File: mbzirc_gazebo_simulation/challenge_worlds/worlds/challenge2.world.xacro (robot description, xacro)
@@ -8,5 +8,6 @@
 <xacro:include filename="$(find challenge_worlds)/urdf/single_colored_brick.xacro" />
 <!-- Global yaw: to change the global position of all the objects in the world -->
-<xacro:property name="yaw" value="0"/>
+<xacro:arg name="arena_yaw" default="0"/>
+<xacro:property name="yaw" value="$(arg arena_yaw)"/>
 <!-- Properties for every object in the world -->
  <!-- 0 => X position , 1 => Y position , 2 => Z position , 3 => Item yaw -->
@@ -15,21 +16,21 @@
 <xacro:property name="green" value="${[0,10,0,0]}"/>
 <xacro:property name="red" value="${[0,-10,0,0]}"/>  -->
-<xacro:property name="ground" value="${[0,0,0,0]}"/>
-<xacro:property name="red01" value="${[0.5,-10.5,0,0]}"/>
-<xacro:property name="red02" value="${[-0.5,-10.5,0,0]}"/>
-<xacro:property name="red03" value="${[-0.5,-9.5,0,0]}"/>
-<xacro:property name="red04" value="${[0.5,-9.5,0,0]}"/>
-<xacro:property name="blue01" value="${[-11,0.5,0,0]}"/>
-<xacro:property name="blue02" value="${[-11,-0.5,0,0]}"/>
-<xacro:property name="blue03" value="${[-9,0.5,0,0]}"/>
-<xacro:property name="blue04" value="${[-9,-0.5,0,0]}"/>
-<xacro:property name="green01" value="${[0.5,10.5,0,0]}"/>
-<xacro:property name="green02" value="${[-0.5,10.5,0,0]}"/>
-<xacro:property name="green03" value="${[0.5,9.5,0,0]}"/>
-<xacro:property name="green04" value="${[-0.5,9.5,0,0]}"/>
-<xacro:property name="orange01" value="${[11,0.5,0,0]}"/>
-<xacro:property name="orange02" value="${[11,-0.5,0,0]}"/>
-<xacro:property name="orange03" value="${[9,0.5,0,0]}"/>
-<xacro:property name="orange04" value="${[9,-0.5,0,0]}"/>
+<xacro:property name="ground" value="${[30,25,0,0]}"/>
+<xacro:property name="red01" value="${[30.5,14.5,0,0]}"/>
+<xacro:property name="red02" value="${[29.5,14.5,0,0]}"/>
+<xacro:property name="red03" value="${[29.5,15.5,0,0]}"/>
+<xacro:property name="red04" value="${[30.5,15.5,0,0]}"/>
+<xacro:property name="blue01" value="${[19,25.5,0,0]}"/>
+<xacro:property name="blue02" value="${[19,24.5,0,0]}"/>
+<xacro:property name="blue03" value="${[21,25.5,0,0]}"/>
+<xacro:property name="blue04" value="${[21,24.5,0,0]}"/>
+<xacro:property name="green01" value="${[30.5,35.5,0,0]}"/>
+<xacro:property name="green02" value="${[29.5,35.5,0,0]}"/>
+<xacro:property name="green03" value="${[30.5,34.5,0,0]}"/>
+<xacro:property name="green04" value="${[29.5,34.5,0,0]}"/>
+<xacro:property name="orange01" value="${[41,25.5,0,0]}"/>
+<xacro:property name="orange02" value="${[41,24.5,0,0]}"/>
+<xacro:property name="orange03" value="${[39,25.5,0,0]}"/>
+<xacro:property name="orange04" value="${[39,24.5,0,0]}"/>
   <world name="default">
     <!-- <include>

Commit message: Set basketball court as arena

File: mbzirc_gazebo_simulation/challenge_worlds/models/ground_plane_asfalt/ground_plane_asfalt.xacro (robot description, xacro)
@@ -35,5 +35,5 @@
             <plane>
               <normal>0 0 1</normal>
-              <size>60 50</size>
+              <size>25.71 15</size>
             </plane>
           </geometry>

File: mbzirc_gazebo_simulation/challenge_worlds/worlds/challenge2.world.xacro (robot description, xacro)
@@ -16,21 +16,21 @@
 <xacro:property name="green" value="${[0,10,0,0]}"/>
 <xacro:property name="red" value="${[0,-10,0,0]}"/>  -->
-<xacro:property name="ground" value="${[30,25,0,0]}"/>
-<xacro:property name="red01" value="${[30.5,14.5,0,0]}"/>
-<xacro:property name="red02" value="${[29.5,14.5,0,0]}"/>
-<xacro:property name="red03" value="${[29.5,15.5,0,0]}"/>
-<xacro:property name="red04" value="${[30.5,15.5,0,0]}"/>
-<xacro:property name="blue01" value="${[19,25.5,0,0]}"/>
-<xacro:property name="blue02" value="${[19,24.5,0,0]}"/>
-<xacro:property name="blue03" value="${[21,25.5,0,0]}"/>
-<xacro:property name="blue04" value="${[21,24.5,0,0]}"/>
-<xacro:property name="green01" value="${[30.5,35.5,0,0]}"/>
-<xacro:property name="green02" value="${[29.5,35.5,0,0]}"/>
-<xacro:property name="green03" value="${[30.5,34.5,0,0]}"/>
-<xacro:property name="green04" value="${[29.5,34.5,0,0]}"/>
-<xacro:property name="orange01" value="${[41,25.5,0,0]}"/>
-<xacro:property name="orange02" value="${[41,24.5,0,0]}"/>
-<xacro:property name="orange03" value="${[39,25.5,0,0]}"/>
-<xacro:property name="orange04" value="${[39,24.5,0,0]}"/>
+<xacro:property name="ground" value="${[12.855,7.5,0,0]}"/>
+<xacro:property name="red01" value="${[5.5,5.5,0,0]}"/>
+<xacro:property name="red02" value="${[5.5,4.5,0,0]}"/>
+<xacro:property name="red03" value="${[4.5,5.5,0,0]}"/>
+<xacro:property name="red04" value="${[4.5,4.5,0,0]}"/>
+<xacro:property name="blue01" value="${[20.5,10.5,0,0]}"/>
+<xacro:property name="blue02" value="${[20.5,9.5,0,0]}"/>
+<!-- <xacro:property name="blue03" value="${[19.5,10.5,0,0]}"/> -->
+<!-- <xacro:property name="blue04" value="${[19.5,9.5,0,0]}"/> -->
+<xacro:property name="green01" value="${[20.5,5.5,0,0]}"/>
+<xacro:property name="green02" value="${[20.5,4.5,0,0]}"/>
+<xacro:property name="green03" value="${[19.5,5.5,0,0]}"/>
+<xacro:property name="green04" value="${[19.5,4.5,0,0]}"/>
+<xacro:property name="orange01" value="${[5.5,10.5,0,0]}"/>
+<xacro:property name="orange02" value="${[5.5,9.5,0,0]}"/>
+<!-- <xacro:property name="orange03" value="${[4.5,10.5,0,0]}"/> -->
+<!-- <xacro:property name="orange04" value="${[4.5,9.5,0,0]}"/> -->
   <world name="default">
     <!-- <include>
@@ -54,6 +54,6 @@
     <single_colored_brick id="Blue_brick_01" pose="${blue01[0]*cos(yaw)-blue01[1]*sin(yaw)} ${blue01[0]*sin(yaw)+blue01[1]*cos(yaw)} ${blue01[2]} 0 0 ${blue01[3]+yaw}" sx="1.2" sy="0.2" sz="0.2" mass="1.0" mat="Gazebo/Blue" />
     <single_colored_brick id="Blue_brick_02" pose="${blue02[0]*cos(yaw)-blue02[1]*sin(yaw)} ${blue02[0]*sin(yaw)+blue02[1]*cos(yaw)} ${blue02[2]} 0 0 ${blue02[3]+yaw}" sx="1.2" sy="0.2" sz="0.2" mass="1.0" mat="Gazebo/Blue" />
-    <single_colored_brick id="Blue_brick_03" pose="${blue03[0]*cos(yaw)-blue03[1]*sin(yaw)} ${blue03[0]*sin(yaw)+blue03[1]*cos(yaw)} ${blue03[2]} 0 0 ${blue03[3]+yaw}" sx="1.2" sy="0.2" sz="0.2" mass="1.0" mat="Gazebo/Blue" />
-    <single_colored_brick id="Blue_brick_04" pose="${blue04[0]*cos(yaw)-blue04[1]*sin(yaw)} ${blue04[0]*sin(yaw)+blue04[1]*cos(yaw)} ${blue04[2]} 0 0 ${blue04[3]+yaw}" sx="1.2" sy="0.2" sz="0.2" mass="1.0" mat="Gazebo/Blue" />
+    <!-- <single_colored_brick id="Blue_brick_03" pose="${blue03[0]*cos(yaw)-blue03[1]*sin(yaw)} ${blue03[0]*sin(yaw)+blue03[1]*cos(yaw)} ${blue03[2]} 0 0 ${blue03[3]+yaw}" sx="1.2" sy="0.2" sz="0.2" mass="1.0" mat="Gazebo/Blue" /> -->
+    <!-- <single_colored_brick id="Blue_brick_04" pose="${blue04[0]*cos(yaw)-blue04[1]*sin(yaw)} ${blue04[0]*sin(yaw)+blue04[1]*cos(yaw)} ${blue04[2]} 0 0 ${blue04[3]+yaw}" sx="1.2" sy="0.2" sz="0.2" mass="1.0" mat="Gazebo/Blue" /> -->
     <single_colored_brick id="Green_brick_01" pose="${green01[0]*cos(yaw)-green01[1]*sin(yaw)} ${green01[0]*sin(yaw)+green01[1]*cos(yaw)} ${green01[2]} 0 0 ${green01[3]+yaw}" sx="0.6" sy="0.2" sz="0.2" mass="1.0" mat="Gazebo/Green" />
     <single_colored_brick id="Green_brick_02" pose="${green02[0]*cos(yaw)-green02[1]*sin(yaw)} ${green02[0]*sin(yaw)+green02[1]*cos(yaw)} ${green02[2]} 0 0 ${green02[3]+yaw}" sx="0.6" sy="0.2" sz="0.2" mass="1.0" mat="Gazebo/Green" />
@@ -62,6 +62,6 @@
     <single_colored_brick id="Orange_brick_01" pose="${orange01[0]*cos(yaw)-orange01[1]*sin(yaw)} ${orange01[0]*sin(yaw)+orange01[1]*cos(yaw)} ${orange01[2]} 0 0 ${orange01[3]+yaw}" sx="1.8" sy="0.2" sz="0.2" mass="1.0" mat="Gazebo/Orange" />
     <single_colored_brick id="Orange_brick_02" pose="${orange02[0]*cos(yaw)-orange02[1]*sin(yaw)} ${orange02[0]*sin(yaw)+orange02[1]*cos(yaw)} ${orange02[2]} 0 0 ${orange02[3]+yaw}" sx="1.8" sy="0.2" sz="0.2" mass="1.0" mat="Gazebo/Orange" />
-    <single_colored_brick id="Orange_brick_03" pose="${orange03[0]*cos(yaw)-orange03[1]*sin(yaw)} ${orange03[0]*sin(yaw)+orange03[1]*cos(yaw)} ${orange03[2]} 0 0 ${orange03[3]+yaw}" sx="1.8" sy="0.2" sz="0.2" mass="1.0" mat="Gazebo/Orange" />
-    <single_colored_brick id="Orange_brick_04" pose="${orange04[0]*cos(yaw)-orange04[1]*sin(yaw)} ${orange04[0]*sin(yaw)+orange04[1]*cos(yaw)} ${orange04[2]} 0 0 ${orange04[3]+yaw}" sx="1.8" sy="0.2" sz="0.2" mass="1.0" mat="Gazebo/Orange" />
+    <!-- <single_colored_brick id="Orange_brick_03" pose="${orange03[0]*cos(yaw)-orange03[1]*sin(yaw)} ${orange03[0]*sin(yaw)+orange03[1]*cos(yaw)} ${orange03[2]} 0 0 ${orange03[3]+yaw}" sx="1.8" sy="0.2" sz="0.2" mass="1.0" mat="Gazebo/Orange" /> -->
+    <!-- <single_colored_brick id="Orange_brick_04" pose="${orange04[0]*cos(yaw)-orange04[1]*sin(yaw)} ${orange04[0]*sin(yaw)+orange04[1]*cos(yaw)} ${orange04[2]} 0 0 ${orange04[3]+yaw}" sx="1.8" sy="0.2" sz="0.2" mass="1.0" mat="Gazebo/Orange" /> -->
   </world>
 </sdf>

Commit message: adjusting arena & standalone bricks

File: mbzirc_gazebo_simulation/challenge_worlds/models/ground_plane_asfalt/ground_plane_asfalt.xacro (robot description, xacro)
@@ -10,5 +10,5 @@
             <plane>
               <normal>0 0 1</normal>
-              <size>100 100</size>
+              <size>50 60</size>
             </plane>
           </geometry>
@@ -35,5 +35,5 @@
             <plane>
               <normal>0 0 1</normal>
-              <size>60 50</size>
+              <size>50 60</size>
             </plane>
           </geometry>

File: mbzirc_gazebo_simulation/challenge_worlds/worlds/challenge2.world.xacro (robot description, xacro)
@@ -15,5 +15,5 @@
     <!-- X'-x= (X-x)*cos(yaw)-(Y-y)*sin(yaw) -->
     <!-- Y'-y= (X-x)*sin(yaw)+(Y-y)*cos(yaw)  -->
-<xacro:property name="ground" value="${[30,25,0,0]}"/>
+<xacro:property name="ground" value="${[25,30,0,0]}"/>
 <!-- UAV BRICKS Location -->
 <!-- Change "basebrick" to modify location and yaw for the entire pile-->

File: mbzirc_gazebo_simulation/challenge_worlds/worlds/challenge3.world.xacro (robot description, xacro)
@@ -37,8 +37,8 @@
 <xacro:property name="f6dp" value="${[b[0]+8.7, b[1]+10, b[2]+12.5, 3.1416]}"/>
 <xacro:property name="f6d" value="${[(f6dp[0]-b[0])*cos(b[3])-(f6dp[1]-b[1])*sin(b[3])+b[0],(f6dp[0]-b[0])*sin(b[3])+(f6dp[1]-b[1])*cos(b[3])+b[1],f6dp[2],f6dp[3]+b[3]]}"/>
-<xacro:property name="f7" value="${[15,10,0,0]}"/>
-<xacro:property name="f8" value="${[20,40,0,-1.570795]}"/>
-<xacro:property name="b" value="${[30,25,0,0]}"/>
-<xacro:property name="g" value="${[30,25,0,0]}"/>
+<xacro:property name="f7" value="${[30,10,0,0]}"/>
+<xacro:property name="f8" value="${[10,40,0,-1.570795]}"/>
+<xacro:property name="b" value="${[20,23,0,0]}"/>
+<xacro:property name="g" value="${[25,30,0,0]}"/>
 <!-- 4.7124 -->
    <!-- The following is the geometric expresion for an axis rotation -->
